File: TSAL/TSAL.sch (KiCad schematic (older format))
At the start: 89 parts, among them P301 CONN_01X02, U301 PQ05RR12, U302 LM555N

Commit message: Add voltage reg and MCP2515 SPI CAN to FS lib
Parts:
- removed P301: CONN_01X02, Molex MiniFit Jr:Molex_39-28-8020, symbol CONN_02_B2B
- removed U301: PQ05RR12, FS FINAL:4 pin reg, symbol PQ05RR12
- removed U302: LM555N, Housings_DIP:DIP-8_W7.62mm, symbol LM555N
- added P?: CONN_01X02, symbol CONN_01X02
- added U?: LM555N, symbol LM555N
- added U?: L78S05CV-DG, TO-220, symbol L78S05CV-DG
Connections:
- no-connect marks 9 -> 8
Changed lines of the file:
@@
 EESchema Schematic File Version 2
+LIBS:FS FINAL
 LIBS:TSAL-rescue
 LIBS:power
@@
 LIBS:contrib
 LIBS:valves
-LIBS:FS FINAL
+LIBS:TSAL-cache
 EELAYER 25 0
 EELAYER END
@@
 Comment4 ""
 $EndDescr
-$Comp
-L LM555N U302
-U 1 1 571D8B4C
-P 4700 1700
-F 0 "U302" H 4700 1700 70  0000 C CNN
-F 1 "LM555N" H 4700 1800 70  0000 C CNN
-F 2 "Housings_DIP:DIP-8_W7.62mm" H 4700 1700 60  0001 C CNN
-F 3 "" H 4700 1700 60  0000 C CNN
-	1    4700 1700
-	1    0    0    -1
-$EndComp
 NoConn ~ 4000 1700
 $Comp
@@
 Text Notes 3500 850  0    60   ~ 0
 TSAL - Oscillator
-$Comp
-L CONN_02_B2B P301
-U 1 1 570D7D07
-P 1200 1750
-F 0 "P301" H 1200 1900 50  0000 C CNN
-F 1 "CONN_01X02" V 1300 1750 50  0000 C CNN
-F 2 "Molex MiniFit Jr:Molex_39-28-8020" H 1200 1750 60  0001 C CNN
-F 3 "" H 1200 1750 60  0000 C CNN
-	1    1200 1750
-	-1   0    0    -1
-$EndComp
-Text HLabel 1400 1800 2    60   Input ~ 0
+Text HLabel 1650 1800 2    60   Input ~ 0
 GND
 Text Label 7500 1400 0    60   ~ 0
@@
 	1    0    0    -1
 $EndComp
-$Comp
-L PQ05RR12 U301
-U 1 1 570AF345
-P 2400 1300
-F 0 "U301" H 2400 1300 60  0000 C CNN
-F 1 "PQ05RR12" H 2400 1400 60  0000 C CNN
-F 2 "FS FINAL:4 pin reg" H 2400 1300 60  0001 C CNN
-F 3 "" H 2400 1300 60  0000 C CNN
-	1    2400 1300
-	1    0    0    -1
-$EndComp
 NoConn ~ 6300 1500
 NoConn ~ 6300 1600
@@
 	1    0    0    -1
 $EndComp
+Text Label 6800 1100 0    60   ~ 0
+5V
+Text HLabel 1650 1700 2    60   Input ~ 0
+12V
+Text HLabel 7100 1100 2    60   Input ~ 0
+12V
 Wire Wire Line
 	4000 1400 3900 1400
@@
 Connection ~ 7000 2300
 Connection ~ 7100 2300
-Wire Wire Line
-	2400 2300 2400 1800
 Connection ~ 3100 2300
-Connection ~ 2400 2300
-NoConn ~ 1900 1500
-Text Label 6800 1100 0    60   ~ 0
-5V
-Wire Wire Line
-	1400 1700 1200 1700
-Wire Wire Line
-	1200 1800 1400 1800
-Text HLabel 1400 1700 2    60   Input ~ 0
+Wire Wire Line
+	1650 1700 1450 1700
+Wire Wire Line
+	1450 1800 1650 1800
+Wire Wire Line
+	7000 1100 7100 1100
+$Comp
+L LM555N U?
+U 1 1 5897EDA1
+P 4700 1700
+F 0 "U?" H 4700 1700 70  0000 C CNN
+F 1 "LM555N" H 4700 1800 70  0000 C CNN
+F 2 "" H 4700 1700 60  0000 C CNN
+F 3 "" H 4700 1700 60  0000 C CNN
+	1    4700 1700
+	1    0    0    -1
+$EndComp
+$Comp
+L CONN_01X02 P?
+U 1 1 5897EFA7
+P 1250 1750
+F 0 "P?" H 1250 1900 50  0000 C CNN
+F 1 "CONN_01X02" V 1350 1750 50  0000 C CNN
+F 2 "" H 1250 1750 50  0000 C CNN
+F 3 "" H 1250 1750 50  0000 C CNN
+	1    1250 1750
+	-1   0    0    1
+$EndComp
+$Comp
+L L78S05CV-DG U?
+U 1 1 5897F17E
+P 2500 1150
+F 0 "U?" H 2300 1350 50  0000 C CNN
+F 1 "L78S05CV-DG" H 2500 1350 50  0000 L CNN
+F 2 "TO-220" H 2500 800 50  0001 C CIN
+F 3 "" H 2500 1150 50  0000 C CNN
+	1    2500 1150
+	1    0    0    -1
+$EndComp
+Wire Wire Line
+	2500 1400 2500 2300
+Connection ~ 2500 2300
+Text HLabel 2100 1100 0    60   Input ~ 0
 12V
-Text HLabel 1900 1100 0    60   Input ~ 0
-12V
-Text HLabel 7100 1100 2    60   Input ~ 0
-12V
-Wire Wire Line
-	7000 1100 7100 1100
 $EndSCHEMATC

Commit message: Revisions for ESF
Parts:
- removed P?: CONN_01X02, symbol CONN_01X02
- added J?: CONN_01X04, symbol CONN_01X04
- added LS?: RTDS Piezo, symbol Speaker
Connections:
- net labels added: +12V, RTDS_OUT, RTDS_SIG, TSAL_SIG
- net labels removed: 12V
- wire segments 86 -> 84
- no-connect marks 8 -> 6
Changed lines of the file:
@@
 	1    0    0    -1
 $EndComp
-Text HLabel 2200 2300 0    60   Input ~ 0
-GND
 Text Notes 3500 850  0    60   ~ 0
 TSAL - Oscillator
-Text HLabel 1650 1800 2    60   Input ~ 0
-GND
 Text Label 7500 1400 0    60   ~ 0
 OSC
 Text Label 900  2800 1    60   ~ 0
 OSC
-Text HLabel 2400 2800 1    60   Input ~ 0
-GND
 $Comp
 L LED_Small D301
@@
 	1    0    0    -1
 $EndComp
-NoConn ~ 6300 1500
 NoConn ~ 6300 1600
 NoConn ~ 6300 1700
 NoConn ~ 6300 2000
-NoConn ~ 7500 1500
 NoConn ~ 7500 1600
 NoConn ~ 7500 1700
@@
 Text Label 6800 1100 0    60   ~ 0
 5V
-Text HLabel 1650 1700 2    60   Input ~ 0
-12V
-Text HLabel 7100 1100 2    60   Input ~ 0
-12V
 Wire Wire Line
 	4000 1400 3900 1400
@@
 Wire Wire Line
 	5400 1400 6300 1400
-Wire Wire Line
-	6300 1900 6200 1900
 Wire Wire Line
 	1200 5500 1100 5500
@@
 Connection ~ 900  5200
 Wire Wire Line
-	2400 2800 2400 7600
-Wire Wire Line
 	900  2800 900  7600
 Connection ~ 5800 1100
-Wire Wire Line
-	6200 1900 6200 1100
-Connection ~ 6200 1100
 Wire Wire Line
 	3100 2000 3100 1100
@@
 Connection ~ 7100 2300
 Connection ~ 3100 2300
-Wire Wire Line
-	1650 1700 1450 1700
-Wire Wire Line
-	1450 1800 1650 1800
-Wire Wire Line
-	7000 1100 7100 1100
 $Comp
 L LM555N U?
@@
 $EndComp
 $Comp
-L CONN_01X02 P?
-U 1 1 5897EFA7
-P 1250 1750
-F 0 "P?" H 1250 1900 50  0000 C CNN
-F 1 "CONN_01X02" V 1350 1750 50  0000 C CNN
-F 2 "" H 1250 1750 50  0000 C CNN
-F 3 "" H 1250 1750 50  0000 C CNN
-	1    1250 1750
-	-1   0    0    1
-$EndComp
-$Comp
 L L78S05CV-DG U?
 U 1 1 5897F17E
@@
 	2500 1400 2500 2300
 Connection ~ 2500 2300
-Text HLabel 2100 1100 0    60   Input ~ 0
-12V
+Wire Wire Line
+	6300 1400 6300 1500
+Wire Wire Line
+	7500 1500 7500 1400
+$Comp
+L CONN_01X04 J?
+U 1 1 58D93057
+P 1250 1850
+F 0 "J?" H 1250 2100 50  0000 C CNN
+F 1 "CONN_01X04" V 1350 1850 50  0000 C CNN
+F 2 "" H 1250 1850 50  0001 C CNN
+F 3 "" H 1250 1850 50  0001 C CNN
+	1    1250 1850
+	-1   0    0    -1
+$EndComp
+Text Label 1450 1800 0    60   ~ 0
+TSAL_SIG
+Text Label 1450 1900 0    60   ~ 0
+RTDS_OUT
+Text Label 6150 1900 1    60   ~ 0
+TSAL_SIG
+Wire Wire Line
+	6150 1900 6300 1900
+$Comp
+L +12V #PWR?
+U 1 1 58D9EAB3
+P 1450 1700
+F 0 "#PWR?" H 1450 1550 50  0001 C CNN
+F 1 "+12V" H 1450 1840 50  0000 C CNN
+F 2 "" H 1450 1700 50  0001 C CNN
+F 3 "" H 1450 1700 50  0001 C CNN
+	1    1450 1700
+	1    0    0    -1
+$EndComp
+$Comp
+L GND #PWR?
+U 1 1 58D9ED99
+P 1450 2000
+F 0 "#PWR?" H 1450 1750 50  0001 C CNN
+F 1 "GND" H 1450 1850 50  0000 C CNN
+F 2 "" H 1450 2000 50  0001 C CNN
+F 3 "" H 1450 2000 50  0001 C CNN
+	1    1450 2000
+	1    0    0    -1
+$EndComp
+$Comp
+L GND #PWR?
+U 1 1 58D9F028
+P 2200 2300
+F 0 "#PWR?" H 2200 2050 50  0001 C CNN
+F 1 "GND" H 2200 2150 50  0000 C CNN
+F 2 "" H 2200 2300 50  0001 C CNN
+F 3 "" H 2200 2300 50  0001 C CNN
+	1    2200 2300
+	1    0    0    -1
+$EndComp
+$Comp
+L +12V #PWR?
+U 1 1 58D9F0EE
+P 2100 1100
+F 0 "#PWR?" H 2100 950 50  0001 C CNN
+F 1 "+12V" H 2100 1240 50  0000 C CNN
+F 2 "" H 2100 1100 50  0001 C CNN
+F 3 "" H 2100 1100 50  0001 C CNN
+	1    2100 1100
+	1    0    0    -1
+$EndComp
+$Comp
+L +12V #PWR?
+U 1 1 58D9F1B4
+P 7000 1100
+F 0 "#PWR?" H 7000 950 50  0001 C CNN
+F 1 "+12V" H 7000 1240 50  0000 C CNN
+F 2 "" H 7000 1100 50  0001 C CNN
+F 3 "" H 7000 1100 50  0001 C CNN
+	1    7000 1100
+	1    0    0    -1
+$EndComp
+$Comp
+L GND #PWR?
+U 1 1 58DA0D98
+P 2400 7800
+F 0 "#PWR?" H 2400 7550 50  0001 C CNN
+F 1 "GND" H 2400 7650 50  0000 C CNN
+F 2 "" H 2400 7800 50  0001 C CNN
+F 3 "" H 2400 7800 50  0001 C CNN
+	1    2400 7800
+	1    0    0    -1
+$EndComp
+Connection ~ 2400 7600
+Wire Wire Line
+	2400 3100 2400 7800
+$Comp
+L Speaker LS?
+U 1 1 58DA5C2D
+P 4300 3150
+F 0 "LS?" H 4350 3375 50  0000 R CNN
+F 1 "RTDS Piezo" H 4350 3300 50  0000 R CNN
+F 2 "" H 4300 2950 50  0001 C CNN
+F 3 "" H 4290 3100 50  0001 C CNN
+	1    4300 3150
+	1    0    0    -1
+$EndComp
+Text Label 4100 3150 2    60   ~ 0
+RTDS_SIG
+$Comp
+L GND #PWR?
+U 1 1 58DA5F1E
+P 4100 3250
+F 0 "#PWR?" H 4100 3000 50  0001 C CNN
+F 1 "GND" H 4100 3100 50  0000 C CNN
+F 2 "" H 4100 3250 50  0001 C CNN
+F 3 "" H 4100 3250 50  0001 C CNN
+	1    4100 3250
+	1    0    0    -1
+$EndComp
 $EndSCHEMATC
