File: TSAL/TSAL.sch (KiCad schematic (older format))
At the start: 90 parts

Commit message: Progress on PE LV and HV boards
Upgraded to Kicad 4.0.7
Parts:
- J?: symbol CONN_01X04 -> Conn_01x04
Connections:
- net labels added: +5V, RTDS_H, SIG_RTDS, SIG_TSAL
- net labels removed: 5V, RTDS_OUT, RTDS_SIG
- wire segments 84 -> 87
- no-connect marks 6 -> 1
Changed lines of the file:
@@
 EESchema Schematic File Version 2
+LIBS:TSAL-rescue
 LIBS:FS FINAL
-LIBS:TSAL-rescue
 LIBS:power
 LIBS:device
@@
 LIBS:contrib
 LIBS:valves
-LIBS:TSAL-cache
 EELAYER 25 0
 EELAYER END
@@
 Text Notes 3500 850  0    60   ~ 0
 TSAL - Oscillator
-Text Label 7500 1400 0    60   ~ 0
-OSC
 Text Label 900  2800 1    60   ~ 0
 OSC
@@
 L SN754410 H301
 U 1 1 570AEAB1
-P 6900 1700
-F 0 "H301" H 6900 1750 60  0000 C CNN
-F 1 "SN754410" H 6900 1650 60  0000 C CNN
-F 2 "Housings_DIP:DIP-16_W7.62mm" H 7100 1100 60  0001 C CNN
-F 3 "" H 7100 1100 60  0000 C CNN
-	1    6900 1700
-	1    0    0    -1
-$EndComp
-NoConn ~ 6300 1600
-NoConn ~ 6300 1700
-NoConn ~ 6300 2000
-NoConn ~ 7500 1600
-NoConn ~ 7500 1700
+P 9100 1700
+F 0 "H301" H 9100 1750 60  0000 C CNN
+F 1 "SN754410" H 9100 1650 60  0000 C CNN
+F 2 "Housings_DIP:DIP-16_W7.62mm" H 9300 1100 60  0001 C CNN
+F 3 "" H 9300 1100 60  0000 C CNN
+	1    9100 1700
+	1    0    0    -1
+$EndComp
 $Comp
 L LED_Small D333
@@
 	1    0    0    -1
 $EndComp
-Text Label 6800 1100 0    60   ~ 0
-5V
 Wire Wire Line
 	4000 1400 3900 1400
@@
 	5400 1850 5400 2000
 Wire Wire Line
-	2900 1100 6800 1100
+	2900 1100 9000 1100
 Wire Wire Line
 	4000 2000 3700 2000
@@
 	5400 2000 5800 2000
 Wire Wire Line
-	2200 2300 7200 2300
+	2200 2300 9400 2300
 Connection ~ 4700 2300
 Wire Wire Line
@@
 Connection ~ 2400 4900
 Wire Wire Line
-	5400 1400 6300 1400
+	5400 1400 8500 1400
 Wire Wire Line
 	1200 5500 1100 5500
@@
 Connection ~ 3100 1100
 Connection ~ 5800 2300
-Connection ~ 6900 2300
-Connection ~ 7000 2300
-Connection ~ 7100 2300
 Connection ~ 3100 2300
 $Comp
@@
 	2500 1400 2500 2300
 Connection ~ 2500 2300
-Wire Wire Line
-	6300 1400 6300 1500
-Wire Wire Line
-	7500 1500 7500 1400
-$Comp
-L CONN_01X04 J?
+$Comp
+L Conn_01x04 J?
 U 1 1 58D93057
-P 1250 1850
-F 0 "J?" H 1250 2100 50  0000 C CNN
-F 1 "CONN_01X04" V 1350 1850 50  0000 C CNN
-F 2 "" H 1250 1850 50  0001 C CNN
-F 3 "" H 1250 1850 50  0001 C CNN
-	1    1250 1850
+P 1250 1800
+F 0 "J?" H 1250 2050 50  0000 C CNN
+F 1 "CONN_01X04" V 1350 1800 50  0000 C CNN
+F 2 "" H 1250 1800 50  0001 C CNN
+F 3 "" H 1250 1800 50  0001 C CNN
+	1    1250 1800
 	-1   0    0    -1
 $EndComp
 Text Label 1450 1800 0    60   ~ 0
+SIG_TSAL
+Text Label 1450 1900 0    60   ~ 0
+SIG_RTDS
+Text Label 8500 1900 2    60   ~ 0
 TSAL_SIG
-Text Label 1450 1900 0    60   ~ 0
-RTDS_OUT
-Text Label 6150 1900 1    60   ~ 0
-TSAL_SIG
-Wire Wire Line
-	6150 1900 6300 1900
 $Comp
 L +12V #PWR?
@@
 L +12V #PWR?
 U 1 1 58D9F1B4
-P 7000 1100
-F 0 "#PWR?" H 7000 950 50  0001 C CNN
-F 1 "+12V" H 7000 1240 50  0000 C CNN
-F 2 "" H 7000 1100 50  0001 C CNN
-F 3 "" H 7000 1100 50  0001 C CNN
-	1    7000 1100
+P 9200 1100
+F 0 "#PWR?" H 9200 950 50  0001 C CNN
+F 1 "+12V" H 9200 1240 50  0000 C CNN
+F 2 "" H 9200 1100 50  0001 C CNN
+F 3 "" H 9200 1100 50  0001 C CNN
+	1    9200 1100
 	1    0    0    -1
 $EndComp
@@
 $EndComp
 Text Label 4100 3150 2    60   ~ 0
-RTDS_SIG
+RTDS_H
 $Comp
 L GND #PWR?
@@
 	1    0    0    -1
 $EndComp
+Connection ~ 9300 2300
+Connection ~ 9200 2300
+Connection ~ 9100 2300
+Wire Wire Line
+	8500 1400 8500 1500
+$Comp
+L +5V #PWR?
+U 1 1 59B27C04
+P 8400 2100
+F 0 "#PWR?" H 8400 1950 50  0001 C CNN
+F 1 "+5V" H 8400 2240 50  0000 C CNN
+F 2 "" H 8400 2100 50  0001 C CNN
+F 3 "" H 8400 2100 50  0001 C CNN
+	1    8400 2100
+	1    0    0    -1
+$EndComp
+Wire Wire Line
+	8500 2000 8500 2100
+Wire Wire Line
+	8500 2100 8400 2100
+$Comp
+L +5V #PWR?
+U 1 1 59B28B57
+P 9000 1100
+F 0 "#PWR?" H 9000 950 50  0001 C CNN
+F 1 "+5V" H 9000 1240 50  0000 C CNN
+F 2 "" H 9000 1100 50  0001 C CNN
+F 3 "" H 9000 1100 50  0001 C CNN
+	1    9000 1100
+	1    0    0    -1
+$EndComp
+Wire Wire Line
+	9700 1400 9700 1500
+Text Label 9700 1500 0    60   ~ 0
+OSC
+Wire Wire Line
+	8500 1600 8500 1700
+Wire Wire Line
+	9700 1700 9700 1600
+Text Label 8500 1700 2    60   ~ 0
+SIG_RTDS
+Text Label 9700 1700 0    60   ~ 0
+RTDS_H
 $EndSCHEMATC

Commit message: Add second piezo to TSAL
Parts:
- added LS?: RTDS Piezo, symbol Speaker
Changed lines of the file:
@@
 EESchema Schematic File Version 2
-LIBS:TSAL-rescue
 LIBS:FS FINAL
 LIBS:power
@@
 Text Label 9700 1700 0    60   ~ 0
 RTDS_H
+$Comp
+L Speaker LS?
+U 1 1 5A59BA97
+P 5250 3150
+F 0 "LS?" H 5300 3375 50  0000 R CNN
+F 1 "RTDS Piezo" H 5300 3300 50  0000 R CNN
+F 2 "" H 5250 2950 50  0001 C CNN
+F 3 "" H 5240 3100 50  0001 C CNN
+	1    5250 3150
+	1    0    0    -1
+$EndComp
+Text Label 5050 3150 2    60   ~ 0
+RTDS_H
+$Comp
+L GND #PWR?
+U 1 1 5A59BA9E
+P 5050 3250
+F 0 "#PWR?" H 5050 3000 50  0001 C CNN
+F 1 "GND" H 5050 3100 50  0000 C CNN
+F 2 "" H 5050 3250 50  0001 C CNN
+F 3 "" H 5050 3250 50  0001 C CNN
+	1    5050 3250
+	1    0    0    -1
+$EndComp
 $EndSCHEMATC
