File: BatteryTempMonitor/BatteryTempMonitor.sch (KiCad schematic (older format))
At the start: 7 parts

Commit message: Fixed battery temp monitor wiring
Connections:
- wire segments 60 -> 70

Commit message: Added voltage regulator, diode, and I/O connectors to CTMS
Parts:
- added D?: D, symbol D
- added P? (x4): CONN_01X08, symbol CONN_01X08
- added P?: CONN_01X06, symbol CONN_01X06
- added U?: L78S05CV-DG, TO-220, symbol L78S05CV-DG
Connections:
- net labels added: +5v, BATT_GND, CANH, CANL, CHIP1, CHIP2, CHIP3, CHIP4, FAULT, SIG1, SIG10, SIG11, SIG12, SIG13, SIG14, SIG15, SIG16, SIG17, SIG18, SIG19, SIG2, SIG20, SIG21, SIG22, SIG23, SIG24, SIG25, SIG26, SIG27, SIG28, SIG3, SIG4, SIG5, SIG6, SIG7, SIG8, SIG9, SYS_GND
- wire segments 70 -> 102

Commit message: Clean up LV accumulator schematic
Need to solidify connections between accumulator LV board and temp board
Parts:
- removed P?: CONN_01X06, symbol CONN_01X06
- added P?: CONN_01X08, symbol CONN_01X08
Connections:
- net labels added: BMS_FLT_5, IMD_FLT_5, IMT_FLT_5, TEMP_FLT
- net labels removed: BATT_GND, FAULT
- wire segments 102 -> 100
- no-connect marks 0 -> 1
Changed lines of the file:
@@
 EESchema Schematic File Version 2
 LIBS:FS FINAL
+LIBS:arduino
 LIBS:BatteryTempMonitor-rescue
 LIBS:power
@@
 LIBS:contrib
 LIBS:valves
-LIBS:arduino
-LIBS:BatteryTempMonitor-cache
 EELAYER 25 0
 EELAYER END
@@
 L GND #PWR?
 U 1 1 58C497C6
-P 2500 2600
-F 0 "#PWR?" H 2500 2350 50  0001 C CNN
-F 1 "GND" H 2500 2450 50  0000 C CNN
-F 2 "" H 2500 2600 50  0000 C CNN
-F 3 "" H 2500 2600 50  0000 C CNN
-	1    2500 2600
+P 2100 2600
+F 0 "#PWR?" H 2100 2350 50  0001 C CNN
+F 1 "GND" H 2100 2450 50  0000 C CNN
+F 2 "" H 2100 2600 50  0000 C CNN
+F 3 "" H 2100 2600 50  0000 C CNN
+	1    2100 2600
 	1    0    0    -1
 $EndComp
@@
 	1    0    0    -1
 $EndComp
-$Comp
-L L78S05CV-DG U?
-U 1 1 58D2F2ED
-P 8550 1200
-F 0 "U?" H 8350 1400 50  0000 C CNN
-F 1 "L78S05CV-DG" H 8300 1500 50  0000 L CNN
-F 2 "TO-220" H 8550 850 50  0001 C CIN
-F 3 "" H 8550 1200 50  0000 C CNN
-	1    8550 1200
-	-1   0    0    -1
-$EndComp
 Text Label 900  1400 0    60   ~ 0
 +5v
@@
 L D D?
 U 1 1 58D2F91F
-P 9200 1150
-F 0 "D?" H 9200 1250 50  0000 C CNN
-F 1 "D" H 9200 1050 50  0000 C CNN
-F 2 "" H 9200 1150 50  0000 C CNN
-F 3 "" H 9200 1150 50  0000 C CNN
-	1    9200 1150
+P 9200 800
+F 0 "D?" H 9200 900 50  0000 C CNN
+F 1 "D" H 9200 700 50  0000 C CNN
+F 2 "" H 9200 800 50  0000 C CNN
+F 3 "" H 9200 800 50  0000 C CNN
+	1    9200 800
 	1    0    0    -1
 $EndComp
@@
 L GND #PWR?
 U 1 1 58D2FC7F
-P 9100 1400
-F 0 "#PWR?" H 9100 1150 50  0001 C CNN
-F 1 "GND" H 9100 1250 50  0000 C CNN
-F 2 "" H 9100 1400 50  0000 C CNN
-F 3 "" H 9100 1400 50  0000 C CNN
-	1    9100 1400
-	1    0    0    -1
-$EndComp
-$Comp
-L GND #PWR?
-U 1 1 58D2FDB7
-P 8550 1450
-F 0 "#PWR?" H 8550 1200 50  0001 C CNN
-F 1 "GND" H 8550 1300 50  0000 C CNN
-F 2 "" H 8550 1450 50  0000 C CNN
-F 3 "" H 8550 1450 50  0000 C CNN
-	1    8550 1450
+P 9100 1050
+F 0 "#PWR?" H 9100 800 50  0001 C CNN
+F 1 "GND" H 9100 900 50  0000 C CNN
+F 2 "" H 9100 1050 50  0000 C CNN
+F 3 "" H 9100 1050 50  0000 C CNN
+	1    9100 1050
 	1    0    0    -1
 $EndComp
@@
 Text Label 1650 850  0    60   ~ 0
 CANL
-Text Label 9250 1500 0    60   ~ 0
+Text Label 9250 1150 0    60   ~ 0
 CANH
-Text Label 9250 1600 0    60   ~ 0
+Text Label 9250 1250 0    60   ~ 0
 CANL
-$Comp
-L GND #PWR?
-U 1 1 58D3035B
-P 9100 1700
-F 0 "#PWR?" H 9100 1450 50  0001 C CNN
-F 1 "GND" H 9100 1550 50  0000 C CNN
-F 2 "" H 9100 1700 50  0000 C CNN
-F 3 "" H 9100 1700 50  0000 C CNN
-	1    9100 1700
-	1    0    0    -1
-$EndComp
-Text Label 9250 1800 0    60   ~ 0
-FAULT
-Text Label 9100 1700 0    60   ~ 0
-BATT_GND
-Text Label 9100 1400 0    60   ~ 0
+Text Label 10100 1350 2    60   ~ 0
+TEMP_FLT
+Text Label 9100 1050 0    60   ~ 0
 SYS_GND
 $Comp
@@
 F 3 "" H 10300 2500 50  0000 C CNN
 	1    10300 2500
-	1    0    0    -1
-$EndComp
-$Comp
-L CONN_01X06 P?
-U 1 1 58D30781
-P 10300 1550
-F 0 "P?" H 10300 1900 50  0000 C CNN
-F 1 "CONN_01X06" V 10400 1550 50  0000 C CNN
-F 2 "" H 10300 1550 50  0000 C CNN
-F 3 "" H 10300 1550 50  0000 C CNN
-	1    10300 1550
 	1    0    0    -1
 $EndComp
@@
 	4150 2100 4300 2100
 Wire Wire Line
-	2850 2400 2500 2400
-Wire Wire Line
-	2500 2400 2500 2600
+	2100 2400 2850 2400
 Wire Wire Line
 	2200 1400 1950 1400
@@
 	6800 1450 6900 1450
 Wire Wire Line
-	10100 1300 9400 1300
-Wire Wire Line
-	9400 1300 9400 1150
-Wire Wire Line
-	9400 1150 9350 1150
-Wire Wire Line
-	8950 1150 9050 1150
-Wire Wire Line
-	9100 1400 10100 1400
-Wire Wire Line
-	10100 1500 9250 1500
-Wire Wire Line
-	10100 1600 9250 1600
-Wire Wire Line
-	10100 1700 9100 1700
-Wire Wire Line
-	10100 1800 9250 1800
+	10100 950  9400 950
+Wire Wire Line
+	9400 950  9400 800
+Wire Wire Line
+	9400 800  9350 800
+Wire Wire Line
+	8950 800  9050 800
+Wire Wire Line
+	9100 1050 10100 1050
+Wire Wire Line
+	10100 1150 9250 1150
+Wire Wire Line
+	10100 1250 9250 1250
 Wire Wire Line
 	10100 2150 9800 2150
@@
 Text Label 5600 1200 2    60   ~ 0
 CHIP1
+Wire Wire Line
+	2100 2400 2100 2600
+Text Label 2850 2700 2    60   ~ 0
+IMD_FLT_5
+Text Label 2850 2800 2    60   ~ 0
+BMS_FLT_5
+$Comp
+L GND #PWR?
+U 1 1 58D2FDB7
+P 8550 1100
+F 0 "#PWR?" H 8550 850 50  0001 C CNN
+F 1 "GND" H 8550 950 50  0000 C CNN
+F 2 "" H 8550 1100 50  0000 C CNN
+F 3 "" H 8550 1100 50  0000 C CNN
+	1    8550 1100
+	1    0    0    -1
+$EndComp
+$Comp
+L L78S05CV-DG U?
+U 1 1 58D2F2ED
+P 8550 850
+F 0 "U?" H 8350 1050 50  0000 C CNN
+F 1 "L78S05CV-DG" H 8300 1150 50  0000 L CNN
+F 2 "TO-220" H 8550 500 50  0001 C CIN
+F 3 "" H 8550 850 50  0000 C CNN
+	1    8550 850
+	-1   0    0    -1
+$EndComp
+Text Label 2850 2600 2    60   ~ 0
+TEMP_FLT
+$Comp
+L CONN_01X08 P?
+U 1 1 59A3AF94
+P 10300 1300
+F 0 "P?" H 10300 1750 50  0000 C CNN
+F 1 "CONN_01X08" V 10400 1300 50  0000 C CNN
+F 2 "" H 10300 1300 50  0000 C CNN
+F 3 "" H 10300 1300 50  0000 C CNN
+	1    10300 1300
+	1    0    0    -1
+$EndComp
+Text Label 10100 1450 2    60   ~ 0
+IMT_FLT_5
+Text Label 10100 1550 2    60   ~ 0
+BMS_FLT_5
+NoConn ~ 10100 1650
 $EndSCHEMATC

Commit message: Add connections to temp board for isolation and fault feedback
Parts:
- removed D?: D, symbol D
- removed P?: CONN_01X08, symbol CONN_01X08
- removed U?: L78S05CV-DG, TO-220, symbol L78S05CV-DG
- added C? (x2): 100uF, symbol CP
- added C? (x2): CP, symbol CP
- added DC?: RDD08110S12, symbol RDD08110S12
- added P?: HV Connection, symbol CONN_01X02
- added P?: CONN_01X10, symbol CONN_01X10
- added U?: DK1A1B-12V, symbol DK1A1B-12V
- added U?: LM7805, symbol LM7805
Connections:
- net labels added: +12V, 5V_HV, BMS_FLT_LATCHED, IMD_FLT_LATCHED, TEMP_FLT_LATCHED, TS_GND
- net labels removed: BMS_FLT_5, IMD_FLT_5, IMT_FLT_5
- wire segments 100 -> 108
- no-connect marks 1 -> 4

Commit message: Progress on PE LV and HV boards
Upgraded to Kicad 4.0.7
Parts:
- removed U?: stm_nucleo_FK303K8, arduino:arduino_mini, symbol stm_nucleo_FK303K8
- removed U?: LM7805, symbol LM7805
- added U?: stm_nucleo_F303K8, arduino:arduino_mini, symbol stm_nucleo_F303K8
- added U?: L7805, symbol L7805
- P? (x4): symbol CONN_01X08 -> Conn_01x08
- P?: symbol CONN_01X02 -> Conn_01x02
- P?: symbol CONN_01X10 -> Conn_01x10
Connections:
- wire segments 108 -> 110
Changed lines of the file:
@@
 EESchema Schematic File Version 2
 LIBS:FS FINAL
-LIBS:arduino
-LIBS:BatteryTempMonitor-rescue
 LIBS:power
 LIBS:device
@@
 $EndComp
 $Comp
-L stm_nucleo_FK303K8 U?
-U 1 1 58C48709
-P 3500 2950
-F 0 "U?" H 3500 2300 70  0000 C CNN
-F 1 "stm_nucleo_FK303K8" H 3450 2100 70  0000 C CNN
-F 2 "arduino:arduino_mini" H 3550 1600 60  0001 C CNN
-F 3 "" H 4100 3100 60  0001 C CNN
-	1    3500 2950
-	1    0    0    -1
-$EndComp
-$Comp
 L MCP3008 U?
 U 1 1 58C48E77
@@
 SYS_GND
 $Comp
-L CONN_01X08 P?
+L Conn_01x08 P?
 U 1 1 58D30739
-P 10300 2500
-F 0 "P?" H 10300 2950 50  0000 C CNN
-F 1 "CONN_01X08" V 10400 2500 50  0000 C CNN
-F 2 "" H 10300 2500 50  0000 C CNN
-F 3 "" H 10300 2500 50  0000 C CNN
-	1    10300 2500
-	1    0    0    -1
-$EndComp
-$Comp
-L CONN_01X08 P?
+P 10300 2450
+F 0 "P?" H 10300 2900 50  0000 C CNN
+F 1 "CONN_01X08" V 10400 2450 50  0000 C CNN
+F 2 "" H 10300 2450 50  0000 C CNN
+F 3 "" H 10300 2450 50  0000 C CNN
+	1    10300 2450
+	1    0    0    -1
+$EndComp
+$Comp
+L Conn_01x08 P?
 U 1 1 58D3080F
-P 10300 3450
-F 0 "P?" H 10300 3900 50  0000 C CNN
-F 1 "CONN_01X08" V 10400 3450 50  0000 C CNN
-F 2 "" H 10300 3450 50  0000 C CNN
-F 3 "" H 10300 3450 50  0000 C CNN
-	1    10300 3450
-	1    0    0    -1
-$EndComp
-$Comp
-L CONN_01X08 P?
+P 10300 3400
+F 0 "P?" H 10300 3850 50  0000 C CNN
+F 1 "CONN_01X08" V 10400 3400 50  0000 C CNN
+F 2 "" H 10300 3400 50  0000 C CNN
+F 3 "" H 10300 3400 50  0000 C CNN
+	1    10300 3400
+	1    0    0    -1
+$EndComp
+$Comp
+L Conn_01x08 P?
 U 1 1 58D3084E
-P 10300 4400
-F 0 "P?" H 10300 4850 50  0000 C CNN
-F 1 "CONN_01X08" V 10400 4400 50  0000 C CNN
-F 2 "" H 10300 4400 50  0000 C CNN
-F 3 "" H 10300 4400 50  0000 C CNN
-	1    10300 4400
-	1    0    0    -1
-$EndComp
-$Comp
-L CONN_01X08 P?
+P 10300 4350
+F 0 "P?" H 10300 4800 50  0000 C CNN
+F 1 "CONN_01X08" V 10400 4350 50  0000 C CNN
+F 2 "" H 10300 4350 50  0000 C CNN
+F 3 "" H 10300 4350 50  0000 C CNN
+	1    10300 4350
+	1    0    0    -1
+$EndComp
+$Comp
+L Conn_01x08 P?
 U 1 1 58D308C3
-P 10300 5350
-F 0 "P?" H 10300 5800 50  0000 C CNN
-F 1 "CONN_01X08" V 10400 5350 50  0000 C CNN
-F 2 "" H 10300 5350 50  0000 C CNN
-F 3 "" H 10300 5350 50  0000 C CNN
-	1    10300 5350
+P 10300 5300
+F 0 "P?" H 10300 5750 50  0000 C CNN
+F 1 "CONN_01X08" V 10400 5300 50  0000 C CNN
+F 2 "" H 10300 5300 50  0000 C CNN
+F 3 "" H 10300 5300 50  0000 C CNN
+	1    10300 5300
 	1    0    0    -1
 $EndComp
@@
 $EndComp
 $Comp
-L CONN_01X02 P?
+L Conn_01x02 P?
 U 1 1 59A6133D
 P 900 6950
@@
 $EndComp
 $Comp
-L CONN_01X10 P?
+L Conn_01x10 P?
 U 1 1 59A61BA1
-P 10300 1300
-F 0 "P?" H 10300 1850 50  0000 C CNN
-F 1 "CONN_01X10" V 10400 1300 50  0000 C CNN
-F 2 "" H 10300 1300 50  0000 C CNN
-F 3 "" H 10300 1300 50  0000 C CNN
-	1    10300 1300
+P 10300 1250
+F 0 "P?" H 10300 1800 50  0000 C CNN
+F 1 "CONN_01X10" V 10400 1250 50  0000 C CNN
+F 2 "" H 10300 1250 50  0000 C CNN
+F 3 "" H 10300 1250 50  0000 C CNN
+	1    10300 1250
 	1    0    0    -1
 $EndComp
@@
 NoConn ~ 1650 6800
 NoConn ~ 3850 7000
-$Comp
-L LM7805 U?
-U 1 1 59A62DDE
-P 5650 7050
-F 0 "U?" H 5800 6854 50  0000 C CNN
-F 1 "LM7805" H 5650 7250 50  0000 C CNN
-F 2 "" H 5650 7050 50  0000 C CNN
-F 3 "" H 5650 7050 50  0000 C CNN
-	1    5650 7050
-	1    0    0    -1
-$EndComp
 Wire Wire Line
 	1300 700  1250 700
@@
 TS_GND
 Connection ~ 6050 7300
+$Comp
+L stm_nucleo_F303K8 U?
+U 1 1 59B244FE
+P 3500 2950
+F 0 "U?" H 3500 2300 70  0000 C CNN
+F 1 "stm_nucleo_F303K8" H 3450 2100 70  0000 C CNN
+F 2 "arduino:arduino_mini" H 3550 1600 60  0001 C CNN
+F 3 "" H 4100 3100 60  0001 C CNN
+	1    3500 2950
+	1    0    0    -1
+$EndComp
+Wire Wire Line
+	6050 7000 5950 7000
+Wire Wire Line
+	5250 7000 5350 7000
+$Comp
+L L7805 U?
+U 1 1 59B246B7
+P 5650 7000
+F 0 "U?" H 5500 7125 50  0000 C CNN
+F 1 "L7805" H 5650 7125 50  0000 L CNN
+F 2 "" H 5675 6850 50  0001 L CIN
+F 3 "" H 5650 6950 50  0001 C CNN
+	1    5650 7000
+	1    0    0    -1
+$EndComp
 $EndSCHEMATC

Commit message: Hopefully finalize PCB schematics
Changed lines of the file:
@@
 L Conn_01x02 P?
 U 1 1 59A6133D
-P 900 6950
-F 0 "P?" H 900 7100 50  0000 C CNN
-F 1 "HV Connection" V 1000 6950 50  0000 C CNN
-F 2 "" H 900 6950 50  0000 C CNN
-F 3 "" H 900 6950 50  0000 C CNN
-	1    900  6950
+P 900 6900
+F 0 "P?" H 900 7050 50  0000 C CNN
+F 1 "HV Connection" V 1000 6900 50  0000 C CNN
+F 2 "" H 900 6900 50  0000 C CNN
+F 3 "" H 900 6900 50  0000 C CNN
+	1    900  6900
 	-1   0    0    -1
 $EndComp

Commit message: Updated non-modular temp and added SPI isolator chip
Parts:
- removed P?: CONN_01X10, symbol Conn_01x10
- removed U?: L7805, symbol L7805
- added C?: C_Bypass, symbol C_Small
- added P?: CONN_01X10, symbol CONN_01X10
- added SPI_ISLTR?: ADUM4154ARIZ, symbol ADUM4154ARIZ
- added U?: LD1117V33, TO-220, symbol LD1117V33
- P? (x4): symbol Conn_01x08 -> CONN_01X08
- P?: symbol Conn_01x02 -> CONN_01X02
Connections:
- net labels added: +3.3V, 3.3V_HV, GND_HV
- net labels removed: +5v, 5V_HV, SYS_GND, TS_GND
- wire segments 110 -> 118
- no-connect marks 4 -> 7

Commit message: Changed vcc1 (digital supply) of CAN transceiver to 3.3V
Connections:
- wire segments 118 -> 117
Changed lines of the file:
@@
 	8450 2000 8650 2000
-Wire Wire Line
-	950  2200 950  2000
 Wire Wire Line
 	5150 2700 4850 2700
@@
 Wire Notes Line
 	9700 550  5750 550
+$Comp
+L +3.3V #PWR?
+U 1 1 59C08CED
+P 950 2200
+F 0 "#PWR?" H 950 2050 50  0001 C CNN
+F 1 "+3.3V" H 950 2340 50  0000 C CNN
+F 2 "" H 950 2200 50  0000 C CNN
+F 3 "" H 950 2200 50  0000 C CNN
+	1    950  2200
+	1    0    0    -1
+$EndComp
 $EndSCHEMATC
