File: BatteryTempMonitor/BatteryTempMonitor.sch (KiCad schematic (older format))
At the start: 22 parts

Commit message: Added bypass cap for HV side of SPI isolator
Parts:
- added C?: .1uF, symbol C_Small
- C?: value C_Bypass -> .1uF
Connections:
- wire segments 117 -> 136
Changed lines of the file:
@@
 EESchema Schematic File Version 2
-LIBS:BatteryTempMonitor-rescue
 LIBS:FS FINAL
 LIBS:power
@@
 LIBS:contrib
 LIBS:valves
-LIBS:BatteryTempMonitor-cache
 EELAYER 25 0
 EELAYER END
@@
 Text Label 7600 5750 2    60   ~ 0
 3.3V_HV
-Text Label 6450 3000 1    60   ~ 0
+Text Label 6450 2700 0    60   ~ 0
 3.3V_HV
 $Comp
 L ADUM4154ARIZ SPI_ISLTR?
 U 1 1 59BF1149
-P 5050 2900
-F 0 "SPI_ISLTR?" H 5750 3100 60  0000 C CNN
-F 1 "ADUM4154ARIZ" H 5800 3000 60  0000 C CNN
-F 2 "" H 5800 2940 60  0001 C CNN
-F 3 "" H 4400 3000 60  0000 C CNN
-	1    5050 2900
+P 4900 2900
+F 0 "SPI_ISLTR?" H 5600 3100 60  0000 C CNN
+F 1 "ADUM4154ARIZ" H 5650 3000 60  0000 C CNN
+F 2 "" H 5650 2940 60  0001 C CNN
+F 3 "" H 4250 3000 60  0000 C CNN
+	1    4900 2900
 	1    0    0    -1
 $EndComp
@@
 P 4850 2900
 F 0 "C?" H 4860 2970 50  0000 L CNN
-F 1 "C_Bypass" V 5000 2750 50  0000 L CNN
+F 1 ".1uF" V 4700 2800 50  0000 L CNN
 F 2 "" H 4850 2900 50  0000 C CNN
 F 3 "" H 4850 2900 50  0000 C CNN
@@
 	1    0    0    -1
 $EndComp
-NoConn ~ 5150 3900
-NoConn ~ 6450 3900
-NoConn ~ 5150 3800
+NoConn ~ 5000 3900
+NoConn ~ 6300 3900
+NoConn ~ 5000 3800
 Text Label 8650 2000 0    60   ~ 0
 GND_HV
@@
 	10800 5650 10500 5650
 Wire Bus Line
-	10400 2000 10400 2700
-Wire Bus Line
-	10400 2950 10400 3650
-Wire Bus Line
-	10400 3900 10400 4600
-Wire Bus Line
-	10400 4850 10400 5550
+	10400 2000 10400 2100
+Wire Bus Line
+	10400 2100 10400 2200
+Wire Bus Line
+	10400 2200 10400 2300
+Wire Bus Line
+	10400 2300 10400 2400
+Wire Bus Line
+	10400 2400 10400 2500
+Wire Bus Line
+	10400 2500 10400 2600
+Wire Bus Line
+	10400 2600 10400 2700
+Wire Bus Line
+	10400 2950 10400 3050
+Wire Bus Line
+	10400 3050 10400 3150
+Wire Bus Line
+	10400 3150 10400 3250
+Wire Bus Line
+	10400 3250 10400 3350
+Wire Bus Line
+	10400 3350 10400 3450
+Wire Bus Line
+	10400 3450 10400 3550
+Wire Bus Line
+	10400 3550 10400 3650
+Wire Bus Line
+	10400 3900 10400 4000
+Wire Bus Line
+	10400 4000 10400 4100
+Wire Bus Line
+	10400 4100 10400 4200
+Wire Bus Line
+	10400 4200 10400 4300
+Wire Bus Line
+	10400 4300 10400 4400
+Wire Bus Line
+	10400 4400 10400 4500
+Wire Bus Line
+	10400 4500 10400 4600
+Wire Bus Line
+	10400 4850 10400 4950
+Wire Bus Line
+	10400 4950 10400 5050
+Wire Bus Line
+	10400 5050 10400 5150
+Wire Bus Line
+	10400 5150 10400 5250
+Wire Bus Line
+	10400 5250 10400 5350
+Wire Bus Line
+	10400 5350 10400 5450
+Wire Bus Line
+	10400 5450 10400 5550
 Wire Bus Line
 	8800 5050 8800 5750
@@
 	2250 7400 2100 7400
 Wire Wire Line
-	4850 7300 6350 7300
+	4850 7300 5250 7300
+Wire Wire Line
+	5250 7300 5750 7300
+Wire Wire Line
+	5750 7300 6200 7300
+Wire Wire Line
+	6200 7300 6350 7300
 Wire Wire Line
 	4850 6800 5250 6800
@@
 	1300 7700 3850 7700
 Wire Wire Line
-	3850 7700 3850 7200
+	3850 7700 3850 7300
+Wire Wire Line
+	3850 7300 3850 7200
 Connection ~ 3850 7300
 Wire Wire Line
-	2250 6900 3850 6900
+	2250 6900 2600 6900
+Wire Wire Line
+	2600 6900 3150 6900
+Wire Wire Line
+	3150 6900 3850 6900
 Wire Wire Line
 	3850 6900 3850 6800
@@
 	5250 7000 5350 7000
 Wire Wire Line
-	4850 3100 5150 3100
+	4850 3100 5000 3100
 Wire Wire Line
 	4150 3400 4950 3400
@@
 	4950 3400 4950 3200
 Wire Wire Line
-	4950 3200 5150 3200
+	4950 3200 5000 3200
 Wire Wire Line
 	4150 3200 4750 3200
@@
 	4750 3200 4750 3300
 Wire Wire Line
-	4750 3300 5150 3300
+	4750 3300 5000 3300
 Wire Wire Line
 	4150 3300 4650 3300
@@
 	5000 3350 5000 3400
 Wire Wire Line
-	5000 3400 5150 3400
-Wire Wire Line
-	4150 3500 5150 3500
-Wire Wire Line
-	4150 3600 5150 3600
-Wire Wire Line
-	4150 3700 5150 3700
-Wire Wire Line
-	5150 2700 5150 3000
+	4150 3500 5000 3500
+Wire Wire Line
+	4150 3600 5000 3600
+Wire Wire Line
+	4150 3700 5000 3700
+Wire Wire Line
+	5000 2700 5000 3000
 Wire Wire Line
 	4850 2700 4850 2800
@@
 Connection ~ 4850 2700
 Wire Wire Line
-	6450 3200 7550 3200
-Wire Wire Line
-	6850 1000 6850 3200
+	6300 3200 6850 3200
+Wire Wire Line
+	6850 3200 7550 3200
+Wire Wire Line
+	6850 1000 6850 2350
+Wire Wire Line
+	6850 2350 6850 3200
 Wire Wire Line
 	6850 1000 7950 1000
@@
 Connection ~ 6850 2350
 Wire Wire Line
-	7550 3200 7550 5050
+	7550 3200 7550 3700
+Wire Wire Line
+	7550 3700 7550 5050
 Wire Wire Line
 	7550 3700 7950 3700
@@
 Connection ~ 7550 3700
 Wire Wire Line
-	6450 3300 7450 3300
-Wire Wire Line
-	6950 1100 6950 3300
+	6300 3300 6950 3300
+Wire Wire Line
+	6950 3300 7450 3300
+Wire Wire Line
+	6950 1100 6950 2450
+Wire Wire Line
+	6950 2450 6950 3300
 Wire Wire Line
 	6950 1100 7950 1100
 Wire Wire Line
-	6450 3400 7350 3400
-Wire Wire Line
-	7050 1200 7050 3400
+	6300 3400 7050 3400
+Wire Wire Line
+	7050 3400 7350 3400
+Wire Wire Line
+	7050 1200 7050 2550
+Wire Wire Line
+	7050 2550 7050 3400
 Wire Wire Line
 	7050 1200 7950 1200
 Wire Wire Line
-	6450 3500 7150 3500
+	6300 3500 7150 3500
 Wire Wire Line
 	7150 3500 7150 1300
@@
 Connection ~ 7050 2550
 Wire Wire Line
-	6450 3600 7250 3600
+	6300 3600 7250 3600
 Wire Wire Line
 	7250 3600 7250 2650
@@
 	7250 2650 7600 2650
 Wire Wire Line
-	7450 3300 7450 5150
+	7450 3300 7450 3800
+Wire Wire Line
+	7450 3800 7450 5150
 Wire Wire Line
 	7450 3800 7950 3800
 Connection ~ 6950 3300
 Wire Wire Line
-	7350 3400 7350 5250
+	7350 3400 7350 3900
+Wire Wire Line
+	7350 3900 7350 5250
 Wire Wire Line
 	7350 3900 7950 3900
 Connection ~ 7050 3400
 Wire Wire Line
-	6450 3700 7250 3700
+	6300 3700 7250 3700
 Wire Wire Line
 	7250 3700 7250 4000
@@
 Connection ~ 7350 3900
 Wire Wire Line
-	6450 3800 7150 3800
+	6300 3800 7150 3800
 Wire Wire Line
 	7150 3800 7150 5350
@@
 	8450 2000 8650 2000
 Wire Wire Line
-	5150 2700 4850 2700
+	5000 2700 4850 2700
 Wire Wire Line
 	4150 4000 4300 4000
@@
 	1    0    0    -1
 $EndComp
+$Comp
+L C_Small C?
+U 1 1 59C09207
+P 6450 2900
+F 0 "C?" H 6460 2970 50  0000 L CNN
+F 1 ".1uF" V 6600 2850 50  0000 L CNN
+F 2 "" H 6450 2900 50  0000 C CNN
+F 3 "" H 6450 2900 50  0000 C CNN
+	1    6450 2900
+	1    0    0    -1
+$EndComp
+Text Label 6450 3100 0    60   ~ 0
+GND_HV
+Wire Wire Line
+	6300 3000 6300 2700
+Wire Wire Line
+	6300 2700 6450 2700
+Wire Wire Line
+	6450 2700 6450 2800
+Wire Wire Line
+	6450 3000 6450 3100
+Wire Wire Line
+	6450 3100 6300 3100
 $EndSCHEMATC

Commit message: Added bypass caps for all SPI ADC chip vref and digital supplies
Parts:
- added C? (x8): .1uF, symbol C_Small
Connections:
- wire segments 136 -> 139
Changed lines of the file:
@@
 	10800 5650 10500 5650
 Wire Bus Line
-	10400 2000 10400 2100
-Wire Bus Line
-	10400 2100 10400 2200
-Wire Bus Line
-	10400 2200 10400 2300
-Wire Bus Line
-	10400 2300 10400 2400
-Wire Bus Line
-	10400 2400 10400 2500
-Wire Bus Line
-	10400 2500 10400 2600
-Wire Bus Line
-	10400 2600 10400 2700
-Wire Bus Line
-	10400 2950 10400 3050
-Wire Bus Line
-	10400 3050 10400 3150
-Wire Bus Line
-	10400 3150 10400 3250
-Wire Bus Line
-	10400 3250 10400 3350
-Wire Bus Line
-	10400 3350 10400 3450
-Wire Bus Line
-	10400 3450 10400 3550
-Wire Bus Line
-	10400 3550 10400 3650
-Wire Bus Line
-	10400 3900 10400 4000
-Wire Bus Line
-	10400 4000 10400 4100
-Wire Bus Line
-	10400 4100 10400 4200
-Wire Bus Line
-	10400 4200 10400 4300
-Wire Bus Line
-	10400 4300 10400 4400
-Wire Bus Line
-	10400 4400 10400 4500
-Wire Bus Line
-	10400 4500 10400 4600
-Wire Bus Line
-	10400 4850 10400 4950
-Wire Bus Line
-	10400 4950 10400 5050
-Wire Bus Line
-	10400 5050 10400 5150
-Wire Bus Line
-	10400 5150 10400 5250
-Wire Bus Line
-	10400 5250 10400 5350
-Wire Bus Line
-	10400 5350 10400 5450
-Wire Bus Line
-	10400 5450 10400 5550
+	10400 2000 10400 2700
+Wire Bus Line
+	10400 2950 10400 3650
+Wire Bus Line
+	10400 3900 10400 4600
+Wire Bus Line
+	10400 4850 10400 5550
 Wire Bus Line
 	8800 5050 8800 5750
@@
 	2250 7400 2100 7400
 Wire Wire Line
-	4850 7300 5250 7300
-Wire Wire Line
-	5250 7300 5750 7300
-Wire Wire Line
-	5750 7300 6200 7300
-Wire Wire Line
-	6200 7300 6350 7300
+	4850 7300 6350 7300
 Wire Wire Line
 	4850 6800 5250 6800
@@
 	1300 7700 3850 7700
 Wire Wire Line
-	3850 7700 3850 7300
-Wire Wire Line
-	3850 7300 3850 7200
+	3850 7700 3850 7200
 Connection ~ 3850 7300
 Wire Wire Line
-	2250 6900 2600 6900
-Wire Wire Line
-	2600 6900 3150 6900
-Wire Wire Line
-	3150 6900 3850 6900
+	2250 6900 3850 6900
 Wire Wire Line
 	3850 6900 3850 6800
@@
 Connection ~ 4850 2700
 Wire Wire Line
-	6300 3200 6850 3200
-Wire Wire Line
-	6850 3200 7550 3200
-Wire Wire Line
-	6850 1000 6850 2350
-Wire Wire Line
-	6850 2350 6850 3200
+	6300 3200 7550 3200
+Wire Wire Line
+	6850 1000 6850 3200
 Wire Wire Line
 	6850 1000 7950 1000
@@
 Connection ~ 6850 2350
 Wire Wire Line
-	7550 3200 7550 3700
-Wire Wire Line
-	7550 3700 7550 5050
+	7550 3200 7550 5050
 Wire Wire Line
 	7550 3700 7950 3700
@@
 Connection ~ 7550 3700
 Wire Wire Line
-	6300 3300 6950 3300
-Wire Wire Line
-	6950 3300 7450 3300
-Wire Wire Line
-	6950 1100 6950 2450
-Wire Wire Line
-	6950 2450 6950 3300
+	6300 3300 7450 3300
+Wire Wire Line
+	6950 1100 6950 3300
 Wire Wire Line
 	6950 1100 7950 1100
 Wire Wire Line
-	6300 3400 7050 3400
-Wire Wire Line
-	7050 3400 7350 3400
-Wire Wire Line
-	7050 1200 7050 2550
-Wire Wire Line
-	7050 2550 7050 3400
+	6300 3400 7350 3400
+Wire Wire Line
+	7050 1200 7050 3400
 Wire Wire Line
 	7050 1200 7950 1200
@@
 	7250 2650 7600 2650
 Wire Wire Line
-	7450 3300 7450 3800
-Wire Wire Line
-	7450 3800 7450 5150
+	7450 3300 7450 5150
 Wire Wire Line
 	7450 3800 7950 3800
 Connection ~ 6950 3300
 Wire Wire Line
-	7350 3400 7350 3900
-Wire Wire Line
-	7350 3900 7350 5250
+	7350 3400 7350 5250
 Wire Wire Line
 	7350 3900 7950 3900
@@
 	7150 5350 7600 5350
 Wire Wire Line
-	8300 6050 8100 6050
-Wire Wire Line
-	8450 4700 8650 4700
-Wire Wire Line
-	8300 3350 8100 3350
-Wire Wire Line
-	8450 2000 8650 2000
+	7600 6050 9350 6050
+Wire Wire Line
+	8300 4700 9550 4700
+Wire Wire Line
+	7600 3350 9250 3350
+Wire Wire Line
+	8300 2000 9550 2000
 Wire Wire Line
 	5000 2700 4850 2700
@@
 Wire Wire Line
 	6450 3100 6300 3100
+$Comp
+L C_Small C?
+U 1 1 59C0A948
+P 7950 1800
+F 0 "C?" H 7960 1870 50  0000 L CNN
+F 1 ".1uF" V 8100 1750 50  0000 L CNN
+F 2 "" H 7950 1800 50  0000 C CNN
+F 3 "" H 7950 1800 50  0000 C CNN
+	1    7950 1800
+	-1   0    0    1
+$EndComp
+Wire Wire Line
+	7950 1900 8300 1900
+Wire Wire Line
+	8300 1900 8300 2000
+Connection ~ 8450 2000
+$Comp
+L C_Small C?
+U 1 1 59C0AAB5
+P 9550 1400
+F 0 "C?" H 9560 1470 50  0000 L CNN
+F 1 ".1uF" V 9700 1350 50  0000 L CNN
+F 2 "" H 9550 1400 50  0000 C CNN
+F 3 "" H 9550 1400 50  0000 C CNN
+	1    9550 1400
+	-1   0    0    1
+$EndComp
+Wire Wire Line
+	8550 700  9550 700
+Wire Wire Line
+	9550 700  9550 1300
+Wire Wire Line
+	9550 2000 9550 1500
+Connection ~ 8650 2000
+$Comp
+L C_Small C?
+U 1 1 59C0AC9D
+P 9250 2700
+F 0 "C?" H 9260 2770 50  0000 L CNN
+F 1 ".1uF" V 9400 2650 50  0000 L CNN
+F 2 "" H 9250 2700 50  0000 C CNN
+F 3 "" H 9250 2700 50  0000 C CNN
+	1    9250 2700
+	-1   0    0    1
+$EndComp
+$Comp
+L C_Small C?
+U 1 1 59C0AD0F
+P 7600 3150
+F 0 "C?" H 7610 3220 50  0000 L CNN
+F 1 ".1uF" V 7750 3100 50  0000 L CNN
+F 2 "" H 7600 3150 50  0000 C CNN
+F 3 "" H 7600 3150 50  0000 C CNN
+	1    7600 3150
+	1    0    0    -1
+$EndComp
+Wire Wire Line
+	7600 3250 7600 3350
+Connection ~ 8100 3350
+Wire Wire Line
+	9250 3350 9250 2800
+Connection ~ 8300 3350
+Wire Wire Line
+	9250 2600 9250 2050
+Wire Wire Line
+	9250 2050 8200 2050
+$Comp
+L C_Small C?
+U 1 1 59C0B102
+P 9550 4000
+F 0 "C?" H 9560 4070 50  0000 L CNN
+F 1 ".1uF" V 9700 3950 50  0000 L CNN
+F 2 "" H 9550 4000 50  0000 C CNN
+F 3 "" H 9550 4000 50  0000 C CNN
+	1    9550 4000
+	-1   0    0    1
+$EndComp
+$Comp
+L C_Small C?
+U 1 1 59C0B180
+P 7950 4500
+F 0 "C?" H 7960 4570 50  0000 L CNN
+F 1 ".1uF" V 8100 4450 50  0000 L CNN
+F 2 "" H 7950 4500 50  0000 C CNN
+F 3 "" H 7950 4500 50  0000 C CNN
+	1    7950 4500
+	-1   0    0    1
+$EndComp
+Wire Wire Line
+	7950 4600 8300 4600
+Wire Wire Line
+	8300 4600 8300 4700
+Connection ~ 8450 4700
+Wire Wire Line
+	9550 4700 9550 4100
+Connection ~ 8650 4700
+Wire Wire Line
+	9550 3900 9550 3400
+Wire Wire Line
+	9550 3400 8550 3400
+$Comp
+L C_Small C?
+U 1 1 59C0B482
+P 9350 5350
+F 0 "C?" H 9360 5420 50  0000 L CNN
+F 1 ".1uF" V 9500 5300 50  0000 L CNN
+F 2 "" H 9350 5350 50  0000 C CNN
+F 3 "" H 9350 5350 50  0000 C CNN
+	1    9350 5350
+	-1   0    0    1
+$EndComp
+Wire Wire Line
+	9350 5250 9350 4750
+Wire Wire Line
+	9350 4750 8200 4750
+Wire Wire Line
+	9350 6050 9350 5450
+Connection ~ 8300 6050
+$Comp
+L C_Small C?
+U 1 1 59C0B6A8
+P 7600 5850
+F 0 "C?" H 7610 5920 50  0000 L CNN
+F 1 ".1uF" V 7750 5800 50  0000 L CNN
+F 2 "" H 7600 5850 50  0000 C CNN
+F 3 "" H 7600 5850 50  0000 C CNN
+	1    7600 5850
+	-1   0    0    1
+$EndComp
+Wire Wire Line
+	7600 5950 7600 6050
+Connection ~ 8100 6050
 $EndSCHEMATC
