File: PEBoardHV/PEBoardHV.sch (KiCad schematic (older format))
At the start: 39 parts, among them J1 CONN_01X12, J1 Right Panel, J10 HV Cable, J11 TSMPs, J2 Brake Light, J2 TSAL, J3 Left Panel, J4 HVD Interlock, J6 Left 3-Phase Interlock, J6 Wheel Interlocks, J7 Left 3-Phase Interlock, J8 Left Connector (Master), J9 Right Connector (Slave), U1 L78S05CV-DG, U2 ISO1050, U3 PS2501, U4 DK1A1B-12V, U5 DK1A1B-12V, U6 L78S05CV-DG

Commit message: Begin work on moving ECU to PE box
Parts:
- removed H1: SN754410, Housings_DIP:DIP-16_W7.62mm, symbol SN754410
- removed J1: Right Panel, symbol CONN_01X05
- removed J2: Brake Light, symbol CONN_01X03
- removed J2: TSAL, symbol CONN_01X04
- removed J3: Left Panel, symbol CONN_01X02
- removed J4: HVD Interlock, symbol CONN_01X02
- removed J6, J7: Left 3-Phase Interlock, symbol CONN_01X02
- removed J6: Wheel Interlocks, symbol CONN_01X04
- removed U1: L78S05CV-DG, TO-220, symbol L78S05CV-DG
Connections:
- net labels added: AIRS_FINAL, SIG_TSAL
- net labels removed: 12V, 12V_SRC, AIRS_DISCH, AIRS_DISCHARGE, AIRS_IN, AIRS_OUT, AIRS_OUT_LEFT, AIRS_OUT_RIGHT, BRAKE_OUT, BRAKE_SIG, RTDS_OUT, RTDS_SIG, TSAL_SIG, V_L
- wire segments 30 -> 19
- no-connect marks 2 -> 1
Other:
- note removed: "Voltage Regulator LV"

Commit message: Progress on PE LV and HV boards
Upgraded to Kicad 4.0.7
Parts:
- removed J1: CONN_01X12, symbol CONN_01X12
- added J?: To PE LV, symbol Conn_01x06
- J10, J11: symbol CONN_01X02 -> Conn_01x02
- J8: symbol CONN_01X08 -> Conn_01x08
- J9: symbol CONN_01X06 -> Conn_01x06
Other:
- note added: "Needs (Small) Heat Sink!"
Changed lines of the file:
@@
 EESchema Schematic File Version 2
+LIBS:PEBoardHV-rescue
 LIBS:FS FINAL
 LIBS:power
@@
 HV+_SWITCHED_R
 $Comp
-L CONN_01X02 J10
+L Conn_01x02 J10
 U 1 1 58916262
-P 10700 3050
-F 0 "J10" H 10700 3200 50  0000 C CNN
-F 1 "HV Cable" V 10800 3050 50  0000 C CNN
-F 2 "" H 10700 3050 50  0000 C CNN
-F 3 "" H 10700 3050 50  0000 C CNN
-	1    10700 3050
+P 10700 3000
+F 0 "J10" H 10700 3150 50  0000 C CNN
+F 1 "HV Cable" V 10800 3000 50  0000 C CNN
+F 2 "" H 10700 3000 50  0000 C CNN
+F 3 "" H 10700 3000 50  0000 C CNN
+	1    10700 3000
 	1    0    0    -1
 $EndComp
@@
 HV-
 $Comp
-L CONN_01X02 J11
+L Conn_01x02 J11
 U 1 1 5891667E
-P 10700 3600
-F 0 "J11" H 10700 3750 50  0000 C CNN
-F 1 "TSMPs" V 10800 3600 50  0000 C CNN
-F 2 "" H 10700 3600 50  0000 C CNN
-F 3 "" H 10700 3600 50  0000 C CNN
-	1    10700 3600
+P 10700 3550
+F 0 "J11" H 10700 3700 50  0000 C CNN
+F 1 "TSMPs" V 10800 3550 50  0000 C CNN
+F 2 "" H 10700 3550 50  0000 C CNN
+F 3 "" H 10700 3550 50  0000 C CNN
+	1    10700 3550
 	1    0    0    -1
 $EndComp
@@
 $EndComp
 $Comp
-L CONN_01X08 J8
+L Conn_01x08 J8
 U 1 1 58BCB06C
-P 10700 1050
-F 0 "J8" H 10700 1500 50  0000 C CNN
-F 1 "Left Connector (Master)" V 10800 1050 50  0000 C CNN
-F 2 "" H 10700 1050 50  0000 C CNN
-F 3 "" H 10700 1050 50  0000 C CNN
-	1    10700 1050
+P 10700 1000
+F 0 "J8" H 10700 1450 50  0000 C CNN
+F 1 "Left Connector (Master)" V 10800 1000 50  0000 C CNN
+F 2 "" H 10700 1000 50  0000 C CNN
+F 3 "" H 10700 1000 50  0000 C CNN
+	1    10700 1000
 	1    0    0    -1
 $EndComp
@@
 CAN_L_CONTROLLER
 $Comp
-L CONN_01X06 J9
+L Conn_01x06 J9
 U 1 1 58BCB682
-P 10700 2200
-F 0 "J9" H 10700 2550 50  0000 C CNN
-F 1 "Right Connector (Slave)" V 10800 2200 50  0000 C CNN
-F 2 "" H 10700 2200 50  0000 C CNN
-F 3 "" H 10700 2200 50  0000 C CNN
-	1    10700 2200
+P 10700 2150
+F 0 "J9" H 10700 2500 50  0000 C CNN
+F 1 "Right Connector (Slave)" V 10800 2150 50  0000 C CNN
+F 2 "" H 10700 2150 50  0000 C CNN
+F 3 "" H 10700 2150 50  0000 C CNN
+	1    10700 2150
 	1    0    0    -1
 $EndComp
@@
 Text Label 6800 3800 0    60   ~ 0
 HV+
-$Comp
-L CONN_01X12 J1
-U 1 1 58D8D93B
-P 800 1300
-F 0 "J1" H 800 1950 50  0000 C CNN
-F 1 "CONN_01X12" V 900 1300 50  0000 C CNN
-F 2 "" H 800 1300 50  0001 C CNN
-F 3 "" H 800 1300 50  0001 C CNN
-	1    800  1300
-	-1   0    0    -1
-$EndComp
 Text Label 1000 750  0    60   ~ 0
 5V_LV
@@
 Text Label 1000 1050 0    60   ~ 0
 CAN_RX
+Text Notes 7700 1800 0    60   ~ 0
+Needs (Small) Heat Sink!
+$Comp
+L Conn_01x06 J?
+U 1 1 59B25E6D
+P 800 950
+F 0 "J?" H 800 1250 50  0000 C CNN
+F 1 "To PE LV" H 800 550 50  0000 C CNN
+F 2 "" H 800 950 50  0001 C CNN
+F 3 "" H 800 950 50  0001 C CNN
+	1    800  950
+	-1   0    0    -1
+$EndComp
 $EndSCHEMATC

Commit message: Hopefully finalize PCB schematics
Parts:
- removed J?: To PE LV, symbol Conn_01x06
- added C? (x2): CP, symbol CP
- added J?: To PE LV, symbol Conn_01x08
- added J?: HV CAN Debug, symbol Conn_01x03
- added J?: E-Meter Internal, symbol Conn_01x04
- added J?: E-Meter External, symbol Conn_01x04
- added R? (x3): R, symbol R
Connections:
- net labels added: +12V, EM_SIG+, EM_SIG-
- wire segments 19 -> 21
- no-connect marks 1 -> 2
Changed lines of the file:
@@
 EESchema Schematic File Version 2
-LIBS:PEBoardHV-rescue
 LIBS:FS FINAL
 LIBS:power
@@
 L Fuse F1
 U 1 1 58C4C02B
-P 6650 2100
-F 0 "F1" V 6730 2100 50  0000 C CNN
-F 1 "Fuse" V 6575 2100 50  0000 C CNN
-F 2 "" V 6580 2100 50  0000 C CNN
-F 3 "" H 6650 2100 50  0000 C CNN
-	1    6650 2100
+P 6950 2100
+F 0 "F1" V 7030 2100 50  0000 C CNN
+F 1 "Fuse" V 6875 2100 50  0000 C CNN
+F 2 "" V 6880 2100 50  0000 C CNN
+F 3 "" H 6950 2100 50  0000 C CNN
+	1    6950 2100
 	0    1    1    0
 $EndComp
@@
 L Fuse F2
 U 1 1 58C4C0C4
-P 6650 2950
-F 0 "F2" V 6730 2950 50  0000 C CNN
-F 1 "Fuse" V 6575 2950 50  0000 C CNN
-F 2 "" V 6580 2950 50  0000 C CNN
-F 3 "" H 6650 2950 50  0000 C CNN
-	1    6650 2950
+P 6950 2950
+F 0 "F2" V 7030 2950 50  0000 C CNN
+F 1 "Fuse" V 6875 2950 50  0000 C CNN
+F 2 "" V 6880 2950 50  0000 C CNN
+F 3 "" H 6950 2950 50  0000 C CNN
+	1    6950 2950
 	0    1    1    0
 $EndComp
@@
 L Fuse F3
 U 1 1 58C4C15E
-P 6650 3800
-F 0 "F3" V 6730 3800 50  0000 C CNN
-F 1 "Fuse" V 6575 3800 50  0000 C CNN
-F 2 "" V 6580 3800 50  0000 C CNN
-F 3 "" H 6650 3800 50  0000 C CNN
-	1    6650 3800
+P 6950 3800
+F 0 "F3" V 7030 3800 50  0000 C CNN
+F 1 "Fuse" V 6875 3800 50  0000 C CNN
+F 2 "" V 6880 3800 50  0000 C CNN
+F 3 "" H 6950 3800 50  0000 C CNN
+	1    6950 3800
 	0    1    1    0
 $EndComp
@@
 Text Label 4950 4250 2    60   ~ 0
 SIG_TSAL
-Text Label 6800 2100 0    60   ~ 0
+Text Label 7100 2100 0    60   ~ 0
 HV+_SWITCHED_L
-Text Label 6800 2950 0    60   ~ 0
+Text Label 7100 2950 0    60   ~ 0
 HV+_SWITCHED_R
-Text Label 6800 3800 0    60   ~ 0
+Text Label 7100 3800 0    60   ~ 0
 HV+
 Text Label 1000 750  0    60   ~ 0
@@
 Needs (Small) Heat Sink!
 $Comp
-L Conn_01x06 J?
-U 1 1 59B25E6D
+L R R?
+U 1 1 59B378CF
+P 6650 3800
+F 0 "R?" V 6730 3800 50  0000 C CNN
+F 1 "R" V 6650 3800 50  0000 C CNN
+F 2 "" V 6580 3800 50  0001 C CNN
+F 3 "" H 6650 3800 50  0001 C CNN
+	1    6650 3800
+	0    1    1    0
+$EndComp
+$Comp
+L R R?
+U 1 1 59B3797A
+P 6650 2950
+F 0 "R?" V 6730 2950 50  0000 C CNN
+F 1 "R" V 6650 2950 50  0000 C CNN
+F 2 "" V 6580 2950 50  0001 C CNN
+F 3 "" H 6650 2950 50  0001 C CNN
+	1    6650 2950
+	0    1    1    0
+$EndComp
+$Comp
+L R R?
+U 1 1 59B37B6E
+P 6650 2100
+F 0 "R?" V 6730 2100 50  0000 C CNN
+F 1 "R" V 6650 2100 50  0000 C CNN
+F 2 "" V 6580 2100 50  0001 C CNN
+F 3 "" H 6650 2100 50  0001 C CNN
+	1    6650 2100
+	0    1    1    0
+$EndComp
+$Comp
+L Conn_01x08 J?
+U 1 1 59B38655
 P 800 950
-F 0 "J?" H 800 1250 50  0000 C CNN
-F 1 "To PE LV" H 800 550 50  0000 C CNN
+F 0 "J?" H 800 1350 50  0000 C CNN
+F 1 "To PE LV" V 900 950 50  0000 C CNN
 F 2 "" H 800 950 50  0001 C CNN
 F 3 "" H 800 950 50  0001 C CNN
@@
 	-1   0    0    -1
 $EndComp
+$Comp
+L +12V #PWR?
+U 1 1 59B389E9
+P 1000 650
+F 0 "#PWR?" H 1000 500 50  0001 C CNN
+F 1 "+12V" H 1000 790 50  0000 C CNN
+F 2 "" H 1000 650 50  0001 C CNN
+F 3 "" H 1000 650 50  0001 C CNN
+	1    1000 650
+	1    0    0    -1
+$EndComp
+NoConn ~ 1000 1350
+$Comp
+L Conn_01x04 J?
+U 1 1 59B395E2
+P 800 2050
+F 0 "J?" H 800 2250 50  0000 C CNN
+F 1 "E-Meter Internal" V 900 2050 50  0000 C CNN
+F 2 "" H 800 2050 50  0001 C CNN
+F 3 "" H 800 2050 50  0001 C CNN
+	1    800  2050
+	-1   0    0    -1
+$EndComp
+$Comp
+L GND #PWR?
+U 1 1 59B39840
+P 1250 1250
+F 0 "#PWR?" H 1250 1000 50  0001 C CNN
+F 1 "GND" H 1250 1100 50  0000 C CNN
+F 2 "" H 1250 1250 50  0001 C CNN
+F 3 "" H 1250 1250 50  0001 C CNN
+	1    1250 1250
+	1    0    0    -1
+$EndComp
+Wire Wire Line
+	1250 1250 1000 1250
+$Comp
+L GND #PWR?
+U 1 1 59B39AB1
+P 1000 2250
+F 0 "#PWR?" H 1000 2000 50  0001 C CNN
+F 1 "GND" H 1000 2100 50  0000 C CNN
+F 2 "" H 1000 2250 50  0001 C CNN
+F 3 "" H 1000 2250 50  0001 C CNN
+	1    1000 2250
+	1    0    0    -1
+$EndComp
+$Comp
+L +12V #PWR?
+U 1 1 59B39B0B
+P 1000 1950
+F 0 "#PWR?" H 1000 1800 50  0001 C CNN
+F 1 "+12V" H 1000 2090 50  0000 C CNN
+F 2 "" H 1000 1950 50  0001 C CNN
+F 3 "" H 1000 1950 50  0001 C CNN
+	1    1000 1950
+	1    0    0    -1
+$EndComp
+Text Label 1000 2050 0    60   ~ 0
+EM_SIG+
+Text Label 1000 2150 0    60   ~ 0
+EM_SIG-
+$Comp
+L Conn_01x04 J?
+U 1 1 59B39C6F
+P 800 2900
+F 0 "J?" H 800 3100 50  0000 C CNN
+F 1 "E-Meter External" V 900 2900 50  0000 C CNN
+F 2 "" H 800 2900 50  0001 C CNN
+F 3 "" H 800 2900 50  0001 C CNN
+	1    800  2900
+	-1   0    0    -1
+$EndComp
+$Comp
+L GND #PWR?
+U 1 1 59B39C75
+P 1000 3100
+F 0 "#PWR?" H 1000 2850 50  0001 C CNN
+F 1 "GND" H 1000 2950 50  0000 C CNN
+F 2 "" H 1000 3100 50  0001 C CNN
+F 3 "" H 1000 3100 50  0001 C CNN
+	1    1000 3100
+	1    0    0    -1
+$EndComp
+$Comp
+L +12V #PWR?
+U 1 1 59B39C7B
+P 1000 2800
+F 0 "#PWR?" H 1000 2650 50  0001 C CNN
+F 1 "+12V" H 1000 2940 50  0000 C CNN
+F 2 "" H 1000 2800 50  0001 C CNN
+F 3 "" H 1000 2800 50  0001 C CNN
+	1    1000 2800
+	1    0    0    -1
+$EndComp
+Text Label 1000 2900 0    60   ~ 0
+EM_SIG+
+Text Label 1000 3000 0    60   ~ 0
+EM_SIG-
+$Comp
+L CP C?
+U 1 1 59B3ABDF
+P 7750 1300
+F 0 "C?" H 7775 1400 50  0000 L CNN
+F 1 "CP" H 7775 1200 50  0000 L CNN
+F 2 "" H 7788 1150 50  0001 C CNN
+F 3 "" H 7750 1300 50  0001 C CNN
+	1    7750 1300
+	1    0    0    -1
+$EndComp
+$Comp
+L CP C?
+U 1 1 59B3AC80
+P 8550 1300
+F 0 "C?" H 8575 1400 50  0000 L CNN
+F 1 "CP" H 8575 1200 50  0000 L CNN
+F 2 "" H 8588 1150 50  0001 C CNN
+F 3 "" H 8550 1300 50  0001 C CNN
+	1    8550 1300
+	1    0    0    -1
+$EndComp
+Wire Wire Line
+	7750 1450 8550 1450
+Connection ~ 8150 1450
+$Comp
+L Conn_01x03 J?
+U 1 1 59B3870A
+P 10700 4800
+F 0 "J?" H 10700 5000 50  0000 C CNN
+F 1 "HV CAN Debug" V 10800 4800 50  0000 C CNN
+F 2 "" H 10700 4800 50  0001 C CNN
+F 3 "" H 10700 4800 50  0001 C CNN
+	1    10700 4800
+	1    0    0    -1
+$EndComp
+Text Label 10500 4700 2    60   ~ 0
+CAN_H_DEBUG
+Text Label 10500 4800 2    60   ~ 0
+CAN_L_DEBUG
+Text Label 10500 4900 2    60   ~ 0
+HV-
 $EndSCHEMATC

Commit message: Add 3.3v rail to PE HV
Connections:
- net labels added: 3.3V_LV
- no-connect marks 2 -> 1
Changed lines of the file:
@@
 	1    0    0    -1
 $EndComp
-Text Label 1000 1250 0    60   ~ 0
+Text Label 1000 1350 0    60   ~ 0
 GND
 Text Label 4350 1150 0    60   ~ 0
@@
 CAN_TX
 Text Label 5150 850  1    60   ~ 0
-5V_LV
+3.3V_LV
 Text Label 5350 850  1    60   ~ 0
 5V_HV
@@
 Text Label 1000 750  0    60   ~ 0
 5V_LV
-Text Label 1000 850  0    60   ~ 0
+Text Label 1000 950  0    60   ~ 0
 SIG_TSAL
-Text Label 1000 950  0    60   ~ 0
+Text Label 1000 1050 0    60   ~ 0
 CAN_TX
+Text Label 1000 1250 0    60   ~ 0
+AIRS_FINAL
 Text Label 1000 1150 0    60   ~ 0
-AIRS_FINAL
-Text Label 1000 1050 0    60   ~ 0
 CAN_RX
 Text Notes 7700 1800 0    60   ~ 0
@@
 	1    0    0    -1
 $EndComp
-NoConn ~ 1000 1350
 $Comp
 L Conn_01x04 J?
@@
 L GND #PWR?
 U 1 1 59B39840
-P 1250 1250
-F 0 "#PWR?" H 1250 1000 50  0001 C CNN
-F 1 "GND" H 1250 1100 50  0000 C CNN
-F 2 "" H 1250 1250 50  0001 C CNN
-F 3 "" H 1250 1250 50  0001 C CNN
-	1    1250 1250
-	1    0    0    -1
-$EndComp
-Wire Wire Line
-	1250 1250 1000 1250
+P 1250 1350
+F 0 "#PWR?" H 1250 1100 50  0001 C CNN
+F 1 "GND" H 1250 1200 50  0000 C CNN
+F 2 "" H 1250 1350 50  0001 C CNN
+F 3 "" H 1250 1350 50  0001 C CNN
+	1    1250 1350
+	1    0    0    -1
+$EndComp
+Wire Wire Line
+	1250 1350 1000 1350
 $Comp
 L GND #PWR?
@@
 Text Label 10500 4900 2    60   ~ 0
 HV-
+Text Label 1000 850  0    60   ~ 0
+3.3V_LV
 $EndSCHEMATC

Commit message: Add wiring for motor sensors
Parts:
- removed J8: Left Connector (Master), symbol Conn_01x08
- removed J9: Right Connector (Slave), symbol Conn_01x06
- removed J?: To PE LV, symbol Conn_01x08
- added J?: To PE LV, symbol Conn_01x10
- added J?: Left Connector (Master), symbol Conn_01x12
- added J?: Right Connector (Slave), symbol Conn_01x12
- added J?: Slave Motor, symbol Conn_01x08
- added J?: Master Motor, symbol Conn_01x08
Connections:
- net labels added: AIRS_ACC_OUT, AIRS_BEAM_OUT, AIRS_MMASTER_OUT, M_DIG, M_ENC+, M_ENC-, M_POT, M_THERM, S_DIG, S_ENC+, S_ENC-, S_POT, S_THERM
