File: PEBoardHV/PEBoardHV.sch (KiCad schematic (older format))
At the start: 37 parts, among them J10 HV Cable, J11 TSMPs, J8 Left Connector (Master), J9 Right Connector (Slave), U2 ISO1050, U3 PS2501, U4 DK1A1B-12V, U5 DK1A1B-12V, U6 L78S05CV-DG

Commit message: Swapped out vreg for temp system, TS/GLV naming convention, added BMS pull up resistor
Parts:
- added C? (x2): C, symbol C
Connections:
- net labels added: 3.3V_GLV, 3.3V_LV, 5V_GLV, 5V_TS, TS+, TS+_SWITCHED_L, TS+_SWITCHED_R, TS-
- net labels removed: 5V_HV, 5V_LV, HV+, HV+_SWITCHED_L, HV+_SWITCHED_R, HV-
- no-connect marks 2 -> 1
Other:
- note added: "GLV TS"
- note removed: "LV HV"

Commit message: Added charger control pins and organized optos
Parts:
- removed U3: PS2501, symbol PS2501
- added J?: EMeter HV, symbol Conn_01x02
- added U? (x3): PS2501-4, symbol PS2501-4
Connections:
- net labels added: TS+_FUSED
- wire segments 21 -> 23
Changed lines of the file:
@@
 $EndComp
 Text Label 10200 3550 2    60   ~ 0
-TS+
+TS+_FUSED
 Text Label 10500 3950 3    60   ~ 0
 TS-
@@
 $EndComp
 $Comp
-L PS2501 U3
-U 1 1 58C4A1CE
-P 5250 2450
-F 0 "U3" H 5050 2650 50  0000 L CNN
-F 1 "PS2501" H 5050 2250 50  0000 L CNN
-F 2 "" H 5050 2250 50  0000 L CIN
-F 3 "" H 5250 2450 50  0000 L CNN
-	1    5250 2450
-	-1   0    0    -1
-$EndComp
-$Comp
 L R R3
 U 1 1 58C4AF19
@@
 Wire Wire Line
 	6200 3800 6200 4000
-$Comp
-L PS2501 U3
-U 2 1 58C4BBB9
-P 5250 3300
-F 0 "U3" H 5050 3500 50  0000 L CNN
-F 1 "PS2501" H 5050 3100 50  0000 L CNN
-F 2 "" H 5050 3100 50  0000 L CIN
-F 3 "" H 5250 3300 50  0000 L CNN
-	2    5250 3300
-	-1   0    0    -1
-$EndComp
-$Comp
-L PS2501 U3
-U 3 1 58C4BCE9
-P 5250 4150
-F 0 "U3" H 5050 4350 50  0000 L CNN
-F 1 "PS2501" H 5050 3950 50  0000 L CNN
-F 2 "" H 5050 3950 50  0000 L CIN
-F 3 "" H 5250 4150 50  0000 L CNN
-	3    5250 4150
-	-1   0    0    -1
-$EndComp
 $Comp
 L Fuse F1
@@
 Text Label 2950 850  0    60   ~ 0
 3.3V_GLV
+$Comp
+L PS2501-4 U?
+U 1 1 5A5D3FBC
+P 5250 2450
+F 0 "U?" H 5050 2650 50  0000 L CNN
+F 1 "PS2501-4" H 5050 2250 50  0000 L CNN
+F 2 "" H 5050 2250 50  0000 L CIN
+F 3 "" H 5250 2450 50  0000 L CNN
+	1    5250 2450
+	-1   0    0    -1
+$EndComp
+$Comp
+L PS2501-4 U?
+U 2 1 5A5D4061
+P 5250 3300
+F 0 "U?" H 5050 3500 50  0000 L CNN
+F 1 "PS2501-4" H 5050 3100 50  0000 L CNN
+F 2 "" H 5050 3100 50  0000 L CIN
+F 3 "" H 5250 3300 50  0000 L CNN
+	2    5250 3300
+	-1   0    0    -1
+$EndComp
+$Comp
+L PS2501-4 U?
+U 3 1 5A5D40FC
+P 5250 4150
+F 0 "U?" H 5050 4350 50  0000 L CNN
+F 1 "PS2501-4" H 5050 3950 50  0000 L CNN
+F 2 "" H 5050 3950 50  0000 L CIN
+F 3 "" H 5250 4150 50  0000 L CNN
+	3    5250 4150
+	-1   0    0    -1
+$EndComp
+$Comp
+L Conn_01x02 J?
+U 1 1 5A5D5996
+P 10700 5300
+F 0 "J?" H 10700 5400 50  0000 C CNN
+F 1 "EMeter HV" H 10700 5100 50  0000 C CNN
+F 2 "" H 10700 5300 50  0001 C CNN
+F 3 "" H 10700 5300 50  0001 C CNN
+	1    10700 5300
+	1    0    0    -1
+$EndComp
+Wire Wire Line
+	6800 3800 6800 3500
+Text Label 6800 3500 0    60   ~ 0
+TS+_FUSED
+Text Label 10500 5400 2    60   ~ 0
+TS+_FUSED
+Wire Wire Line
+	10500 5300 10500 5400
 $EndSCHEMATC

Commit message: Begin PE/dash footprints, continue with accumulator footprints
Parts:
- C1, C2, C3, C4: renamed from C?; footprint (none) -> Capacitors_THT:CP_Radial_D8.0mm_P2.50mm
- D1: renamed from D4; footprint (none) -> Diodes_THT:Diode_DO-35_SOD27_Horizontal_RM10
- D2: renamed from D1; footprint (none) -> Diodes_THT:Diode_DO-35_SOD27_Horizontal_RM10
- D3: renamed from D5; footprint (none) -> Diodes_THT:Diode_DO-35_SOD27_Horizontal_RM10
- D4: renamed from D2; footprint (none) -> Diodes_THT:Diode_DO-35_SOD27_Horizontal_RM10
- D5: renamed from D6; footprint (none) -> Diodes_THT:Diode_DO-35_SOD27_Horizontal_RM10
- D6: renamed from D3; footprint (none) -> Diodes_THT:Diode_DO-35_SOD27_Horizontal_RM10
- F1, F2, F3: footprint (none) -> FSFootprints:SMD Fuse
- J1: renamed from J?; footprint (none) -> Connectors_Molex:Molex_NanoFit_2x04x2.50mm_Straight
- J2: renamed from J8; footprint (none) -> Connectors_Molex:Molex_NanoFit_2x04x2.50mm_Straight
- J3, J5: renamed from J?; footprint (none) -> Connectors_Molex:Molex_NanoFit_1x04x2.50mm_Straight
- J4: renamed from J9; footprint (none) -> Connectors_Molex:Molex_NanoFit_2x03x2.50mm_Straight
- J6: renamed from J10; footprint (none) -> Connectors_Molex:Molex_MiniFit-JR-5556-02B_2x01x4.20mm_Straight
- J7: renamed from J11; footprint (none) -> Connectors_Molex:Molex_NanoFit_1x02x2.50mm_Straight
- J8: renamed from J?; footprint (none) -> Connectors_Molex:Molex_NanoFit_1x03x2.50mm_Straight
- J9: renamed from J?; footprint (none) -> Connectors_Molex:Molex_NanoFit_1x02x2.50mm_Straight
- R1, R4, R8: renamed from R?; footprint (none) -> Resistors_THT:R_Axial_DIN0411_L9.9mm_D3.6mm_P12.70mm_Horizontal
- R10: renamed from R5; footprint (none) -> Resistors_THT:R_Axial_DIN0411_L9.9mm_D3.6mm_P12.70mm_Horizontal
- R11: renamed from R8; footprint (none) -> Resistors_THT:R_Axial_DIN0411_L9.9mm_D3.6mm_P12.70mm_Horizontal
- R12: renamed from R1; footprint (none) -> Resistors_THT:R_Axial_DIN0411_L9.9mm_D3.6mm_P12.70mm_Horizontal
- R13: renamed from R2; footprint (none) -> Resistors_THT:R_Axial_DIN0411_L9.9mm_D3.6mm_P12.70mm_Horizontal
- R2: renamed from R3; footprint (none) -> Resistors_THT:R_Axial_DIN0411_L9.9mm_D3.6mm_P12.70mm_Horizontal
- R3: renamed from R6; footprint (none) -> Resistors_THT:R_Axial_DIN0411_L9.9mm_D3.6mm_P12.70mm_Horizontal
- R5: renamed from R4; footprint (none) -> Resistors_THT:R_Axial_DIN0411_L9.9mm_D3.6mm_P12.70mm_Horizontal
- R6: renamed from R7; footprint (none) -> Resistors_THT:R_Axial_DIN0411_L9.9mm_D3.6mm_P12.70mm_Horizontal
- R7: renamed from R9; footprint (none) -> Resistors_THT:R_Axial_DIN0411_L9.9mm_D3.6mm_P12.70mm_Horizontal
- R9: renamed from R10; footprint (none) -> Resistors_THT:R_Axial_DIN0411_L9.9mm_D3.6mm_P12.70mm_Horizontal
- U1: renamed from U6; footprint TO-220 -> Power_Integrations:TO-220
- U3: renamed from U?; footprint (none) -> Housings_DIP:DIP-16_W7.62mm
- U4, U5: footprint (none) -> FSFootprints:DK1A1B-12V

Commit message: Revise Accumulator HV and LV, route Dash Switchbox, begin PE HV
Parts:
- D1, D2, D3, D4, D5, D6: footprint Diodes_THT:Diode_DO-35_SOD27_Horizontal_RM10 -> Diodes_THT:D_DO-35_SOD27_P12.70mm_Horizontal
- J6: footprint Connectors_Molex:Molex_MiniFit-JR-5556-02B_2x01x4.20mm_Straight -> Connectors_Molex:Molex_MiniFit-JR-5556-02A_2x01x4.20mm_Straight
- R12, R13: value 20R -> 1K; footprint Resistors_THT:R_Axial_DIN0411_L9.9mm_D3.6mm_P12.70mm_Horizontal -> TO_SOT_Packages_THT:TO-247-2_Horizontal
- U1: footprint Power_Integrations:TO-220 -> TO_SOT_Packages_THT:TO-220-3_Horizontal
Changed lines of the file:
@@
 P 5600 5200
 F 0 "R12" V 5680 5200 50  0000 C CNN
-F 1 "20R" V 5600 5200 50  0000 C CNN
-F 2 "Resistors_THT:R_Axial_DIN0411_L9.9mm_D3.6mm_P12.70mm_Horizontal" V 5530 5200 50  0001 C CNN
+F 1 "1K" V 5600 5200 50  0000 C CNN
+F 2 "TO_SOT_Packages_THT:TO-247-2_Horizontal" V 5530 5200 50  0001 C CNN
 F 3 "" H 5600 5200 50  0000 C CNN
 	1    5600 5200
@@
 P 5600 6500
 F 0 "R13" V 5680 6500 50  0000 C CNN
-F 1 "20R" V 5600 6500 50  0000 C CNN
-F 2 "Resistors_THT:R_Axial_DIN0411_L9.9mm_D3.6mm_P12.70mm_Horizontal" V 5530 6500 50  0001 C CNN
+F 1 "1K" V 5600 6500 50  0000 C CNN
+F 2 "TO_SOT_Packages_THT:TO-247-2_Horizontal" V 5530 6500 50  0001 C CNN
 F 3 "" H 5600 6500 50  0000 C CNN
 	1    5600 6500
@@
 F 0 "J6" H 10700 3150 50  0000 C CNN
 F 1 "HV Cable" V 10800 3000 50  0000 C CNN
-F 2 "Connectors_Molex:Molex_MiniFit-JR-5556-02B_2x01x4.20mm_Straight" H 10700 3000 50  0001 C CNN
+F 2 "Connectors_Molex:Molex_MiniFit-JR-5556-02A_2x01x4.20mm_Straight" H 10700 3000 50  0001 C CNN
 F 3 "" H 10700 3000 50  0000 C CNN
 	1    10700 3000
@@
 F 0 "U1" H 7950 1400 50  0000 C CNN
 F 1 "L78S05CV-DG" H 8150 1400 50  0000 L CNN
-F 2 "Power_Integrations:TO-220" H 8150 850 50  0001 C CIN
+F 2 "TO_SOT_Packages_THT:TO-220-3_Horizontal" H 8150 850 50  0001 C CIN
 F 3 "" H 8150 1200 50  0000 C CNN
 	1    8150 1200
@@
 F 0 "D1" H 6350 2200 50  0000 C CNN
 F 1 "48V Zener" H 6350 2000 50  0000 C CNN
-F 2 "Diodes_THT:Diode_DO-35_SOD27_Horizontal_RM10" H 6350 2100 50  0001 C CNN
+F 2 "Diodes_THT:D_DO-35_SOD27_P12.70mm_Horizontal" H 6350 2100 50  0001 C CNN
 F 3 "" H 6350 2100 50  0000 C CNN
 	1    6350 2100
@@
 F 0 "D2" H 6200 2550 50  0000 C CNN
 F 1 "12V Zener" H 6200 2350 50  0000 C CNN
-F 2 "Diodes_THT:Diode_DO-35_SOD27_Horizontal_RM10" H 6200 2450 50  0001 C CNN
+F 2 "Diodes_THT:D_DO-35_SOD27_P12.70mm_Horizontal" H 6200 2450 50  0001 C CNN
 F 3 "" H 6200 2450 50  0000 C CNN
 	1    6200 2450
@@
 F 0 "D3" H 6350 3050 50  0000 C CNN
 F 1 "48V Zener" H 6350 2850 50  0000 C CNN
-F 2 "Diodes_THT:Diode_DO-35_SOD27_Horizontal_RM10" H 6350 2950 50  0001 C CNN
+F 2 "Diodes_THT:D_DO-35_SOD27_P12.70mm_Horizontal" H 6350 2950 50  0001 C CNN
 F 3 "" H 6350 2950 50  0000 C CNN
 	1    6350 2950
@@
 F 0 "D4" H 6200 3400 50  0000 C CNN
 F 1 "12V Zener" H 6200 3200 50  0000 C CNN
-F 2 "Diodes_THT:Diode_DO-35_SOD27_Horizontal_RM10" H 6200 3300 50  0001 C CNN
+F 2 "Diodes_THT:D_DO-35_SOD27_P12.70mm_Horizontal" H 6200 3300 50  0001 C CNN
 F 3 "" H 6200 3300 50  0000 C CNN
 	1    6200 3300
@@
 F 0 "D5" H 6350 3900 50  0000 C CNN
 F 1 "48V Zener" H 6350 3700 50  0000 C CNN
-F 2 "Diodes_THT:Diode_DO-35_SOD27_Horizontal_RM10" H 6350 3800 50  0001 C CNN
+F 2 "Diodes_THT:D_DO-35_SOD27_P12.70mm_Horizontal" H 6350 3800 50  0001 C CNN
 F 3 "" H 6350 3800 50  0000 C CNN
 	1    6350 3800
@@
 F 0 "D6" H 6200 4250 50  0000 C CNN
 F 1 "12V Zener" H 6200 4050 50  0000 C CNN
-F 2 "Diodes_THT:Diode_DO-35_SOD27_Horizontal_RM10" H 6200 4150 50  0001 C CNN
+F 2 "Diodes_THT:D_DO-35_SOD27_P12.70mm_Horizontal" H 6200 4150 50  0001 C CNN
 F 3 "" H 6200 4150 50  0000 C CNN
 	1    6200 4150

Commit message: Progress on PE HV PCB layout
Parts:
- added R1: 120, Resistors_THT:R_Axial_DIN0411_L9.9mm_D3.6mm_P12.70mm_Horizontal, symbol R
- J5: footprint Connectors_Molex:Molex_NanoFit_1x04x2.50mm_Straight -> FSFootprints:DT13-4P
- R13: renamed from R12; footprint TO_SOT_Packages_THT:TO-247-2_Horizontal -> TO_SOT_Packages_THT:TO-220-2_Horizontal
- R14: renamed from R13; footprint TO_SOT_Packages_THT:TO-247-2_Horizontal -> TO_SOT_Packages_THT:TO-220-2_Horizontal
- U1: footprint TO_SOT_Packages_THT:TO-220-3_Horizontal -> FSFootprints:TO-220-3_Horizontal_HeatSunk
- renumbered R9 to R10, R10 to R11, R11 to R12, R1 to R2, R2 to R3, R3 to R4, R4 to R5, R5 to R6, R6 to R7, R7 to R8, R8 to R9
Connections:
- wire segments 23 -> 25
Changed lines of the file:
@@
 CAN_H_BOARD
 $Comp
-L R R12
+L R R13
 U 1 1 588D76FB
-P 5600 5200
-F 0 "R12" V 5680 5200 50  0000 C CNN
-F 1 "1K" V 5600 5200 50  0000 C CNN
-F 2 "TO_SOT_Packages_THT:TO-247-2_Horizontal" V 5530 5200 50  0001 C CNN
-F 3 "" H 5600 5200 50  0000 C CNN
-	1    5600 5200
-	0    1    1    0
-$EndComp
-$Comp
-L R R13
+P 5600 6200
+F 0 "R13" V 5680 6200 50  0000 C CNN
+F 1 "1K" V 5600 6200 50  0000 C CNN
+F 2 "TO_SOT_Packages_THT:TO-220-2_Horizontal" V 5530 6200 50  0001 C CNN
+F 3 "" H 5600 6200 50  0000 C CNN
+	1    5600 6200
+	0    1    1    0
+$EndComp
+$Comp
+L R R14
 U 1 1 588D7799
-P 5600 6500
-F 0 "R13" V 5680 6500 50  0000 C CNN
-F 1 "1K" V 5600 6500 50  0000 C CNN
-F 2 "TO_SOT_Packages_THT:TO-247-2_Horizontal" V 5530 6500 50  0001 C CNN
-F 3 "" H 5600 6500 50  0000 C CNN
-	1    5600 6500
-	0    1    1    0
-$EndComp
-Text Label 5750 5200 0    60   ~ 0
+P 5600 7500
+F 0 "R14" V 5680 7500 50  0000 C CNN
+F 1 "1K" V 5600 7500 50  0000 C CNN
+F 2 "TO_SOT_Packages_THT:TO-220-2_Horizontal" V 5530 7500 50  0001 C CNN
+F 3 "" H 5600 7500 50  0000 C CNN
+	1    5600 7500
+	0    1    1    0
+$EndComp
+Text Label 5450 5500 0    60   ~ 0
 TS+_SWITCHED_L
-Text Label 5750 6500 0    60   ~ 0
+Text Label 5450 6800 0    60   ~ 0
 TS+_SWITCHED_R
-Text Label 5450 6100 3    60   ~ 0
-TS-
-Text Label 5450 7400 3    60   ~ 0
+Text Label 5750 6200 0    60   ~ 0
+TS-
+Text Label 5750 7500 0    60   ~ 0
 TS-
 Text Notes 8550 900  2    60   ~ 0
@@
 $EndComp
 $Comp
-L R R7
+L R R8
 U 1 1 58916788
 P 10350 3550
-F 0 "R7" V 10430 3550 50  0000 C CNN
+F 0 "R8" V 10430 3550 50  0000 C CNN
 F 1 "5kR" V 10350 3550 50  0000 C CNN
 F 2 "Resistors_THT:R_Axial_DIN0411_L9.9mm_D3.6mm_P12.70mm_Horizontal" V 10280 3550 50  0001 C CNN
@@
 $EndComp
 $Comp
-L R R9
+L R R10
 U 1 1 58916808
 P 10500 3800
-F 0 "R9" V 10580 3800 50  0000 C CNN
+F 0 "R10" V 10580 3800 50  0000 C CNN
 F 1 "5kR" V 10500 3800 50  0000 C CNN
 F 2 "Resistors_THT:R_Axial_DIN0411_L9.9mm_D3.6mm_P12.70mm_Horizontal" V 10430 3800 50  0001 C CNN
@@
 F 0 "U1" H 7950 1400 50  0000 C CNN
 F 1 "L78S05CV-DG" H 8150 1400 50  0000 L CNN
-F 2 "TO_SOT_Packages_THT:TO-220-3_Horizontal" H 8150 850 50  0001 C CIN
+F 2 "FSFootprints:TO-220-3_Horizontal_HeatSunk" H 8150 850 50  0001 C CIN
 F 3 "" H 8150 1200 50  0000 C CNN
 	1    8150 1200
@@
 $EndComp
 $Comp
-L R R2
+L R R3
 U 1 1 58C4AF19
 P 5700 2350
-F 0 "R2" V 5780 2350 50  0000 C CNN
+F 0 "R3" V 5780 2350 50  0000 C CNN
 F 1 "1.2kR" V 5700 2350 50  0000 C CNN
 F 2 "Resistors_THT:R_Axial_DIN0411_L9.9mm_D3.6mm_P12.70mm_Horizontal" V 5630 2350 50  0001 C CNN
@@
 Wire Notes Line
 	5250 500  5250 7750
-Wire Wire Line
-	5450 6800 5450 6500
-Wire Wire Line
-	5450 5500 5450 5200
 Wire Wire Line
 	6200 2300 5850 2300
@@
 $EndComp
 $Comp
-L R R5
+L R R6
 U 1 1 58C4B7BC
 P 5700 3200
-F 0 "R5" V 5780 3200 50  0000 C CNN
+F 0 "R6" V 5780 3200 50  0000 C CNN
 F 1 "1.2kR" V 5700 3200 50  0000 C CNN
 F 2 "Resistors_THT:R_Axial_DIN0411_L9.9mm_D3.6mm_P12.70mm_Horizontal" V 5630 3200 50  0001 C CNN
@@
 $EndComp
 $Comp
-L R R10
+L R R11
 U 1 1 58C4BA41
 P 5700 4050
-F 0 "R10" V 5780 4050 50  0000 C CNN
+F 0 "R11" V 5780 4050 50  0000 C CNN
 F 1 "1.2kR" V 5700 4050 50  0000 C CNN
 F 2 "Resistors_THT:R_Axial_DIN0411_L9.9mm_D3.6mm_P12.70mm_Horizontal" V 5630 4050 50  0001 C CNN
@@
 $EndComp
 $Comp
-L R R3
+L R R4
 U 1 1 58C4C8E9
 P 6350 2600
-F 0 "R3" V 6430 2600 50  0000 C CNN
+F 0 "R4" V 6430 2600 50  0000 C CNN
 F 1 "3kR" V 6350 2600 50  0000 C CNN
 F 2 "Resistors_THT:R_Axial_DIN0411_L9.9mm_D3.6mm_P12.70mm_Horizontal" V 6280 2600 50  0001 C CNN
@@
 $EndComp
 $Comp
-L R R6
+L R R7
 U 1 1 58C4CA42
 P 6350 3450
-F 0 "R6" V 6430 3450 50  0000 C CNN
+F 0 "R7" V 6430 3450 50  0000 C CNN
 F 1 "3kR" V 6350 3450 50  0000 C CNN
 F 2 "Resistors_THT:R_Axial_DIN0411_L9.9mm_D3.6mm_P12.70mm_Horizontal" V 6280 3450 50  0001 C CNN
@@
 $EndComp
 $Comp
-L R R11
+L R R12
 U 1 1 58C4CBDA
 P 6350 4300
-F 0 "R11" V 6430 4300 50  0000 C CNN
+F 0 "R12" V 6430 4300 50  0000 C CNN
 F 1 "3kR" V 6350 4300 50  0000 C CNN
 F 2 "Resistors_THT:R_Axial_DIN0411_L9.9mm_D3.6mm_P12.70mm_Horizontal" V 6280 4300 50  0001 C CNN
@@
 Needs (Small) Heat Sink!
 $Comp
-L R R8
+L R R9
 U 1 1 59B378CF
 P 6650 3800
-F 0 "R8" V 6730 3800 50  0000 C CNN
+F 0 "R9" V 6730 3800 50  0000 C CNN
 F 1 "R" V 6650 3800 50  0000 C CNN
 F 2 "Resistors_THT:R_Axial_DIN0411_L9.9mm_D3.6mm_P12.70mm_Horizontal" V 6580 3800 50  0001 C CNN
@@
 $EndComp
 $Comp
-L R R4
+L R R5
 U 1 1 59B3797A
 P 6650 2950
-F 0 "R4" V 6730 2950 50  0000 C CNN
+F 0 "R5" V 6730 2950 50  0000 C CNN
 F 1 "R" V 6650 2950 50  0000 C CNN
 F 2 "Resistors_THT:R_Axial_DIN0411_L9.9mm_D3.6mm_P12.70mm_Horizontal" V 6580 2950 50  0001 C CNN
@@
 $EndComp
 $Comp
-L R R1
+L R R2
 U 1 1 59B37B6E
 P 6650 2100
-F 0 "R1" V 6730 2100 50  0000 C CNN
+F 0 "R2" V 6730 2100 50  0000 C CNN
 F 1 "R" V 6650 2100 50  0000 C CNN
 F 2 "Resistors_THT:R_Axial_DIN0411_L9.9mm_D3.6mm_P12.70mm_Horizontal" V 6580 2100 50  0001 C CNN
@@
 F 0 "J5" H 800 3100 50  0000 C CNN
 F 1 "E-Meter External" V 900 2900 50  0000 C CNN
-F 2 "Connectors_Molex:Molex_NanoFit_1x04x2.50mm_Straight" H 800 2900 50  0001 C CNN
+F 2 "FSFootprints:DT13-4P" H 800 2900 50  0001 C CNN
 F 3 "" H 800 2900 50  0001 C CNN
 	1    800  2900
@@
 Wire Wire Line
 	10500 5300 10500 5400
+Wire Wire Line
+	5450 6200 5450 6100
+Wire Wire Line
+	5450 7400 5450 7500
+$Comp
+L R R1
+U 1 1 5A837AFE
+P 5850 1450
+F 0 "R1" V 5930 1450 50  0000 C CNN
+F 1 "120" V 5850 1450 50  0000 C CNN
+F 2 "Resistors_THT:R_Axial_DIN0411_L9.9mm_D3.6mm_P12.70mm_Horizontal" V 5780 1450 50  0001 C CNN
+F 3 "" H 5850 1450 50  0001 C CNN
+	1    5850 1450
+	1    0    0    -1
+$EndComp
+Wire Wire Line
+	5850 1300 5850 1250
+Wire Wire Line
+	5850 1600 5850 1650
 $EndSCHEMATC

Commit message: Layout and route PE HV board
Parts:
- added C1: CP, Capacitors_THT:CP_Radial_D8.0mm_P2.50mm, symbol CP
- J6: footprint Connectors_Molex:Molex_MiniFit-JR-5556-02A_2x01x4.20mm_Straight -> Connectors_Molex:Molex_NanoFit_1x02x2.50mm_Straight
- J7: footprint Connectors_Molex:Molex_NanoFit_1x02x2.50mm_Straight -> FSFootprints:DT15-2P
- R13, R14: footprint TO_SOT_Packages_THT:TO-220-2_Horizontal -> TO_SOT_Packages_THT:TO-220-2_Vertical
- renumbered C1 to C2, C2 to C3, C3 to C4, C4 to C5
Connections:
- net labels removed: 3.3V_LV
Changed lines of the file:
@@
 CAN_TX
 Text Label 5150 950  1    60   ~ 0
-3.3V_LV
+3.3V_GLV
 Text Label 5350 950  1    60   ~ 0
 5V_TS
@@
 F 0 "R13" V 5680 6200 50  0000 C CNN
 F 1 "1K" V 5600 6200 50  0000 C CNN
-F 2 "TO_SOT_Packages_THT:TO-220-2_Horizontal" V 5530 6200 50  0001 C CNN
+F 2 "TO_SOT_Packages_THT:TO-220-2_Vertical" V 5530 6200 50  0001 C CNN
 F 3 "" H 5600 6200 50  0000 C CNN
 	1    5600 6200
@@
 F 0 "R14" V 5680 7500 50  0000 C CNN
 F 1 "1K" V 5600 7500 50  0000 C CNN
-F 2 "TO_SOT_Packages_THT:TO-220-2_Horizontal" V 5530 7500 50  0001 C CNN
+F 2 "TO_SOT_Packages_THT:TO-220-2_Vertical" V 5530 7500 50  0001 C CNN
 F 3 "" H 5600 7500 50  0000 C CNN
 	1    5600 7500
@@
 F 0 "J6" H 10700 3150 50  0000 C CNN
 F 1 "HV Cable" V 10800 3000 50  0000 C CNN
-F 2 "Connectors_Molex:Molex_MiniFit-JR-5556-02A_2x01x4.20mm_Straight" H 10700 3000 50  0001 C CNN
+F 2 "Connectors_Molex:Molex_NanoFit_1x02x2.50mm_Straight" H 10700 3000 50  0001 C CNN
 F 3 "" H 10700 3000 50  0000 C CNN
 	1    10700 3000
@@
 F 0 "J7" H 10700 3700 50  0000 C CNN
 F 1 "TSMPs" V 10800 3550 50  0000 C CNN
-F 2 "Connectors_Molex:Molex_NanoFit_1x02x2.50mm_Straight" H 10700 3550 50  0001 C CNN
+F 2 "FSFootprints:DT15-2P" H 10700 3550 50  0001 C CNN
 F 3 "" H 10700 3550 50  0000 C CNN
 	1    10700 3550
@@
 EM_SIG-
 $Comp
-L CP C3
+L CP C4
 U 1 1 59B3ABDF
 P 7750 1300
-F 0 "C3" H 7775 1400 50  0000 L CNN
+F 0 "C4" H 7775 1400 50  0000 L CNN
 F 1 "CP" H 7775 1200 50  0000 L CNN
 F 2 "Capacitors_THT:CP_Radial_D8.0mm_P2.50mm" H 7788 1150 50  0001 C CNN
@@
 $EndComp
 $Comp
-L CP C4
+L CP C5
 U 1 1 59B3AC80
 P 8550 1300
-F 0 "C4" H 8575 1400 50  0000 L CNN
+F 0 "C5" H 8575 1400 50  0000 L CNN
 F 1 "CP" H 8575 1200 50  0000 L CNN
 F 2 "Capacitors_THT:CP_Radial_D8.0mm_P2.50mm" H 8588 1150 50  0001 C CNN
@@
 3.3V_GLV
 $Comp
-L C C1
+L C C2
 U 1 1 5A3F30B7
 P 2450 1000
-F 0 "C1" H 2475 1100 50  0000 L CNN
+F 0 "C2" H 2475 1100 50  0000 L CNN
 F 1 "C" H 2475 900 50  0000 L CNN
 F 2 "Capacitors_THT:CP_Radial_D8.0mm_P2.50mm" H 2488 850 50  0001 C CNN
@@
 $EndComp
 $Comp
-L C C2
+L C C3
 U 1 1 5A3F31B6
 P 2950 1000
-F 0 "C2" H 2975 1100 50  0000 L CNN
+F 0 "C3" H 2975 1100 50  0000 L CNN
 F 1 "C" H 2975 900 50  0000 L CNN
 F 2 "Capacitors_THT:CP_Radial_D8.0mm_P2.50mm" H 2988 850 50  0001 C CNN
@@
 Wire Wire Line
 	5850 1600 5850 1650
+$Comp
+L CP C1
+U 1 1 5A84D24A
+P 5500 950
+F 0 "C1" H 5525 1050 50  0000 L CNN
+F 1 "CP" H 5525 850 50  0000 L CNN
+F 2 "Capacitors_THT:CP_Radial_D8.0mm_P2.50mm" H 5538 800 50  0001 C CNN
+F 3 "" H 5500 950 50  0001 C CNN
+	1    5500 950
+	0    -1   -1   0
+$EndComp
+Text Label 5650 950  0    60   ~ 0
+TS-
 $EndSCHEMATC

Commit message: Tweak PE HV board
Parts:
- added H1, H2: MtngHole, Mounting_Holes:MountingHole_4.5mm, symbol Conn_01x01
- C1, C2, C3, C4, C5: footprint Capacitors_THT:CP_Radial_D8.0mm_P2.50mm -> Capacitors_THT:CP_Radial_D5.0mm_P2.50mm
- J3: footprint Connectors_Molex:Molex_NanoFit_1x04x2.50mm_Straight -> Connectors_Molex:Molex_NanoFit_2x02x2.50mm_Straight
Changed lines of the file:
@@
 LIBS:contrib
 LIBS:valves
-LIBS:PEBoardHV-cache
 EELAYER 25 0
 EELAYER END
@@
 F 0 "J3" H 800 2250 50  0000 C CNN
 F 1 "E-Meter Internal" V 900 2050 50  0000 C CNN
-F 2 "Connectors_Molex:Molex_NanoFit_1x04x2.50mm_Straight" H 800 2050 50  0001 C CNN
+F 2 "Connectors_Molex:Molex_NanoFit_2x02x2.50mm_Straight" H 800 2050 50  0001 C CNN
 F 3 "" H 800 2050 50  0001 C CNN
 	1    800  2050
@@
 F 0 "C4" H 7775 1400 50  0000 L CNN
 F 1 "CP" H 7775 1200 50  0000 L CNN
-F 2 "Capacitors_THT:CP_Radial_D8.0mm_P2.50mm" H 7788 1150 50  0001 C CNN
+F 2 "Capacitors_THT:CP_Radial_D5.0mm_P2.50mm" H 7788 1150 50  0001 C CNN
 F 3 "" H 7750 1300 50  0001 C CNN
 	1    7750 1300
@@
 F 0 "C5" H 8575 1400 50  0000 L CNN
 F 1 "CP" H 8575 1200 50  0000 L CNN
-F 2 "Capacitors_THT:CP_Radial_D8.0mm_P2.50mm" H 8588 1150 50  0001 C CNN
+F 2 "Capacitors_THT:CP_Radial_D5.0mm_P2.50mm" H 8588 1150 50  0001 C CNN
 F 3 "" H 8550 1300 50  0001 C CNN
 	1    8550 1300
@@
 F 0 "C2" H 2475 1100 50  0000 L CNN
 F 1 "C" H 2475 900 50  0000 L CNN
-F 2 "Capacitors_THT:CP_Radial_D8.0mm_P2.50mm" H 2488 850 50  0001 C CNN
+F 2 "Capacitors_THT:CP_Radial_D5.0mm_P2.50mm" H 2488 850 50  0001 C CNN
 F 3 "" H 2450 1000 50  0001 C CNN
 	1    2450 1000
@@
 F 0 "C3" H 2975 1100 50  0000 L CNN
 F 1 "C" H 2975 900 50  0000 L CNN
-F 2 "Capacitors_THT:CP_Radial_D8.0mm_P2.50mm" H 2988 850 50  0001 C CNN
+F 2 "Capacitors_THT:CP_Radial_D5.0mm_P2.50mm" H 2988 850 50  0001 C CNN
 F 3 "" H 2950 1000 50  0001 C CNN
 	1    2950 1000
@@
 F 0 "C1" H 5525 1050 50  0000 L CNN
 F 1 "CP" H 5525 850 50  0000 L CNN
-F 2 "Capacitors_THT:CP_Radial_D8.0mm_P2.50mm" H 5538 800 50  0001 C CNN
+F 2 "Capacitors_THT:CP_Radial_D5.0mm_P2.50mm" H 5538 800 50  0001 C CNN
 F 3 "" H 5500 950 50  0001 C CNN
 	1    5500 950
@@
 Text Label 5650 950  0    60   ~ 0
 TS-
+$Comp
+L Conn_01x01 H1
+U 1 1 5A94B007
+P 10950 6050
+F 0 "H1" H 10950 6150 50  0000 C CNN
+F 1 "MtngHole" H 10950 5950 50  0000 C CNN
+F 2 "Mounting_Holes:MountingHole_4.5mm" H 10950 6050 50  0001 C CNN
+F 3 "" H 10950 6050 50  0001 C CNN
+	1    10950 6050
+	1    0    0    -1
+$EndComp
+$Comp
+L Conn_01x01 H2
+U 1 1 5A94B644
+P 10950 6350
+F 0 "H2" H 10950 6450 50  0000 C CNN
+F 1 "MtngHole" H 10950 6250 50  0000 C CNN
+F 2 "Mounting_Holes:MountingHole_4.5mm" H 10950 6350 50  0001 C CNN
+F 3 "" H 10950 6350 50  0001 C CNN
+	1    10950 6350
+	1    0    0    -1
+$EndComp
 $EndSCHEMATC
