File: PEBoardHV/PEBoardHV.sch (KiCad schematic (older format))
At the start: 44 parts, among them J1 To PE LV, J2 Left Connector (Master), J3 E-Meter Internal, J4 Right Connector (Slave), J5 E-Meter External, J6 HV Cable, J7 TSMPs, J8 HV CAN Debug, J9 EMeter HV, U1 L78S05CV-DG, U2 ISO1050, U3 PS2501-4, U4 DK1A1B-12V, U5 DK1A1B-12V

Commit message: Add ground planes to PE HV PCB and add an additional mounting hole
Parts:
- added H3: MtngHole, Mounting_Holes:MountingHole_4.5mm, symbol Conn_01x01
- D1, D2, D3, D4, D5, D6: footprint Diodes_THT:D_DO-35_SOD27_P12.70mm_Horizontal -> Diodes_THT:D_A-405_P10.16mm_Horizontal
- R1, R10, R11, R12, R2, R3, R4, R5, R6, R7, R8, R9: footprint Resistors_THT:R_Axial_DIN0411_L9.9mm_D3.6mm_P12.70mm_Horizontal -> Resistors_THT:R_Axial_DIN0207_L6.3mm_D2.5mm_P10.16mm_Horizontal
Changed lines of the file:
@@
 LIBS:contrib
 LIBS:valves
+LIBS:PEBoardHV-cache
 EELAYER 25 0
 EELAYER END
@@
 F 0 "R8" V 10430 3550 50  0000 C CNN
 F 1 "5kR" V 10350 3550 50  0000 C CNN
-F 2 "Resistors_THT:R_Axial_DIN0411_L9.9mm_D3.6mm_P12.70mm_Horizontal" V 10280 3550 50  0001 C CNN
+F 2 "Resistors_THT:R_Axial_DIN0207_L6.3mm_D2.5mm_P10.16mm_Horizontal" V 10280 3550 50  0001 C CNN
 F 3 "" H 10350 3550 50  0000 C CNN
 	1    10350 3550
@@
 F 0 "R10" V 10580 3800 50  0000 C CNN
 F 1 "5kR" V 10500 3800 50  0000 C CNN
-F 2 "Resistors_THT:R_Axial_DIN0411_L9.9mm_D3.6mm_P12.70mm_Horizontal" V 10430 3800 50  0001 C CNN
+F 2 "Resistors_THT:R_Axial_DIN0207_L6.3mm_D2.5mm_P10.16mm_Horizontal" V 10430 3800 50  0001 C CNN
 F 3 "" H 10500 3800 50  0000 C CNN
 	1    10500 3800
@@
 F 0 "D1" H 6350 2200 50  0000 C CNN
 F 1 "48V Zener" H 6350 2000 50  0000 C CNN
-F 2 "Diodes_THT:D_DO-35_SOD27_P12.70mm_Horizontal" H 6350 2100 50  0001 C CNN
+F 2 "Diodes_THT:D_A-405_P10.16mm_Horizontal" H 6350 2100 50  0001 C CNN
 F 3 "" H 6350 2100 50  0000 C CNN
 	1    6350 2100
@@
 F 0 "D2" H 6200 2550 50  0000 C CNN
 F 1 "12V Zener" H 6200 2350 50  0000 C CNN
-F 2 "Diodes_THT:D_DO-35_SOD27_P12.70mm_Horizontal" H 6200 2450 50  0001 C CNN
+F 2 "Diodes_THT:D_A-405_P10.16mm_Horizontal" H 6200 2450 50  0001 C CNN
 F 3 "" H 6200 2450 50  0000 C CNN
 	1    6200 2450
@@
 F 0 "R3" V 5780 2350 50  0000 C CNN
 F 1 "1.2kR" V 5700 2350 50  0000 C CNN
-F 2 "Resistors_THT:R_Axial_DIN0411_L9.9mm_D3.6mm_P12.70mm_Horizontal" V 5630 2350 50  0001 C CNN
+F 2 "Resistors_THT:R_Axial_DIN0207_L6.3mm_D2.5mm_P10.16mm_Horizontal" V 5630 2350 50  0001 C CNN
 F 3 "" H 5700 2350 50  0000 C CNN
 	1    5700 2350
@@
 F 0 "D3" H 6350 3050 50  0000 C CNN
 F 1 "48V Zener" H 6350 2850 50  0000 C CNN
-F 2 "Diodes_THT:D_DO-35_SOD27_P12.70mm_Horizontal" H 6350 2950 50  0001 C CNN
+F 2 "Diodes_THT:D_A-405_P10.16mm_Horizontal" H 6350 2950 50  0001 C CNN
 F 3 "" H 6350 2950 50  0000 C CNN
 	1    6350 2950
@@
 F 0 "D4" H 6200 3400 50  0000 C CNN
 F 1 "12V Zener" H 6200 3200 50  0000 C CNN
-F 2 "Diodes_THT:D_DO-35_SOD27_P12.70mm_Horizontal" H 6200 3300 50  0001 C CNN
+F 2 "Diodes_THT:D_A-405_P10.16mm_Horizontal" H 6200 3300 50  0001 C CNN
 F 3 "" H 6200 3300 50  0000 C CNN
 	1    6200 3300
@@
 F 0 "R6" V 5780 3200 50  0000 C CNN
 F 1 "1.2kR" V 5700 3200 50  0000 C CNN
-F 2 "Resistors_THT:R_Axial_DIN0411_L9.9mm_D3.6mm_P12.70mm_Horizontal" V 5630 3200 50  0001 C CNN
+F 2 "Resistors_THT:R_Axial_DIN0207_L6.3mm_D2.5mm_P10.16mm_Horizontal" V 5630 3200 50  0001 C CNN
 F 3 "" H 5700 3200 50  0000 C CNN
 	1    5700 3200
@@
 F 0 "D5" H 6350 3900 50  0000 C CNN
 F 1 "48V Zener" H 6350 3700 50  0000 C CNN
-F 2 "Diodes_THT:D_DO-35_SOD27_P12.70mm_Horizontal" H 6350 3800 50  0001 C CNN
+F 2 "Diodes_THT:D_A-405_P10.16mm_Horizontal" H 6350 3800 50  0001 C CNN
 F 3 "" H 6350 3800 50  0000 C CNN
 	1    6350 3800
@@
 F 0 "D6" H 6200 4250 50  0000 C CNN
 F 1 "12V Zener" H 6200 4050 50  0000 C CNN
-F 2 "Diodes_THT:D_DO-35_SOD27_P12.70mm_Horizontal" H 6200 4150 50  0001 C CNN
+F 2 "Diodes_THT:D_A-405_P10.16mm_Horizontal" H 6200 4150 50  0001 C CNN
 F 3 "" H 6200 4150 50  0000 C CNN
 	1    6200 4150
@@
 F 0 "R11" V 5780 4050 50  0000 C CNN
 F 1 "1.2kR" V 5700 4050 50  0000 C CNN
-F 2 "Resistors_THT:R_Axial_DIN0411_L9.9mm_D3.6mm_P12.70mm_Horizontal" V 5630 4050 50  0001 C CNN
+F 2 "Resistors_THT:R_Axial_DIN0207_L6.3mm_D2.5mm_P10.16mm_Horizontal" V 5630 4050 50  0001 C CNN
 F 3 "" H 5700 4050 50  0000 C CNN
 	1    5700 4050
@@
 F 0 "R4" V 6430 2600 50  0000 C CNN
 F 1 "3kR" V 6350 2600 50  0000 C CNN
-F 2 "Resistors_THT:R_Axial_DIN0411_L9.9mm_D3.6mm_P12.70mm_Horizontal" V 6280 2600 50  0001 C CNN
+F 2 "Resistors_THT:R_Axial_DIN0207_L6.3mm_D2.5mm_P10.16mm_Horizontal" V 6280 2600 50  0001 C CNN
 F 3 "" H 6350 2600 50  0000 C CNN
 	1    6350 2600
@@
 F 0 "R7" V 6430 3450 50  0000 C CNN
 F 1 "3kR" V 6350 3450 50  0000 C CNN
-F 2 "Resistors_THT:R_Axial_DIN0411_L9.9mm_D3.6mm_P12.70mm_Horizontal" V 6280 3450 50  0001 C CNN
+F 2 "Resistors_THT:R_Axial_DIN0207_L6.3mm_D2.5mm_P10.16mm_Horizontal" V 6280 3450 50  0001 C CNN
 F 3 "" H 6350 3450 50  0000 C CNN
 	1    6350 3450
@@
 F 0 "R12" V 6430 4300 50  0000 C CNN
 F 1 "3kR" V 6350 4300 50  0000 C CNN
-F 2 "Resistors_THT:R_Axial_DIN0411_L9.9mm_D3.6mm_P12.70mm_Horizontal" V 6280 4300 50  0001 C CNN
+F 2 "Resistors_THT:R_Axial_DIN0207_L6.3mm_D2.5mm_P10.16mm_Horizontal" V 6280 4300 50  0001 C CNN
 F 3 "" H 6350 4300 50  0000 C CNN
 	1    6350 4300
@@
 Text Label 1000 950  0    60   ~ 0
 SIG_TSAL
-Text Label 1000 1050 0    60   ~ 0
+Text Label 1000 1150 0    60   ~ 0
 CAN_TX
 Text Label 1000 1250 0    60   ~ 0
 AIRS_FINAL
-Text Label 1000 1150 0    60   ~ 0
+Text Label 1000 1050 0    60   ~ 0
 CAN_RX
 Text Notes 7700 1800 0    60   ~ 0
@@
 F 0 "R9" V 6730 3800 50  0000 C CNN
 F 1 "R" V 6650 3800 50  0000 C CNN
-F 2 "Resistors_THT:R_Axial_DIN0411_L9.9mm_D3.6mm_P12.70mm_Horizontal" V 6580 3800 50  0001 C CNN
+F 2 "Resistors_THT:R_Axial_DIN0207_L6.3mm_D2.5mm_P10.16mm_Horizontal" V 6580 3800 50  0001 C CNN
 F 3 "" H 6650 3800 50  0001 C CNN
 	1    6650 3800
@@
 F 0 "R5" V 6730 2950 50  0000 C CNN
 F 1 "R" V 6650 2950 50  0000 C CNN
-F 2 "Resistors_THT:R_Axial_DIN0411_L9.9mm_D3.6mm_P12.70mm_Horizontal" V 6580 2950 50  0001 C CNN
+F 2 "Resistors_THT:R_Axial_DIN0207_L6.3mm_D2.5mm_P10.16mm_Horizontal" V 6580 2950 50  0001 C CNN
 F 3 "" H 6650 2950 50  0001 C CNN
 	1    6650 2950
@@
 F 0 "R2" V 6730 2100 50  0000 C CNN
 F 1 "R" V 6650 2100 50  0000 C CNN
-F 2 "Resistors_THT:R_Axial_DIN0411_L9.9mm_D3.6mm_P12.70mm_Horizontal" V 6580 2100 50  0001 C CNN
+F 2 "Resistors_THT:R_Axial_DIN0207_L6.3mm_D2.5mm_P10.16mm_Horizontal" V 6580 2100 50  0001 C CNN
 F 3 "" H 6650 2100 50  0001 C CNN
 	1    6650 2100
@@
 F 0 "R1" V 5930 1450 50  0000 C CNN
 F 1 "120" V 5850 1450 50  0000 C CNN
-F 2 "Resistors_THT:R_Axial_DIN0411_L9.9mm_D3.6mm_P12.70mm_Horizontal" V 5780 1450 50  0001 C CNN
+F 2 "Resistors_THT:R_Axial_DIN0207_L6.3mm_D2.5mm_P10.16mm_Horizontal" V 5780 1450 50  0001 C CNN
 F 3 "" H 5850 1450 50  0001 C CNN
 	1    5850 1450
@@
 L Conn_01x01 H1
 U 1 1 5A94B007
+P 10950 5750
+F 0 "H1" H 10950 5850 50  0000 C CNN
+F 1 "MtngHole" H 10950 5650 50  0000 C CNN
+F 2 "Mounting_Holes:MountingHole_4.5mm" H 10950 5750 50  0001 C CNN
+F 3 "" H 10950 5750 50  0001 C CNN
+	1    10950 5750
+	1    0    0    -1
+$EndComp
+$Comp
+L Conn_01x01 H2
+U 1 1 5A94B644
 P 10950 6050
-F 0 "H1" H 10950 6150 50  0000 C CNN
+F 0 "H2" H 10950 6150 50  0000 C CNN
 F 1 "MtngHole" H 10950 5950 50  0000 C CNN
 F 2 "Mounting_Holes:MountingHole_4.5mm" H 10950 6050 50  0001 C CNN
@@
 $EndComp
 $Comp
-L Conn_01x01 H2
-U 1 1 5A94B644
+L Conn_01x01 H3
+U 1 1 5A9A4C65
 P 10950 6350
-F 0 "H2" H 10950 6450 50  0000 C CNN
+F 0 "H3" H 10950 6450 50  0000 C CNN
 F 1 "MtngHole" H 10950 6250 50  0000 C CNN
 F 2 "Mounting_Holes:MountingHole_4.5mm" H 10950 6350 50  0001 C CNN
