File: PEBoardHV/PEBoardHV.sch (KiCad schematic (older format))
At the start: 45 parts, among them J1 To PE LV, J2 Left Connector (Master), J3 E-Meter Internal, J4 Right Connector (Slave), J5 E-Meter External, J6 HV Cable, J7 TSMPs, J8 HV CAN Debug, J9 EMeter HV, U1 L78S05CV-DG, U2 ISO1050, U3 PS2501-4, U4 DK1A1B-12V, U5 DK1A1B-12V

Commit message: Un-fuse TSMPs
Changed lines of the file:
@@
 $EndComp
 Text Label 10200 3550 2    60   ~ 0
-TS+_FUSED
+TS+
 Text Label 10500 3950 3    60   ~ 0
 TS-

Commit message: edit PCBs based on actual parts that have arrived
Parts:
- added V1, V2, V3, V4, V5, V6, V7, V8, V9: ViaBlock, FSFootprints:ViaBlock-0.8mm, symbol Conn_01x01
- R13, R14: footprint TO_SOT_Packages_THT:TO-220-2_Vertical -> FSFootprints:TO-220-2_Horizontal_HeatSunk
- U2: footprint SMD_Packages:DIP-8_SMD -> Housings_DIP:DIP-8_W8.89mm_SMDSocket_LongPads
Changed lines of the file:
@@
 F 0 "U2" H 5500 1450 60  0000 C CNN
 F 1 "ISO1050" H 5200 1450 60  0000 C CNN
-F 2 "SMD_Packages:DIP-8_SMD" H 4400 1050 60  0001 C CNN
+F 2 "Housings_DIP:DIP-8_W8.89mm_SMDSocket_LongPads" H 4400 1050 60  0001 C CNN
 F 3 "" H 5200 1450 60  0000 C CNN
 	1    5250 1450
@@
 F 0 "R13" V 5680 6200 50  0000 C CNN
 F 1 "1K" V 5600 6200 50  0000 C CNN
-F 2 "TO_SOT_Packages_THT:TO-220-2_Vertical" V 5530 6200 50  0001 C CNN
+F 2 "FSFootprints:TO-220-2_Horizontal_HeatSunk" V 5530 6200 50  0001 C CNN
 F 3 "" H 5600 6200 50  0000 C CNN
 	1    5600 6200
-	0    1    1    0
+	0    -1   -1   0
 $EndComp
 $Comp
@@
 F 0 "R14" V 5680 7500 50  0000 C CNN
 F 1 "1K" V 5600 7500 50  0000 C CNN
-F 2 "TO_SOT_Packages_THT:TO-220-2_Vertical" V 5530 7500 50  0001 C CNN
+F 2 "FSFootprints:TO-220-2_Horizontal_HeatSunk" V 5530 7500 50  0001 C CNN
 F 3 "" H 5600 7500 50  0000 C CNN
 	1    5600 7500
-	0    1    1    0
+	0    -1   -1   0
 $EndComp
 Text Label 5450 5500 0    60   ~ 0
@@
 $EndComp
 $Comp
-L +12V #PWR01
+L +12V #PWR1
 U 1 1 59B389E9
 P 1000 650
-F 0 "#PWR01" H 1000 500 50  0001 C CNN
+F 0 "#PWR1" H 1000 500 50  0001 C CNN
 F 1 "+12V" H 1000 790 50  0000 C CNN
 F 2 "" H 1000 650 50  0001 C CNN
@@
 $EndComp
 $Comp
-L GND #PWR02
+L GND #PWR4
 U 1 1 59B39840
 P 1250 1350
-F 0 "#PWR02" H 1250 1100 50  0001 C CNN
+F 0 "#PWR4" H 1250 1100 50  0001 C CNN
 F 1 "GND" H 1250 1200 50  0000 C CNN
 F 2 "" H 1250 1350 50  0001 C CNN
@@
 	1250 1350 1000 1350
 $Comp
-L GND #PWR03
+L GND #PWR6
 U 1 1 59B39AB1
 P 1000 2250
-F 0 "#PWR03" H 1000 2000 50  0001 C CNN
+F 0 "#PWR6" H 1000 2000 50  0001 C CNN
 F 1 "GND" H 1000 2100 50  0000 C CNN
 F 2 "" H 1000 2250 50  0001 C CNN
@@
 $EndComp
 $Comp
-L +12V #PWR04
+L +12V #PWR5
 U 1 1 59B39B0B
 P 1000 1950
-F 0 "#PWR04" H 1000 1800 50  0001 C CNN
+F 0 "#PWR5" H 1000 1800 50  0001 C CNN
 F 1 "+12V" H 1000 2090 50  0000 C CNN
 F 2 "" H 1000 1950 50  0001 C CNN
@@
 $EndComp
 $Comp
-L GND #PWR05
+L GND #PWR8
 U 1 1 59B39C75
 P 1000 3100
-F 0 "#PWR05" H 1000 2850 50  0001 C CNN
+F 0 "#PWR8" H 1000 2850 50  0001 C CNN
 F 1 "GND" H 1000 2950 50  0000 C CNN
 F 2 "" H 1000 3100 50  0001 C CNN
@@
 $EndComp
 $Comp
-L +12V #PWR06
+L +12V #PWR7
 U 1 1 59B39C7B
 P 1000 2800
-F 0 "#PWR06" H 1000 2650 50  0001 C CNN
+F 0 "#PWR7" H 1000 2650 50  0001 C CNN
 F 1 "+12V" H 1000 2940 50  0000 C CNN
 F 2 "" H 1000 2800 50  0001 C CNN
@@
 $EndComp
 $Comp
-L GND #PWR07
+L GND #PWR2
 U 1 1 5A3F3240
 P 2450 1150
-F 0 "#PWR07" H 2450 900 50  0001 C CNN
+F 0 "#PWR2" H 2450 900 50  0001 C CNN
 F 1 "GND" H 2450 1000 50  0000 C CNN
 F 2 "" H 2450 1150 50  0001 C CNN
@@
 $EndComp
 $Comp
-L GND #PWR08
+L GND #PWR3
 U 1 1 5A3F32CD
 P 2950 1150
-F 0 "#PWR08" H 2950 900 50  0001 C CNN
+F 0 "#PWR3" H 2950 900 50  0001 C CNN
 F 1 "GND" H 2950 1000 50  0000 C CNN
 F 2 "" H 2950 1150 50  0001 C CNN
@@
 L Conn_01x01 H1
 U 1 1 5A94B007
-P 10950 5750
-F 0 "H1" H 10950 5850 50  0000 C CNN
-F 1 "MtngHole" H 10950 5650 50  0000 C CNN
-F 2 "Mounting_Holes:MountingHole_4.5mm" H 10950 5750 50  0001 C CNN
-F 3 "" H 10950 5750 50  0001 C CNN
-	1    10950 5750
+P 12400 5750
+F 0 "H1" H 12400 5850 50  0000 C CNN
+F 1 "MtngHole" H 12400 5650 50  0000 C CNN
+F 2 "Mounting_Holes:MountingHole_4.5mm" H 12400 5750 50  0001 C CNN
+F 3 "" H 12400 5750 50  0001 C CNN
+	1    12400 5750
 	1    0    0    -1
 $EndComp
@@
 L Conn_01x01 H2
 U 1 1 5A94B644
-P 10950 6050
-F 0 "H2" H 10950 6150 50  0000 C CNN
-F 1 "MtngHole" H 10950 5950 50  0000 C CNN
-F 2 "Mounting_Holes:MountingHole_4.5mm" H 10950 6050 50  0001 C CNN
-F 3 "" H 10950 6050 50  0001 C CNN
-	1    10950 6050
+P 12400 6050
+F 0 "H2" H 12400 6150 50  0000 C CNN
+F 1 "MtngHole" H 12400 5950 50  0000 C CNN
+F 2 "Mounting_Holes:MountingHole_4.5mm" H 12400 6050 50  0001 C CNN
+F 3 "" H 12400 6050 50  0001 C CNN
+	1    12400 6050
 	1    0    0    -1
 $EndComp
@@
 L Conn_01x01 H3
 U 1 1 5A9A4C65
-P 10950 6350
-F 0 "H3" H 10950 6450 50  0000 C CNN
-F 1 "MtngHole" H 10950 6250 50  0000 C CNN
-F 2 "Mounting_Holes:MountingHole_4.5mm" H 10950 6350 50  0001 C CNN
-F 3 "" H 10950 6350 50  0001 C CNN
-	1    10950 6350
-	1    0    0    -1
-$EndComp
+P 12400 6350
+F 0 "H3" H 12400 6450 50  0000 C CNN
+F 1 "MtngHole" H 12400 6250 50  0000 C CNN
+F 2 "Mounting_Holes:MountingHole_4.5mm" H 12400 6350 50  0001 C CNN
+F 3 "" H 12400 6350 50  0001 C CNN
+	1    12400 6350
+	1    0    0    -1
+$EndComp
+$Comp
+L Conn_01x01 V1
+U 1 1 5AB46FBF
+P 12900 5750
+F 0 "V1" H 12900 5850 50  0000 C CNN
+F 1 "ViaBlock" H 12900 5650 50  0000 C CNN
+F 2 "FSFootprints:ViaBlock-0.8mm" H 12900 5750 50  0001 C CNN
+F 3 "" H 12900 5750 50  0001 C CNN
+	1    12900 5750
+	1    0    0    -1
+$EndComp
+$Comp
+L Conn_01x01 V4
+U 1 1 5AB474B5
+P 12900 6050
+F 0 "V4" H 12900 6150 50  0000 C CNN
+F 1 "ViaBlock" H 12900 5950 50  0000 C CNN
+F 2 "FSFootprints:ViaBlock-0.8mm" H 12900 6050 50  0001 C CNN
+F 3 "" H 12900 6050 50  0001 C CNN
+	1    12900 6050
+	1    0    0    -1
+$EndComp
+$Comp
+L Conn_01x01 V7
+U 1 1 5AB4755E
+P 12900 6350
+F 0 "V7" H 12900 6450 50  0000 C CNN
+F 1 "ViaBlock" H 12900 6250 50  0000 C CNN
+F 2 "FSFootprints:ViaBlock-0.8mm" H 12900 6350 50  0001 C CNN
+F 3 "" H 12900 6350 50  0001 C CNN
+	1    12900 6350
+	1    0    0    -1
+$EndComp
+$Comp
+L Conn_01x01 V2
+U 1 1 5AB4779F
+P 13350 5750
+F 0 "V2" H 13350 5850 50  0000 C CNN
+F 1 "ViaBlock" H 13350 5650 50  0000 C CNN
+F 2 "FSFootprints:ViaBlock-0.8mm" H 13350 5750 50  0001 C CNN
+F 3 "" H 13350 5750 50  0001 C CNN
+	1    13350 5750
+	1    0    0    -1
+$EndComp
+$Comp
+L Conn_01x01 V5
+U 1 1 5AB477A5
+P 13350 6050
+F 0 "V5" H 13350 6150 50  0000 C CNN
+F 1 "ViaBlock" H 13350 5950 50  0000 C CNN
+F 2 "FSFootprints:ViaBlock-0.8mm" H 13350 6050 50  0001 C CNN
+F 3 "" H 13350 6050 50  0001 C CNN
+	1    13350 6050
+	1    0    0    -1
+$EndComp
+$Comp
+L Conn_01x01 V8
+U 1 1 5AB477AB
+P 13350 6350
+F 0 "V8" H 13350 6450 50  0000 C CNN
+F 1 "ViaBlock" H 13350 6250 50  0000 C CNN
+F 2 "FSFootprints:ViaBlock-0.8mm" H 13350 6350 50  0001 C CNN
+F 3 "" H 13350 6350 50  0001 C CNN
+	1    13350 6350
+	1    0    0    -1
+$EndComp
+Text Label 12700 5750 2    60   ~ 0
+TS-
+Text Label 12700 6050 2    60   ~ 0
+TS-
+Text Label 12700 6350 2    60   ~ 0
+TS-
+Text Label 13150 6350 2    60   ~ 0
+TS-
+Text Label 13150 6050 2    60   ~ 0
+TS-
+Text Label 13150 5750 2    60   ~ 0
+TS-
+$Comp
+L Conn_01x01 V9
+U 1 1 5AB48E7B
+P 13800 6350
+F 0 "V9" H 13800 6450 50  0000 C CNN
+F 1 "ViaBlock" H 13800 6250 50  0000 C CNN
+F 2 "FSFootprints:ViaBlock-0.8mm" H 13800 6350 50  0001 C CNN
+F 3 "" H 13800 6350 50  0001 C CNN
+	1    13800 6350
+	1    0    0    -1
+$EndComp
+Text Label 13600 6350 2    60   ~ 0
+TS-
+$Comp
+L Conn_01x01 V6
+U 1 1 5AB4A9C2
+P 13800 6050
+F 0 "V6" H 13800 6150 50  0000 C CNN
+F 1 "ViaBlock" H 13800 5950 50  0000 C CNN
+F 2 "FSFootprints:ViaBlock-0.8mm" H 13800 6050 50  0001 C CNN
+F 3 "" H 13800 6050 50  0001 C CNN
+	1    13800 6050
+	1    0    0    -1
+$EndComp
+$Comp
+L Conn_01x01 V3
+U 1 1 5AB4AA7F
+P 13800 5750
+F 0 "V3" H 13800 5850 50  0000 C CNN
+F 1 "ViaBlock" H 13800 5650 50  0000 C CNN
+F 2 "FSFootprints:ViaBlock-0.8mm" H 13800 5750 50  0001 C CNN
+F 3 "" H 13800 5750 50  0001 C CNN
+	1    13800 5750
+	1    0    0    -1
+$EndComp
+Text Label 13600 6050 2    60   ~ 0
+TS-
+Text Label 13600 5750 2    60   ~ 0
+TS-
 $EndSCHEMATC

Commit message: add fuse to CAN+ line on PE HV board
Parts:
- removed H3: MtngHole, Mounting_Holes:MountingHole_4.5mm, symbol Conn_01x01
- added F1: Fuse, FSFootprints:SMD Fuse, symbol Fuse
- added J10: Discharge Jumper, Pin_Headers:Pin_Header_Straight_2x01_Pitch2.54mm, symbol Conn_01x02
- D1, D2, D3, D4, D5, D6: footprint Diodes_THT:D_A-405_P10.16mm_Horizontal -> Diodes_THT:D_A-405_P7.62mm_Horizontal
- renumbered F1 to F2, F2 to F3, F3 to F4
Connections:
- net labels added: DISCHARGE_L, DISCHARGE_R
Changed lines of the file:
@@
 Text Notes 8550 900  2    60   ~ 0
 Voltage Regulator HV
-Text Label 7750 1150 2    60   ~ 0
+Text Label 7450 1150 2    60   ~ 0
 CAN+
 Text Label 8550 1150 0    60   ~ 0
@@
 F 0 "D1" H 6350 2200 50  0000 C CNN
 F 1 "48V Zener" H 6350 2000 50  0000 C CNN
-F 2 "Diodes_THT:D_A-405_P10.16mm_Horizontal" H 6350 2100 50  0001 C CNN
+F 2 "Diodes_THT:D_A-405_P7.62mm_Horizontal" H 6350 2100 50  0001 C CNN
 F 3 "" H 6350 2100 50  0000 C CNN
 	1    6350 2100
@@
 F 0 "D2" H 6200 2550 50  0000 C CNN
 F 1 "12V Zener" H 6200 2350 50  0000 C CNN
-F 2 "Diodes_THT:D_A-405_P10.16mm_Horizontal" H 6200 2450 50  0001 C CNN
+F 2 "Diodes_THT:D_A-405_P7.62mm_Horizontal" H 6200 2450 50  0001 C CNN
 F 3 "" H 6200 2450 50  0000 C CNN
 	1    6200 2450
@@
 F 0 "D3" H 6350 3050 50  0000 C CNN
 F 1 "48V Zener" H 6350 2850 50  0000 C CNN
-F 2 "Diodes_THT:D_A-405_P10.16mm_Horizontal" H 6350 2950 50  0001 C CNN
+F 2 "Diodes_THT:D_A-405_P7.62mm_Horizontal" H 6350 2950 50  0001 C CNN
 F 3 "" H 6350 2950 50  0000 C CNN
 	1    6350 2950
@@
 F 0 "D4" H 6200 3400 50  0000 C CNN
 F 1 "12V Zener" H 6200 3200 50  0000 C CNN
-F 2 "Diodes_THT:D_A-405_P10.16mm_Horizontal" H 6200 3300 50  0001 C CNN
+F 2 "Diodes_THT:D_A-405_P7.62mm_Horizontal" H 6200 3300 50  0001 C CNN
 F 3 "" H 6200 3300 50  0000 C CNN
 	1    6200 3300
@@
 F 0 "D5" H 6350 3900 50  0000 C CNN
 F 1 "48V Zener" H 6350 3700 50  0000 C CNN
-F 2 "Diodes_THT:D_A-405_P10.16mm_Horizontal" H 6350 3800 50  0001 C CNN
+F 2 "Diodes_THT:D_A-405_P7.62mm_Horizontal" H 6350 3800 50  0001 C CNN
 F 3 "" H 6350 3800 50  0000 C CNN
 	1    6350 3800
@@
 F 0 "D6" H 6200 4250 50  0000 C CNN
 F 1 "12V Zener" H 6200 4050 50  0000 C CNN
-F 2 "Diodes_THT:D_A-405_P10.16mm_Horizontal" H 6200 4150 50  0001 C CNN
+F 2 "Diodes_THT:D_A-405_P7.62mm_Horizontal" H 6200 4150 50  0001 C CNN
 F 3 "" H 6200 4150 50  0000 C CNN
 	1    6200 4150
@@
 	6200 3800 6200 4000
 $Comp
-L Fuse F1
+L Fuse F2
 U 1 1 58C4C02B
 P 6950 2100
-F 0 "F1" V 7030 2100 50  0000 C CNN
+F 0 "F2" V 7030 2100 50  0000 C CNN
 F 1 "Fuse" V 6875 2100 50  0000 C CNN
 F 2 "FSFootprints:SMD Fuse" V 6880 2100 50  0001 C CNN
@@
 $EndComp
 $Comp
-L Fuse F2
+L Fuse F3
 U 1 1 58C4C0C4
 P 6950 2950
-F 0 "F2" V 7030 2950 50  0000 C CNN
+F 0 "F3" V 7030 2950 50  0000 C CNN
 F 1 "Fuse" V 6875 2950 50  0000 C CNN
 F 2 "FSFootprints:SMD Fuse" V 6880 2950 50  0001 C CNN
@@
 $EndComp
 $Comp
-L Fuse F3
+L Fuse F4
 U 1 1 58C4C15E
 P 6950 3800
-F 0 "F3" V 7030 3800 50  0000 C CNN
+F 0 "F4" V 7030 3800 50  0000 C CNN
 F 1 "Fuse" V 6875 3800 50  0000 C CNN
 F 2 "FSFootprints:SMD Fuse" V 6880 3800 50  0001 C CNN
@@
 $EndComp
 $Comp
-L Conn_01x01 H3
-U 1 1 5A9A4C65
-P 12400 6350
-F 0 "H3" H 12400 6450 50  0000 C CNN
-F 1 "MtngHole" H 12400 6250 50  0000 C CNN
-F 2 "Mounting_Holes:MountingHole_4.5mm" H 12400 6350 50  0001 C CNN
-F 3 "" H 12400 6350 50  0001 C CNN
-	1    12400 6350
-	1    0    0    -1
-$EndComp
-$Comp
 L Conn_01x01 V1
 U 1 1 5AB46FBF
@@
 Text Label 13600 5750 2    60   ~ 0
 TS-
+Text Label 5450 6200 2    60   ~ 0
+DISCHARGE_L
+Text Label 5450 7500 2    60   ~ 0
+DISCHARGE_R
+Text Label 6350 6400 2    60   ~ 0
+DISCHARGE_L
+Text Label 6350 6500 2    60   ~ 0
+DISCHARGE_R
+$Comp
+L Conn_01x02 J10
+U 1 1 5AB89F55
+P 6550 6400
+F 0 "J10" H 6550 6500 50  0000 C CNN
+F 1 "Discharge Jumper" H 6550 6200 50  0000 C CNN
+F 2 "Pin_Headers:Pin_Header_Straight_2x01_Pitch2.54mm" H 6550 6400 50  0001 C CNN
+F 3 "" H 6550 6400 50  0001 C CNN
+	1    6550 6400
+	1    0    0    -1
+$EndComp
+$Comp
+L Fuse F1
+U 1 1 5AB87628
+P 7600 1150
+F 0 "F1" V 7680 1150 50  0000 C CNN
+F 1 "Fuse" V 7525 1150 50  0000 C CNN
+F 2 "FSFootprints:SMD Fuse" V 7530 1150 50  0001 C CNN
+F 3 "" H 7600 1150 50  0000 C CNN
+	1    7600 1150
+	0    1    1    0
+$EndComp
 $EndSCHEMATC

Commit message: Tweak 60v circuits based on testing results
Parts:
- removed R2, R5, R9: R, Resistors_THT:R_Axial_DIN0207_L6.3mm_D2.5mm_P10.16mm_Horizontal, symbol R
- D1, D3, D5: value 48V Zener -> 56V Zener
- R12, R4, R7: value 3kR -> 1.5k
Changed lines of the file:
@@
 P 6350 2100
 F 0 "D1" H 6350 2200 50  0000 C CNN
-F 1 "48V Zener" H 6350 2000 50  0000 C CNN
+F 1 "56V Zener" H 6350 2000 50  0000 C CNN
 F 2 "Diodes_THT:D_A-405_P7.62mm_Horizontal" H 6350 2100 50  0001 C CNN
 F 3 "" H 6350 2100 50  0000 C CNN
@@
 P 6350 2950
 F 0 "D3" H 6350 3050 50  0000 C CNN
-F 1 "48V Zener" H 6350 2850 50  0000 C CNN
+F 1 "56V Zener" H 6350 2850 50  0000 C CNN
 F 2 "Diodes_THT:D_A-405_P7.62mm_Horizontal" H 6350 2950 50  0001 C CNN
 F 3 "" H 6350 2950 50  0000 C CNN
@@
 P 6350 3800
 F 0 "D5" H 6350 3900 50  0000 C CNN
-F 1 "48V Zener" H 6350 3700 50  0000 C CNN
+F 1 "56V Zener" H 6350 3700 50  0000 C CNN
 F 2 "Diodes_THT:D_A-405_P7.62mm_Horizontal" H 6350 3800 50  0001 C CNN
 F 3 "" H 6350 3800 50  0000 C CNN
@@
 L Fuse F2
 U 1 1 58C4C02B
-P 6950 2100
-F 0 "F2" V 7030 2100 50  0000 C CNN
-F 1 "Fuse" V 6875 2100 50  0000 C CNN
-F 2 "FSFootprints:SMD Fuse" V 6880 2100 50  0001 C CNN
-F 3 "" H 6950 2100 50  0000 C CNN
-	1    6950 2100
+P 6650 2100
+F 0 "F2" V 6730 2100 50  0000 C CNN
+F 1 "Fuse" V 6575 2100 50  0000 C CNN
+F 2 "FSFootprints:SMD Fuse" V 6580 2100 50  0001 C CNN
+F 3 "" H 6650 2100 50  0000 C CNN
+	1    6650 2100
 	0    1    1    0
 $EndComp
@@
 L Fuse F3
 U 1 1 58C4C0C4
-P 6950 2950
-F 0 "F3" V 7030 2950 50  0000 C CNN
-F 1 "Fuse" V 6875 2950 50  0000 C CNN
-F 2 "FSFootprints:SMD Fuse" V 6880 2950 50  0001 C CNN
-F 3 "" H 6950 2950 50  0000 C CNN
-	1    6950 2950
+P 6650 2950
+F 0 "F3" V 6730 2950 50  0000 C CNN
+F 1 "Fuse" V 6575 2950 50  0000 C CNN
+F 2 "FSFootprints:SMD Fuse" V 6580 2950 50  0001 C CNN
+F 3 "" H 6650 2950 50  0000 C CNN
+	1    6650 2950
 	0    1    1    0
 $EndComp
@@
 L Fuse F4
 U 1 1 58C4C15E
-P 6950 3800
-F 0 "F4" V 7030 3800 50  0000 C CNN
-F 1 "Fuse" V 6875 3800 50  0000 C CNN
-F 2 "FSFootprints:SMD Fuse" V 6880 3800 50  0001 C CNN
-F 3 "" H 6950 3800 50  0000 C CNN
-	1    6950 3800
+P 6650 3800
+F 0 "F4" V 6730 3800 50  0000 C CNN
+F 1 "Fuse" V 6575 3800 50  0000 C CNN
+F 2 "FSFootprints:SMD Fuse" V 6580 3800 50  0001 C CNN
+F 3 "" H 6650 3800 50  0000 C CNN
+	1    6650 3800
 	0    1    1    0
 $EndComp
@@
 P 6350 2600
 F 0 "R4" V 6430 2600 50  0000 C CNN
-F 1 "3kR" V 6350 2600 50  0000 C CNN
+F 1 "1.5k" V 6350 2600 50  0000 C CNN
 F 2 "Resistors_THT:R_Axial_DIN0207_L6.3mm_D2.5mm_P10.16mm_Horizontal" V 6280 2600 50  0001 C CNN
 F 3 "" H 6350 2600 50  0000 C CNN
@@
 P 6350 3450
 F 0 "R7" V 6430 3450 50  0000 C CNN
-F 1 "3kR" V 6350 3450 50  0000 C CNN
+F 1 "1.5k" V 6350 3450 50  0000 C CNN
 F 2 "Resistors_THT:R_Axial_DIN0207_L6.3mm_D2.5mm_P10.16mm_Horizontal" V 6280 3450 50  0001 C CNN
 F 3 "" H 6350 3450 50  0000 C CNN
@@
 P 6350 4300
 F 0 "R12" V 6430 4300 50  0000 C CNN
-F 1 "3kR" V 6350 4300 50  0000 C CNN
+F 1 "1.5k" V 6350 4300 50  0000 C CNN
 F 2 "Resistors_THT:R_Axial_DIN0207_L6.3mm_D2.5mm_P10.16mm_Horizontal" V 6280 4300 50  0001 C CNN
 F 3 "" H 6350 4300 50  0000 C CNN
@@
 Text Label 4950 4250 2    60   ~ 0
 SIG_TSAL
-Text Label 7100 2100 0    60   ~ 0
+Text Label 6800 2100 0    60   ~ 0
 TS+_SWITCHED_L
-Text Label 7100 2950 0    60   ~ 0
+Text Label 6800 2950 0    60   ~ 0
 TS+_SWITCHED_R
-Text Label 7100 3800 0    60   ~ 0
+Text Label 6800 3800 0    60   ~ 0
 TS+
 Text Label 1000 750  0    60   ~ 0
@@
 Needs (Small) Heat Sink!
 $Comp
-L R R9
-U 1 1 59B378CF
-P 6650 3800
-F 0 "R9" V 6730 3800 50  0000 C CNN
-F 1 "R" V 6650 3800 50  0000 C CNN
-F 2 "Resistors_THT:R_Axial_DIN0207_L6.3mm_D2.5mm_P10.16mm_Horizontal" V 6580 3800 50  0001 C CNN
-F 3 "" H 6650 3800 50  0001 C CNN
-	1    6650 3800
-	0    1    1    0
-$EndComp
-$Comp
-L R R5
-U 1 1 59B3797A
-P 6650 2950
-F 0 "R5" V 6730 2950 50  0000 C CNN
-F 1 "R" V 6650 2950 50  0000 C CNN
-F 2 "Resistors_THT:R_Axial_DIN0207_L6.3mm_D2.5mm_P10.16mm_Horizontal" V 6580 2950 50  0001 C CNN
-F 3 "" H 6650 2950 50  0001 C CNN
-	1    6650 2950
-	0    1    1    0
-$EndComp
-$Comp
-L R R2
-U 1 1 59B37B6E
-P 6650 2100
-F 0 "R2" V 6730 2100 50  0000 C CNN
-F 1 "R" V 6650 2100 50  0000 C CNN
-F 2 "Resistors_THT:R_Axial_DIN0207_L6.3mm_D2.5mm_P10.16mm_Horizontal" V 6580 2100 50  0001 C CNN
-F 3 "" H 6650 2100 50  0001 C CNN
-	1    6650 2100
-	0    1    1    0
-$EndComp
-$Comp
 L +12V #PWR1
 U 1 1 59B389E9
@@
 	1    0    0    -1
 $EndComp
-Wire Wire Line
-	6800 3800 6800 3500
-Text Label 6800 3500 0    60   ~ 0
+Text Label 6500 4000 0    60   ~ 0
 TS+_FUSED
 Text Label 10500 5400 2    60   ~ 0
@@
 	0    1    1    0
 $EndComp
+Wire Wire Line
+	6500 4000 6500 3800
 $EndSCHEMATC

Commit message: push schematic updates for 60V on PE HV
Parts:
- renumbered R13 to R10, R14 to R11, R3 to R2, R4 to R3, R6 to R4, R7 to R5, R8 to R6, R10 to R7, R11 to R8, R12 to R9
Changed lines of the file:
@@
 CAN_H_BOARD
 $Comp
-L R R13
+L R R10
 U 1 1 588D76FB
 P 5600 6200
-F 0 "R13" V 5680 6200 50  0000 C CNN
+F 0 "R10" V 5680 6200 50  0000 C CNN
 F 1 "1K" V 5600 6200 50  0000 C CNN
 F 2 "FSFootprints:TO-220-2_Horizontal_HeatSunk" V 5530 6200 50  0001 C CNN
@@
 $EndComp
 $Comp
-L R R14
+L R R11
 U 1 1 588D7799
 P 5600 7500
-F 0 "R14" V 5680 7500 50  0000 C CNN
+F 0 "R11" V 5680 7500 50  0000 C CNN
 F 1 "1K" V 5600 7500 50  0000 C CNN
 F 2 "FSFootprints:TO-220-2_Horizontal_HeatSunk" V 5530 7500 50  0001 C CNN
@@
 $EndComp
 $Comp
-L R R8
+L R R6
 U 1 1 58916788
 P 10350 3550
-F 0 "R8" V 10430 3550 50  0000 C CNN
+F 0 "R6" V 10430 3550 50  0000 C CNN
 F 1 "5kR" V 10350 3550 50  0000 C CNN
 F 2 "Resistors_THT:R_Axial_DIN0414_L11.9mm_D4.5mm_P20.32mm_Horizontal" V 10280 3550 50  0001 C CNN
@@
 $EndComp
 $Comp
-L R R10
+L R R7
 U 1 1 58916808
 P 10500 3800
-F 0 "R10" V 10580 3800 50  0000 C CNN
+F 0 "R7" V 10580 3800 50  0000 C CNN
 F 1 "5kR" V 10500 3800 50  0000 C CNN
 F 2 "Resistors_THT:R_Axial_DIN0414_L11.9mm_D4.5mm_P20.32mm_Horizontal" V 10430 3800 50  0001 C CNN
@@
 $EndComp
 $Comp
-L R R3
+L R R2
 U 1 1 58C4AF19
 P 5700 2350
-F 0 "R3" V 5780 2350 50  0000 C CNN
+F 0 "R2" V 5780 2350 50  0000 C CNN
 F 1 "1.2kR" V 5700 2350 50  0000 C CNN
 F 2 "Resistors_THT:R_Axial_DIN0207_L6.3mm_D2.5mm_P10.16mm_Horizontal" V 5630 2350 50  0001 C CNN
@@
 $EndComp
 $Comp
-L R R6
+L R R4
 U 1 1 58C4B7BC
 P 5700 3200
-F 0 "R6" V 5780 3200 50  0000 C CNN
+F 0 "R4" V 5780 3200 50  0000 C CNN
 F 1 "1.2kR" V 5700 3200 50  0000 C CNN
 F 2 "Resistors_THT:R_Axial_DIN0207_L6.3mm_D2.5mm_P10.16mm_Horizontal" V 5630 3200 50  0001 C CNN
@@
 $EndComp
 $Comp
-L R R11
+L R R8
 U 1 1 58C4BA41
 P 5700 4050
-F 0 "R11" V 5780 4050 50  0000 C CNN
+F 0 "R8" V 5780 4050 50  0000 C CNN
 F 1 "1.2kR" V 5700 4050 50  0000 C CNN
 F 2 "Resistors_THT:R_Axial_DIN0207_L6.3mm_D2.5mm_P10.16mm_Horizontal" V 5630 4050 50  0001 C CNN
@@
 $EndComp
 $Comp
-L R R4
+L R R3
 U 1 1 58C4C8E9
 P 6350 2600
-F 0 "R4" V 6430 2600 50  0000 C CNN
+F 0 "R3" V 6430 2600 50  0000 C CNN
 F 1 "1.5k" V 6350 2600 50  0000 C CNN
 F 2 "Resistors_THT:R_Axial_DIN0207_L6.3mm_D2.5mm_P10.16mm_Horizontal" V 6280 2600 50  0001 C CNN
@@
 $EndComp
 $Comp
-L R R7
+L R R5
 U 1 1 58C4CA42
 P 6350 3450
-F 0 "R7" V 6430 3450 50  0000 C CNN
+F 0 "R5" V 6430 3450 50  0000 C CNN
 F 1 "1.5k" V 6350 3450 50  0000 C CNN
 F 2 "Resistors_THT:R_Axial_DIN0207_L6.3mm_D2.5mm_P10.16mm_Horizontal" V 6280 3450 50  0001 C CNN
@@
 $EndComp
 $Comp
-L R R12
+L R R9
 U 1 1 58C4CBDA
 P 6350 4300
-F 0 "R12" V 6430 4300 50  0000 C CNN
+F 0 "R9" V 6430 4300 50  0000 C CNN
 F 1 "1.5k" V 6350 4300 50  0000 C CNN
 F 2 "Resistors_THT:R_Axial_DIN0207_L6.3mm_D2.5mm_P10.16mm_Horizontal" V 6280 4300 50  0001 C CNN
@@
 Needs (Small) Heat Sink!
 $Comp
-L +12V #PWR1
+L +12V #PWR01
 U 1 1 59B389E9
 P 1000 650
-F 0 "#PWR1" H 1000 500 50  0001 C CNN
+F 0 "#PWR01" H 1000 500 50  0001 C CNN
 F 1 "+12V" H 1000 790 50  0000 C CNN
 F 2 "" H 1000 650 50  0001 C CNN
@@
 $EndComp
 $Comp
-L GND #PWR4
+L GND #PWR02
 U 1 1 59B39840
 P 1250 1350
-F 0 "#PWR4" H 1250 1100 50  0001 C CNN
+F 0 "#PWR02" H 1250 1100 50  0001 C CNN
 F 1 "GND" H 1250 1200 50  0000 C CNN
 F 2 "" H 1250 1350 50  0001 C CNN
@@
 	1250 1350 1000 1350
 $Comp
-L GND #PWR6
+L GND #PWR03
 U 1 1 59B39AB1
 P 1000 2250
-F 0 "#PWR6" H 1000 2000 50  0001 C CNN
+F 0 "#PWR03" H 1000 2000 50  0001 C CNN
 F 1 "GND" H 1000 2100 50  0000 C CNN
 F 2 "" H 1000 2250 50  0001 C CNN
@@
 $EndComp
 $Comp
-L +12V #PWR5
+L +12V #PWR04
 U 1 1 59B39B0B
 P 1000 1950
-F 0 "#PWR5" H 1000 1800 50  0001 C CNN
+F 0 "#PWR04" H 1000 1800 50  0001 C CNN
 F 1 "+12V" H 1000 2090 50  0000 C CNN
 F 2 "" H 1000 1950 50  0001 C CNN
@@
 $EndComp
 $Comp
-L GND #PWR8
+L GND #PWR05
 U 1 1 59B39C75
 P 1000 3100
-F 0 "#PWR8" H 1000 2850 50  0001 C CNN
+F 0 "#PWR05" H 1000 2850 50  0001 C CNN
 F 1 "GND" H 1000 2950 50  0000 C CNN
 F 2 "" H 1000 3100 50  0001 C CNN
@@
 $EndComp
 $Comp
-L +12V #PWR7
+L +12V #PWR06
 U 1 1 59B39C7B
 P 1000 2800
-F 0 "#PWR7" H 1000 2650 50  0001 C CNN
+F 0 "#PWR06" H 1000 2650 50  0001 C CNN
 F 1 "+12V" H 1000 2940 50  0000 C CNN
 F 2 "" H 1000 2800 50  0001 C CNN
@@
 $EndComp
 $Comp
-L GND #PWR2
+L GND #PWR07
 U 1 1 5A3F3240
 P 2450 1150
-F 0 "#PWR2" H 2450 900 50  0001 C CNN
+F 0 "#PWR07" H 2450 900 50  0001 C CNN
 F 1 "GND" H 2450 1000 50  0000 C CNN
 F 2 "" H 2450 1150 50  0001 C CNN
@@
 $EndComp
 $Comp
-L GND #PWR3
+L GND #PWR08
 U 1 1 5A3F32CD
 P 2950 1150
-F 0 "#PWR3" H 2950 900 50  0001 C CNN
+F 0 "#PWR08" H 2950 900 50  0001 C CNN
 F 1 "GND" H 2950 1000 50  0000 C CNN
 F 2 "" H 2950 1150 50  0001 C CNN
