File: PEBoardHV/PEBoardHV.sch (KiCad schematic (older format))
At the start: 52 parts, among them J1 To PE LV, J10 Discharge Jumper, J2 Left Connector (Master), J3 E-Meter Internal, J4 Right Connector (Slave), J5 E-Meter External, J6 HV Cable, J7 TSMPs, J8 HV CAN Debug, J9 EMeter HV, U1 L78S05CV-DG, U2 ISO1050, U3 PS2501-4, U4 DK1A1B-12V, U5 DK1A1B-12V

Commit message: Add TVS diode and choke to PE HV board
Parts:
- added D1: D_TVS_x2_AAC, TO_SOT_Packages_SMD:SOT-23_Handsoldering, symbol D_TVS_x2_AAC
- added FL1: EMI_Choke, FSFootprints:L_CommonMode_Choke, symbol EMI_Choke
- renumbered D1 to D2, D2 to D3, D3 to D4, D4 to D5, D5 to D6, D6 to D7
Connections:
- net labels added: CAN_H_PRE, CAN_L_PRE
- wire segments 25 -> 33
Changed lines of the file:
@@
 Text Notes 5450 7700 2    60   ~ 0
 GLV      TS
-Text Label 5850 1250 0    60   ~ 0
+Text Label 6750 1100 0    60   ~ 0
 CAN_H_BOARD
-Text Label 5850 1650 0    60   ~ 0
+Text Label 6750 1800 0    60   ~ 0
 CAN_L_BOARD
 $Comp
@@
 Text Notes 8550 900  2    60   ~ 0
 Voltage Regulator HV
-Text Label 7450 1150 2    60   ~ 0
+Text Label 7450 1150 3    60   ~ 0
 CAN+
 Text Label 8550 1150 0    60   ~ 0
@@
 NoConn ~ 10500 1400
 $Comp
-L D_Zener D1
+L D_Zener D2
 U 1 1 58C314A3
 P 6350 2100
-F 0 "D1" H 6350 2200 50  0000 C CNN
+F 0 "D2" H 6350 2200 50  0000 C CNN
 F 1 "56V Zener" H 6350 2000 50  0000 C CNN
 F 2 "Diodes_THT:D_A-405_P7.62mm_Horizontal" H 6350 2100 50  0001 C CNN
@@
 $EndComp
 $Comp
-L D_Zener D2
+L D_Zener D3
 U 1 1 58C31526
 P 6200 2450
-F 0 "D2" H 6200 2550 50  0000 C CNN
+F 0 "D3" H 6200 2550 50  0000 C CNN
 F 1 "12V Zener" H 6200 2350 50  0000 C CNN
 F 2 "Diodes_THT:D_A-405_P7.62mm_Horizontal" H 6200 2450 50  0001 C CNN
@@
 	6200 2100 6200 2300
 $Comp
-L D_Zener D3
+L D_Zener D4
 U 1 1 58C4B7AA
 P 6350 2950
-F 0 "D3" H 6350 3050 50  0000 C CNN
+F 0 "D4" H 6350 3050 50  0000 C CNN
 F 1 "56V Zener" H 6350 2850 50  0000 C CNN
 F 2 "Diodes_THT:D_A-405_P7.62mm_Horizontal" H 6350 2950 50  0001 C CNN
@@
 $EndComp
 $Comp
-L D_Zener D4
+L D_Zener D5
 U 1 1 58C4B7B0
 P 6200 3300
-F 0 "D4" H 6200 3400 50  0000 C CNN
+F 0 "D5" H 6200 3400 50  0000 C CNN
 F 1 "12V Zener" H 6200 3200 50  0000 C CNN
 F 2 "Diodes_THT:D_A-405_P7.62mm_Horizontal" H 6200 3300 50  0001 C CNN
@@
 	6200 2950 6200 3150
 $Comp
-L D_Zener D5
+L D_Zener D6
 U 1 1 58C4BA2F
 P 6350 3800
-F 0 "D5" H 6350 3900 50  0000 C CNN
+F 0 "D6" H 6350 3900 50  0000 C CNN
 F 1 "56V Zener" H 6350 3700 50  0000 C CNN
 F 2 "Diodes_THT:D_A-405_P7.62mm_Horizontal" H 6350 3800 50  0001 C CNN
@@
 $EndComp
 $Comp
-L D_Zener D6
+L D_Zener D7
 U 1 1 58C4BA35
 P 6200 4150
-F 0 "D6" H 6200 4250 50  0000 C CNN
+F 0 "D7" H 6200 4250 50  0000 C CNN
 F 1 "12V Zener" H 6200 4050 50  0000 C CNN
 F 2 "Diodes_THT:D_A-405_P7.62mm_Horizontal" H 6200 4150 50  0001 C CNN
@@
 L R R1
 U 1 1 5A837AFE
-P 5850 1450
-F 0 "R1" V 5930 1450 50  0000 C CNN
-F 1 "120" V 5850 1450 50  0000 C CNN
-F 2 "Resistors_THT:R_Axial_DIN0207_L6.3mm_D2.5mm_P10.16mm_Horizontal" V 5780 1450 50  0001 C CNN
-F 3 "" H 5850 1450 50  0001 C CNN
-	1    5850 1450
-	1    0    0    -1
-$EndComp
-Wire Wire Line
-	5850 1300 5850 1250
-Wire Wire Line
-	5850 1600 5850 1650
+P 7100 1450
+F 0 "R1" V 7180 1450 50  0000 C CNN
+F 1 "120" V 7100 1450 50  0000 C CNN
+F 2 "Resistors_THT:R_Axial_DIN0207_L6.3mm_D2.5mm_P10.16mm_Horizontal" V 7030 1450 50  0001 C CNN
+F 3 "" H 7100 1450 50  0001 C CNN
+	1    7100 1450
+	1    0    0    -1
+$EndComp
 $Comp
 L CP C1
@@
 Wire Wire Line
 	6500 4000 6500 3800
+$Comp
+L D_TVS_x2_AAC D1
+U 1 1 5AC2D38B
+P 6750 1450
+F 0 "D1" H 6750 1625 50  0000 C CNN
+F 1 "D_TVS_x2_AAC" H 6750 1550 50  0000 C CNN
+F 2 "TO_SOT_Packages_SMD:SOT-23_Handsoldering" H 6600 1450 50  0001 C CNN
+F 3 "" H 6600 1450 50  0001 C CNN
+	1    6750 1450
+	0    1    1    0
+$EndComp
+Text Label 5850 1250 1    60   ~ 0
+CAN_H_PRE
+Text Label 5850 1650 3    60   ~ 0
+CAN_L_PRE
+$Comp
+L EMI_Choke FL1
+U 1 1 5AC2DC18
+P 6200 1450
+F 0 "FL1" H 6200 1625 50  0000 C CNN
+F 1 "EMI_Choke" H 6200 1275 50  0000 C CNN
+F 2 "FSFootprints:L_CommonMode_Choke" V 6200 1490 50  0001 C CNN
+F 3 "" V 6200 1490 50  0000 C CNN
+	1    6200 1450
+	1    0    0    -1
+$EndComp
+Wire Wire Line
+	5850 1250 5850 1350
+Wire Wire Line
+	5850 1350 6000 1350
+Wire Wire Line
+	5850 1650 5850 1550
+Wire Wire Line
+	5850 1550 6000 1550
+Wire Wire Line
+	6400 1350 6400 1100
+Wire Wire Line
+	6400 1100 7100 1100
+Wire Wire Line
+	6400 1550 6400 1800
+Wire Wire Line
+	6400 1800 7100 1800
+Wire Wire Line
+	7100 1100 7100 1300
+Connection ~ 6750 1100
+Wire Wire Line
+	7100 1800 7100 1600
+Connection ~ 6750 1800
+Text Label 6600 1450 1    60   ~ 0
+TS-
 $EndSCHEMATC

Commit message: tweak boards slightly
Parts:
- C1, C2, C3: footprint Capacitors_THT:CP_Radial_D5.0mm_P2.50mm -> Capacitors_THT:C_Disc_D3.0mm_W1.6mm_P2.50mm
Changed lines of the file:
@@
 F 0 "C2" H 2475 1100 50  0000 L CNN
 F 1 "C" H 2475 900 50  0000 L CNN
-F 2 "Capacitors_THT:CP_Radial_D5.0mm_P2.50mm" H 2488 850 50  0001 C CNN
+F 2 "Capacitors_THT:C_Disc_D3.0mm_W1.6mm_P2.50mm" H 2488 850 50  0001 C CNN
 F 3 "" H 2450 1000 50  0001 C CNN
 	1    2450 1000
@@
 F 0 "C3" H 2975 1100 50  0000 L CNN
 F 1 "C" H 2975 900 50  0000 L CNN
-F 2 "Capacitors_THT:CP_Radial_D5.0mm_P2.50mm" H 2988 850 50  0001 C CNN
+F 2 "Capacitors_THT:C_Disc_D3.0mm_W1.6mm_P2.50mm" H 2988 850 50  0001 C CNN
 F 3 "" H 2950 1000 50  0001 C CNN
 	1    2950 1000
@@
 F 0 "C1" H 5525 1050 50  0000 L CNN
 F 1 "CP" H 5525 850 50  0000 L CNN
-F 2 "Capacitors_THT:CP_Radial_D5.0mm_P2.50mm" H 5538 800 50  0001 C CNN
+F 2 "Capacitors_THT:C_Disc_D3.0mm_W1.6mm_P2.50mm" H 5538 800 50  0001 C CNN
 F 3 "" H 5500 950 50  0001 C CNN
 	1    5500 950

Commit message: add diodes to relay coils among other things
Parts:
- removed J2: Left Connector (Master), Connectors_Molex:Molex_NanoFit_2x04x2.50mm_Straight, symbol Conn_01x08
- removed J4: Right Connector (Slave), Connectors_Molex:Molex_NanoFit_2x03x2.50mm_Straight, symbol Conn_01x06
- added D8, D9: D, Diodes_SMD:D_1206, symbol D
- added J1: Left Connector (Master), Connectors_Molex:Molex_NanoFit_2x03x2.50mm_Straight, symbol Conn_02x03_Top_Bottom
- added J3: Right Connector (Slave), Connectors_Molex:Molex_NanoFit_2x03x2.50mm_Straight, symbol Conn_02x03_Top_Bottom
- added J4: Ring Terminal Connector, Connectors_Molex:Molex_NanoFit_1x02x2.50mm_Straight, symbol Conn_01x02
- C1, C3: footprint Capacitors_THT:C_Disc_D3.0mm_W1.6mm_P2.50mm -> Capacitors_THT:C_Disc_D4.3mm_W1.9mm_P5.00mm
- R1: footprint Resistors_THT:R_Axial_DIN0207_L6.3mm_D2.5mm_P10.16mm_Horizontal -> Resistors_SMD:R_0805_HandSoldering
- renumbered J9 to J10, J10 to J11, J1 to J2, J3 to J5, J5 to J7, J7 to J8, J8 to J9, R6 to R4, R4 to R5, R7 to R6, R5 to R7
