File: AccumulatorBoardHV/AccumulatorBoardHV.sch (KiCad schematic (older format))
At the start: 42 parts, among them P1 Batt Voltage, P2 HV (Switched), P3 IMD HV, P4 HV -> LV Regulator Jumper, P5 Acc LED 1, P6 Acc LED 2, U1 V110C12E100BL

Commit message: Swapped out vreg for temp system, TS/GLV naming convention, added BMS pull up resistor
Parts:
- removed C?: CP, symbol CP
- removed DC?: RDD08110S12, symbol RDD08110S12
- removed U?: LD1117V33, TO-220, symbol LD1117V33
- added U?: RDD08110S3V3, symbol RDD08110S3V3
- P2: value HV (Switched) -> TS (Switched)
- P3: value IMD HV -> IMD TS
- P4: value HV -> LV Regulator Jumper -> TS -> GLV Regulator Jumper
Connections:
- net labels added: 3.3V_TS, TS+, TS-
- net labels removed: 3.3V_HV, HV+, HV-
Other:
- note added: "TS GLV"
- note removed: "HV LV"
Changed lines of the file:
@@
 LIBS:valves
 LIBS:arduino
-LIBS:AccumulatorBoardHV-cache
 EELAYER 25 0
 EELAYER END
@@
 P 1600 1800
 F 0 "P2" H 1600 1950 50  0000 C CNN
-F 1 "HV (Switched)" V 1700 1800 50  0000 C CNN
+F 1 "TS (Switched)" V 1700 1800 50  0000 C CNN
 F 2 "Connectors_Molex:Molex_MiniFit-JR-5556-02A_2x01x4.20mm_Straight" H 1600 1800 50  0001 C CNN
 F 3 "" H 1600 1800 50  0000 C CNN
@@
 $EndComp
 Text Label 1800 1800 0    60   ~ 0
-HV+
+TS+
 Text Label 1800 1900 0    60   ~ 0
-HV-
+TS-
 Text Label 1800 1250 0    60   ~ 0
 BATT-
@@
 P 2900 1850
 F 0 "P3" H 2900 2000 50  0000 C CNN
-F 1 "IMD HV" V 3000 1850 50  0000 C CNN
+F 1 "IMD TS" V 3000 1850 50  0000 C CNN
 F 2 "Connectors_Molex:Molex_NanoFit_1x02x2.50mm_Straight" H 2900 1850 50  0001 C CNN
 F 3 "" H 2900 1850 50  0000 C CNN
@@
 $EndComp
 Text Label 3550 4250 2    60   ~ 0
-HV-
+TS-
 Text Label 2250 3650 2    60   ~ 0
-HV+
+TS+
 Text Label 5050 3850 0    60   ~ 0
 12V_INDICATOR
@@
 P 2200 950
 F 0 "P4" H 2200 1100 50  0000 C CNN
-F 1 "HV -> LV Regulator Jumper" V 2300 950 50  0000 C CNN
+F 1 "TS -> GLV Regulator Jumper" V 2300 950 50  0000 C CNN
 F 2 "Connectors_Molex:Molex_MiniFit-JR-5556-02A_2x01x4.20mm_Straight" H 2200 950 50  0001 C CNN
 F 3 "" H 2200 950 50  0000 C CNN
@@
 12V_SRC
 Text Notes 4500 7700 0    60   ~ 0
-HV      LV
+TS      GLV
 Text Notes 4500 5550 0    60   ~ 0
-HV      LV
+TS      GLV
 Text Notes 4500 600  0    60   ~ 0
-HV      LV
+TS      GLV
 Text Notes 1950 3350 0    60   ~ 0
 60V Threshold Accumulator Indicators Circuit
@@
 Text Label 5200 2450 0    60   ~ 0
 GND
-$Comp
-L RDD08110S12 DC?
-U 1 1 59C0CBF2
-P 1300 2800
-F 0 "DC?" H 1000 2350 60  0000 L CNN
-F 1 "RDD08110S12" H 1000 3200 60  0000 L CNN
-F 2 "" H 1450 2750 60  0000 C CNN
-F 3 "" H 1450 2750 60  0000 C CNN
-	1    1300 2800
-	1    0    0    -1
-$EndComp
 NoConn ~ 800  2750
 Text Label 800  3050 2    60   ~ 0
@@
 $Comp
 L CP C?
-U 1 1 59C0ECA6
-P 2150 2900
-F 0 "C?" H 2175 3000 50  0000 L CNN
-F 1 "CP" H 2175 2800 50  0000 L CNN
-F 2 "" H 2188 2750 50  0001 C CNN
-F 3 "" H 2150 2900 50  0001 C CNN
-	1    2150 2900
-	1    0    0    -1
-$EndComp
-$Comp
-L LD1117V33 U?
-U 1 1 59C0ED27
-P 2550 2800
-F 0 "U?" H 2350 3000 50  0000 C CNN
-F 1 "LD1117V33" H 2550 3000 50  0000 L CNN
-F 2 "TO-220" H 2550 2450 50  0001 C CIN
-F 3 "" H 2550 2800 50  0000 C CNN
-	1    2550 2800
-	1    0    0    -1
-$EndComp
-$Comp
-L CP C?
 U 1 1 59C0EDAC
 P 2950 2900
@@
 Wire Wire Line
 	1800 3050 3800 3050
-Connection ~ 2550 3050
-Connection ~ 2150 3050
 Wire Wire Line
 	1800 2550 2150 2550
@@
 $EndComp
 Wire Wire Line
-	2950 2750 3150 2750
+	2150 2750 3150 2750
 Wire Wire Line
 	3450 2750 3800 2750
 Text Label 3450 2750 0    60   ~ 0
-3.3V_HV
+3.3V_TS
 Wire Notes Line
 	4750 7700 4750 500
 Connection ~ 2100 2100
 Connection ~ 2500 2100
+Connection ~ 2950 2750
+$Comp
+L RDD08110S3V3 U?
+U 1 1 5A3F2C66
+P 1300 2800
+F 0 "U?" H 1000 2400 60  0000 L CNN
+F 1 "RDD08110S3V3" H 1000 3200 60  0000 L CNN
+F 2 "" H 1450 2750 60  0000 C CNN
+F 3 "" H 1450 2750 60  0000 C CNN
+	1    1300 2800
+	1    0    0    -1
+$EndComp
 $EndSCHEMATC

Commit message: Reconfigure dash schematic to take advantage of spare pin
Parts:
- removed P?: To Temp Board, symbol Conn_01x02
- added R? (x2): R, symbol R
Connections:
- wire segments 58 -> 62
Other:
- moved on the sheet: D?, F?, R?

Commit message: Added charger control pins and organized optos
Parts:
- removed J?: To LV Board, symbol Conn_01x04
- removed U? (x2): DK1A1B-12V, symbol DK1A1B-12V
- removed U?: PS2501-4, symbol PS2501-4
- added J?: To LV Board, symbol Conn_01x04
- added U?: PS2501-4-1, symbol PS2501-4-1
- added U? (x2): G2RL-1A-E, symbol G2RL-1A-E
Connections:
- wire segments 62 -> 60
Changed lines of the file:
@@
 	1    0    0    -1
 $EndComp
-$Comp
-L DK1A1B-12V U?
-U 1 1 5959B6E5
-P 4650 6150
-F 0 "U?" H 4550 6150 60  0000 C CNN
-F 1 "DK1A1B-12V" V 4900 6150 60  0000 C CNN
-F 2 "" H 4650 6150 60  0000 C CNN
-F 3 "" H 4650 6150 60  0000 C CNN
-	1    4650 6150
-	-1   0    0    -1
-$EndComp
-$Comp
-L DK1A1B-12V U?
-U 1 1 5959B75A
-P 4650 7250
-F 0 "U?" H 4550 7250 60  0000 C CNN
-F 1 "DK1A1B-12V" V 4900 7250 60  0000 C CNN
-F 2 "" H 4650 7250 60  0000 C CNN
-F 3 "" H 4650 7250 60  0000 C CNN
-	1    4650 7250
-	-1   0    0    -1
-$EndComp
-Text Label 5150 6000 0    60   ~ 0
+Text Label 5150 6200 0    60   ~ 0
 AIRS_FINAL_CHARGER
 Text Label 5150 7100 0    60   ~ 0
@@
 L GND #PWR?
 U 1 1 5959BDAF
-P 5150 6300
-F 0 "#PWR?" H 5150 6050 50  0001 C CNN
-F 1 "GND" H 5150 6150 50  0000 C CNN
-F 2 "" H 5150 6300 50  0001 C CNN
-F 3 "" H 5150 6300 50  0001 C CNN
-	1    5150 6300
+P 5150 6500
+F 0 "#PWR?" H 5150 6250 50  0001 C CNN
+F 1 "GND" H 5150 6350 50  0000 C CNN
+F 2 "" H 5150 6500 50  0001 C CNN
+F 3 "" H 5150 6500 50  0001 C CNN
+	1    5150 6500
 	1    0    0    -1
 $EndComp
@@
 L Conn_01x02 J?
 U 1 1 5959BFDF
-P 2900 6450
-F 0 "J?" H 2900 6600 50  0000 C CNN
-F 1 "Charger Current" V 3000 6450 50  0000 C CNN
-F 2 "" H 2900 6450 50  0001 C CNN
-F 3 "" H 2900 6450 50  0001 C CNN
-	1    2900 6450
+P 2900 6650
+F 0 "J?" H 2900 6800 50  0000 C CNN
+F 1 "Charger Current" V 3000 6650 50  0000 C CNN
+F 2 "" H 2900 6650 50  0001 C CNN
+F 3 "" H 2900 6650 50  0001 C CNN
+	1    2900 6650
 	-1   0    0    -1
 $EndComp
-Text Label 3100 6450 0    60   ~ 0
+Text Label 3100 6650 0    60   ~ 0
 CHARGER+
-Text Label 3100 6550 0    60   ~ 0
+Text Label 3100 6750 0    60   ~ 0
 CHARGER-
-Text Label 4650 5850 1    60   ~ 0
+Text Label 4650 6050 1    60   ~ 0
 BATT+
 Text Label 4650 6950 1    60   ~ 0
@@
 Text Notes 4500 7700 0    60   ~ 0
 TS      GLV
-Text Notes 4500 5550 0    60   ~ 0
+Text Notes 4500 5250 0    60   ~ 0
 TS      GLV
 Text Notes 4500 600  0    60   ~ 0
@@
 F 3 "" H 5050 800 50  0000 C CNN
 	1    5050 800
-	1    0    0    -1
-$EndComp
-$Comp
-L PS2501-4 U?
-U 1 1 59A394ED
-P 4750 4300
-F 0 "U?" H 5050 4300 60  0000 C CNN
-F 1 "PS2501-4" H 4650 4300 60  0000 C CNN
-F 2 "" H 4750 4300 60  0000 C CNN
-F 3 "" H 4750 4300 60  0000 C CNN
-	1    4750 4300
 	1    0    0    -1
 $EndComp
@@
 Text Label 5050 4600 0    60   ~ 0
 12V_INDICATOR
-$Comp
-L Conn_01x04 J?
-U 1 1 59C0BC37
-P 6400 1050
-F 0 "J?" H 6400 1250 50  0000 C CNN
-F 1 "To LV Board" H 6400 750 50  0000 C CNN
-F 2 "" H 6400 1050 50  0001 C CNN
-F 3 "" H 6400 1050 50  0001 C CNN
-	1    6400 1050
-	-1   0    0    -1
-$EndComp
 Text Label 6600 1050 0    60   ~ 0
 12V
@@
 Connection ~ 3650 3950
 Wire Wire Line
-	3100 6550 3100 7600
-Wire Wire Line
-	3100 7600 4650 7600
-Wire Wire Line
-	4650 7600 4650 7550
-Wire Wire Line
-	3100 6450 4050 6450
-Wire Wire Line
-	4050 6450 4050 6550
-Wire Wire Line
-	4050 6550 4650 6550
-Wire Wire Line
-	4650 6550 4650 6450
+	3100 6650 4650 6650
 Wire Wire Line
 	2900 1650 2900 1150
@@
 	4150 4000 4450 4000
 Wire Notes Line
-	1700 3250 1700 5450
-Wire Notes Line
-	1700 5450 7200 5450
-Wire Notes Line
-	7200 5450 7200 3250
+	1700 5150 7200 5150
 Wire Wire Line
 	1800 1150 2200 1150
@@
 	3450 2750 3800 2750
 Wire Notes Line
-	4750 7700 4750 500
+	4750 7750 4750 550
 Connection ~ 2100 2100
 Connection ~ 2500 2100
@@
 	4350 4600 4350 4950
 Connection ~ 4350 4950
+$Comp
+L G2RL-1A-E U?
+U 1 1 5A5D3039
+P 4650 6350
+F 0 "U?" H 4550 6350 60  0000 C CNN
+F 1 "G2RL-1A-E" V 4900 6350 60  0000 C CNN
+F 2 "" H 4650 6350 60  0000 C CNN
+F 3 "" H 4650 6350 60  0000 C CNN
+	1    4650 6350
+	-1   0    0    -1
+$EndComp
+$Comp
+L G2RL-1A-E U?
+U 1 1 5A5D341A
+P 4650 7250
+F 0 "U?" H 4550 7250 60  0000 C CNN
+F 1 "G2RL-1A-E" V 4900 7250 60  0000 C CNN
+F 2 "" H 4650 7250 60  0000 C CNN
+F 3 "" H 4650 7250 60  0000 C CNN
+	1    4650 7250
+	-1   0    0    -1
+$EndComp
+Wire Wire Line
+	4650 6950 4550 6950
+Wire Wire Line
+	4550 6050 4650 6050
+Connection ~ 4550 7550
+Connection ~ 4550 6650
+Wire Notes Line
+	7200 5150 7200 3250
+Wire Notes Line
+	1700 3250 1700 5150
+Wire Wire Line
+	3100 6750 3100 7550
+Wire Wire Line
+	3100 7550 4650 7550
+$Comp
+L PS2501-4-1 U?
+U 1 1 5A5D2C74
+P 4750 4300
+F 0 "U?" H 4550 5050 50  0000 L CNN
+F 1 "PS2501-4-1" H 4550 3550 50  0000 L CNN
+F 2 "" H 4550 4650 50  0000 L CIN
+F 3 "" H 4750 4850 50  0000 L CNN
+	1    4750 4300
+	1    0    0    -1
+$EndComp
+$Comp
+L Conn_01x04 J?
+U 1 1 5A5D61FA
+P 6400 1050
+F 0 "J?" H 6400 1250 50  0000 C CNN
+F 1 "To LV Board" H 6400 750 50  0000 C CNN
+F 2 "" H 6400 1050 50  0001 C CNN
+F 3 "" H 6400 1050 50  0001 C CNN
+	1    6400 1050
+	-1   0    0    -1
+$EndComp
 $EndSCHEMATC

Commit message: Set footprints for Accumulator HV board, creating necessary ones
Parts:
- F1: renamed from F3; footprint (none) -> fs-1-schematics:SMD Fuse
- F3, F5: renamed from F?; footprint (none) -> fs-1-schematics:SMD Fuse
- F4: renamed from F2; footprint (none) -> fs-1-schematics:SMD Fuse
- J2: renamed from J?; footprint (none) -> Connectors_Molex:Molex_NanoFit_1x04x2.50mm_Straight
- J6: renamed from J?; footprint (none) -> Connectors_Molex:Molex_NanoFit_1x02x2.50mm_Straight
- J9: renamed from J?; footprint (none) -> Connectors_Molex:Molex_MiniFit-JR-5556-02A_2x01x4.20mm_Straight
- R1, R2, R3, R5, R6, R7, R8: renamed from R?; footprint (none) -> Resistors_THT:R_Axial_DIN0207_L6.3mm_D2.5mm_P10.16mm_Horizontal
- R4: renamed from R1; footprint (none) -> Resistors_THT:R_Axial_DIN0207_L6.3mm_D2.5mm_P10.16mm_Horizontal
- U2: renamed from U?; footprint (none) -> fs-1-schematics:DK1A1B-12V
- U3: renamed from U?; footprint (none) -> fs-1-schematics:RDD08110S12
- U4: renamed from U?; footprint (none) -> Housings_DIP:DIP-16_W7.62mm
- gave numbers to parts that had none: 10
- renumbered C2 to C1, C1 to C3, C3 to C5, F1 to F2, P4 to J1, P1 to J3, P2 to J4, P3 to J5, P5 to J7, P6 to J8

Commit message: Set footprints for Accumulator LV board, creating necessary ones
Parts:
- U3: footprint fs-1-schematics:RDD08110S12 -> fs-1-schematics:RDD08110S3V3
Changed lines of the file:
@@
 F 0 "U3" H 1000 2400 60  0000 L CNN
 F 1 "RDD08110S3V3" H 1000 3200 60  0000 L CNN
-F 2 "fs-1-schematics:RDD08110S12" H 1450 2750 60  0001 C CNN
+F 2 "fs-1-schematics:RDD08110S3V3" H 1450 2750 60  0001 C CNN
 F 3 "" H 1450 2750 60  0000 C CNN
 	1    1300 2800

Commit message: Begin PE/dash footprints, continue with accumulator footprints
Parts:
- C1, C2, C3, C4, C5, C6, C9: footprint (none) -> Capacitors_THT:CP_Radial_D8.0mm_P2.50mm
- C7, C8: footprint (none) -> Capacitors_THT:CP_Radial_D16.0mm_P7.50mm
- F1, F2, F3, F4, F5: footprint fs-1-schematics:SMD Fuse -> FSFootprints:SMD Fuse
- U1: footprint fs-1-schematics:VICOR-DCDC -> FSFootprints:VICOR-DCDC
- U2: footprint fs-1-schematics:DK1A1B-12V -> FSFootprints:DK1A1B-12V
- U3: footprint fs-1-schematics:RDD08110S3V3 -> FSFootprints:RDD08110S3V3
- U5, U6: footprint (none) -> FSFootprints:G2RL-1A-E
Changed lines of the file:
@@
 F 0 "F2" V 2830 1150 50  0000 C CNN
 F 1 "IMD/DCDC Fuse" V 2675 1150 50  0000 C CNN
-F 2 "fs-1-schematics:SMD Fuse" V 2680 1150 50  0001 C CNN
+F 2 "FSFootprints:SMD Fuse" V 2680 1150 50  0001 C CNN
 F 3 "" H 2750 1150 50  0000 C CNN
 	1    2750 1150
@@
 F 0 "C3" H 3375 1400 50  0000 L CNN
 F 1 "0.47uF" H 3375 1200 50  0000 L CNN
-F 2 "" H 3388 1150 50  0001 C CNN
+F 2 "Capacitors_THT:CP_Radial_D8.0mm_P2.50mm" H 3388 1150 50  0001 C CNN
 F 3 "" H 3350 1300 50  0000 C CNN
 	1    3350 1300
@@
 F 0 "U1" H 4550 1500 60  0000 C CNN
 F 1 "V110C12E100BL" H 4550 1650 60  0000 C CNN
-F 2 "fs-1-schematics:VICOR-DCDC" H 4550 1200 60  0001 C CNN
+F 2 "FSFootprints:VICOR-DCDC" H 4550 1200 60  0001 C CNN
 F 3 "" H 4550 1200 60  0001 C CNN
 	1    4550 1200
@@
 F 0 "C5" H 4075 1700 50  0000 L CNN
 F 1 "C" H 4075 1500 50  0000 L CNN
-F 2 "" H 4088 1450 50  0001 C CNN
+F 2 "Capacitors_THT:CP_Radial_D8.0mm_P2.50mm" H 4088 1450 50  0001 C CNN
 F 3 "" H 4050 1600 50  0000 C CNN
 	1    4050 1600
@@
 F 0 "C1" H 4075 900 50  0000 L CNN
 F 1 "C" H 4075 700 50  0000 L CNN
-F 2 "" H 4088 650 50  0001 C CNN
+F 2 "Capacitors_THT:CP_Radial_D8.0mm_P2.50mm" H 4088 650 50  0001 C CNN
 F 3 "" H 4050 800 50  0000 C CNN
 	1    4050 800
@@
 F 0 "F1" V 5530 950 50  0000 C CNN
 F 1 "Fuse" V 5375 950 50  0000 C CNN
-F 2 "fs-1-schematics:SMD Fuse" V 5380 950 50  0001 C CNN
+F 2 "FSFootprints:SMD Fuse" V 5380 950 50  0001 C CNN
 F 3 "" H 5450 950 50  0000 C CNN
 	1    5450 950
@@
 F 0 "F4" V 2480 3650 50  0000 C CNN
 F 1 "Fuse" V 2325 3650 50  0000 C CNN
-F 2 "fs-1-schematics:SMD Fuse" V 2330 3650 50  0001 C CNN
+F 2 "FSFootprints:SMD Fuse" V 2330 3650 50  0001 C CNN
 F 3 "" H 2400 3650 50  0000 C CNN
 	1    2400 3650
@@
 F 0 "C4" H 5625 1400 50  0000 L CNN
 F 1 "CP" H 5625 1200 50  0000 L CNN
-F 2 "" H 5638 1150 50  0001 C CNN
+F 2 "Capacitors_THT:CP_Radial_D8.0mm_P2.50mm" H 5638 1150 50  0001 C CNN
 F 3 "" H 5600 1300 50  0000 C CNN
 	1    5600 1300
@@
 F 0 "C6" H 5075 1700 50  0000 L CNN
 F 1 "C" H 5075 1500 50  0000 L CNN
-F 2 "" H 5088 1450 50  0001 C CNN
+F 2 "Capacitors_THT:CP_Radial_D8.0mm_P2.50mm" H 5088 1450 50  0001 C CNN
 F 3 "" H 5050 1600 50  0000 C CNN
 	1    5050 1600
@@
 F 0 "C2" H 5075 900 50  0000 L CNN
 F 1 "C" H 5075 700 50  0000 L CNN
-F 2 "" H 5088 650 50  0001 C CNN
+F 2 "Capacitors_THT:CP_Radial_D8.0mm_P2.50mm" H 5088 650 50  0001 C CNN
 F 3 "" H 5050 800 50  0000 C CNN
 	1    5050 800
@@
 F 0 "F5" V 2480 4500 50  0000 C CNN
 F 1 "Fuse" V 2325 4500 50  0000 C CNN
-F 2 "fs-1-schematics:SMD Fuse" V 2330 4500 50  0001 C CNN
+F 2 "FSFootprints:SMD Fuse" V 2330 4500 50  0001 C CNN
 F 3 "" H 2400 4500 50  0000 C CNN
 	1    2400 4500
@@
 F 0 "U2" H 4600 2300 60  0000 C CNN
 F 1 "DK1A1B-12V" V 4950 2300 60  0000 C CNN
-F 2 "fs-1-schematics:DK1A1B-12V" H 4700 2300 60  0001 C CNN
+F 2 "FSFootprints:DK1A1B-12V" H 4700 2300 60  0001 C CNN
 F 3 "" H 4700 2300 60  0000 C CNN
 	1    4700 2300
@@
 F 0 "C7" H 2125 2350 50  0000 L CNN
 F 1 "100uF" H 2125 2150 50  0000 L CNN
-F 2 "" H 2138 2100 50  0001 C CNN
+F 2 "Capacitors_THT:CP_Radial_D16.0mm_P7.50mm" H 2138 2100 50  0001 C CNN
 F 3 "" H 2100 2250 50  0001 C CNN
 	1    2100 2250
@@
 F 0 "C8" H 2525 2350 50  0000 L CNN
 F 1 "100uF" H 2525 2150 50  0000 L CNN
-F 2 "" H 2538 2100 50  0001 C CNN
+F 2 "Capacitors_THT:CP_Radial_D16.0mm_P7.50mm" H 2538 2100 50  0001 C CNN
 F 3 "" H 2500 2250 50  0001 C CNN
 	1    2500 2250
@@
 F 0 "C9" H 2975 3000 50  0000 L CNN
 F 1 "CP" H 2975 2800 50  0000 L CNN
-F 2 "" H 2988 2750 50  0001 C CNN
+F 2 "Capacitors_THT:CP_Radial_D8.0mm_P2.50mm" H 2988 2750 50  0001 C CNN
 F 3 "" H 2950 2900 50  0001 C CNN
 	1    2950 2900
@@
 F 0 "F3" V 3380 2750 50  0000 C CNN
 F 1 "Fuse" V 3225 2750 50  0000 C CNN
-F 2 "fs-1-schematics:SMD Fuse" V 3230 2750 50  0001 C CNN
+F 2 "FSFootprints:SMD Fuse" V 3230 2750 50  0001 C CNN
 F 3 "" H 3300 2750 50  0001 C CNN
 	1    3300 2750
@@
 F 0 "U3" H 1000 2400 60  0000 L CNN
 F 1 "RDD08110S3V3" H 1000 3200 60  0000 L CNN
-F 2 "fs-1-schematics:RDD08110S3V3" H 1450 2750 60  0001 C CNN
+F 2 "FSFootprints:RDD08110S3V3" H 1450 2750 60  0001 C CNN
 F 3 "" H 1450 2750 60  0000 C CNN
 	1    1300 2800
@@
 F 0 "U5" H 4550 6350 60  0000 C CNN
 F 1 "G2RL-1A-E" V 4900 6350 60  0000 C CNN
-F 2 "" H 4650 6350 60  0001 C CNN
+F 2 "FSFootprints:G2RL-1A-E" H 4650 6350 60  0001 C CNN
 F 3 "" H 4650 6350 60  0000 C CNN
 	1    4650 6350
@@
 F 0 "U6" H 4550 7250 60  0000 C CNN
 F 1 "G2RL-1A-E" V 4900 7250 60  0000 C CNN
-F 2 "" H 4650 7250 60  0001 C CNN
+F 2 "FSFootprints:G2RL-1A-E" H 4650 7250 60  0001 C CNN
 F 3 "" H 4650 7250 60  0000 C CNN
 	1    4650 7250

Commit message: Begin layout of AccumulatorHV board
Parts:
- removed U4: PS2501-4-1, Housings_DIP:DIP-16_W7.62mm, symbol PS2501-4-1
- added F6: Fuse, FSFootprints:SMD Fuse, symbol Fuse
- added U4: PS2501-4, symbol PS2501-4
- C1, C2, C5, C6: footprint Capacitors_THT:CP_Radial_D8.0mm_P2.50mm -> Capacitors_THT:C_Disc_D4.7mm_W2.5mm_P5.00mm
- F4: value Fuse -> TS 60V Fuse
- F5: value Fuse -> Charger 60V Fuse
- J4: footprint Connectors_Molex:Molex_MiniFit-JR-5556-02A_2x01x4.20mm_Straight -> Connectors_Molex:Molex_NanoFit_1x02x2.50mm_Straight
Connections:
- net labels added: BATT+_DIRECT, BATT+_LVBOARD
Changed lines of the file:
@@
 L Conn_01x02 J4
 U 1 1 589D2B01
-P 1600 1800
-F 0 "J4" H 1600 1950 50  0000 C CNN
-F 1 "TS (Switched)" V 1700 1800 50  0000 C CNN
-F 2 "Connectors_Molex:Molex_MiniFit-JR-5556-02A_2x01x4.20mm_Straight" H 1600 1800 50  0001 C CNN
-F 3 "" H 1600 1800 50  0000 C CNN
-	1    1600 1800
+P 1150 1800
+F 0 "J4" H 1150 1950 50  0000 C CNN
+F 1 "TS (Switched)" V 1250 1800 50  0000 C CNN
+F 2 "Connectors_Molex:Molex_NanoFit_1x02x2.50mm_Straight" H 1150 1800 50  0001 C CNN
+F 3 "" H 1150 1800 50  0000 C CNN
+	1    1150 1800
 	-1   0    0    -1
 $EndComp
@@
 L Conn_01x02 J3
 U 1 1 589D2D5E
-P 1600 1150
-F 0 "J3" H 1600 1300 50  0000 C CNN
-F 1 "Batt Voltage" V 1700 1150 50  0000 C CNN
-F 2 "Connectors_Molex:Molex_MiniFit-JR-5556-02A_2x01x4.20mm_Straight" H 1600 1150 50  0001 C CNN
-F 3 "" H 1600 1150 50  0000 C CNN
-	1    1600 1150
-	-1   0    0    -1
-$EndComp
-Text Label 1800 1800 0    60   ~ 0
+P 1150 1150
+F 0 "J3" H 1150 1300 50  0000 C CNN
+F 1 "Batt Voltage" V 1250 1150 50  0000 C CNN
+F 2 "Connectors_Molex:Molex_MiniFit-JR-5556-02A_2x01x4.20mm_Straight" H 1150 1150 50  0001 C CNN
+F 3 "" H 1150 1150 50  0000 C CNN
+	1    1150 1150
+	-1   0    0    -1
+$EndComp
+Text Label 1350 1800 0    60   ~ 0
 TS+
-Text Label 1800 1900 0    60   ~ 0
+Text Label 1350 1900 0    60   ~ 0
 TS-
-Text Label 1800 1250 0    60   ~ 0
+Text Label 1350 1250 0    60   ~ 0
 BATT-
 $Comp
@@
 Text Label 3550 4250 2    60   ~ 0
 TS-
-Text Label 2250 3650 2    60   ~ 0
+Text Label 2250 3650 3    60   ~ 0
 TS+
 Text Label 5050 3850 0    60   ~ 0
@@
 F 0 "C5" H 4075 1700 50  0000 L CNN
 F 1 "C" H 4075 1500 50  0000 L CNN
-F 2 "Capacitors_THT:CP_Radial_D8.0mm_P2.50mm" H 4088 1450 50  0001 C CNN
+F 2 "Capacitors_THT:C_Disc_D4.7mm_W2.5mm_P5.00mm" H 4088 1450 50  0001 C CNN
 F 3 "" H 4050 1600 50  0000 C CNN
 	1    4050 1600
@@
 F 0 "C1" H 4075 900 50  0000 L CNN
 F 1 "C" H 4075 700 50  0000 L CNN
-F 2 "Capacitors_THT:CP_Radial_D8.0mm_P2.50mm" H 4088 650 50  0001 C CNN
+F 2 "Capacitors_THT:C_Disc_D4.7mm_W2.5mm_P5.00mm" H 4088 650 50  0001 C CNN
 F 3 "" H 4050 800 50  0000 C CNN
 	1    4050 800
@@
 GND
 $Comp
-L GND #PWR01
+L GND #PWR1
 U 1 1 58B2C1BD
 P 5350 1450
-F 0 "#PWR01" H 5350 1200 50  0001 C CNN
+F 0 "#PWR1" H 5350 1200 50  0001 C CNN
 F 1 "GND" H 5350 1300 50  0000 C CNN
 F 2 "" H 5350 1450 50  0000 C CNN
@@
 P 2400 3650
 F 0 "F4" V 2480 3650 50  0000 C CNN
-F 1 "Fuse" V 2325 3650 50  0000 C CNN
+F 1 "TS 60V Fuse" V 2325 3650 50  0000 C CNN
 F 2 "FSFootprints:SMD Fuse" V 2330 3650 50  0001 C CNN
 F 3 "" H 2400 3650 50  0000 C CNN
@@
 AIRS_FINAL_CHARGER
 $Comp
-L GND #PWR02
+L GND #PWR2
 U 1 1 5959BDAF
 P 5150 6500
-F 0 "#PWR02" H 5150 6250 50  0001 C CNN
+F 0 "#PWR2" H 5150 6250 50  0001 C CNN
 F 1 "GND" H 5150 6350 50  0000 C CNN
 F 2 "" H 5150 6500 50  0001 C CNN
@@
 $EndComp
 $Comp
-L GND #PWR03
+L GND #PWR3
 U 1 1 5959BDF7
 P 5150 7400
-F 0 "#PWR03" H 5150 7150 50  0001 C CNN
+F 0 "#PWR3" H 5150 7150 50  0001 C CNN
 F 1 "GND" H 5150 7250 50  0000 C CNN
 F 2 "" H 5150 7400 50  0001 C CNN
@@
 Text Label 3100 6750 0    60   ~ 0
 CHARGER-
-Text Label 4650 6050 1    60   ~ 0
-BATT+
+Text Label 4550 5750 2    60   ~ 0
+BATT+_DIRECT
 Text Label 4650 6950 1    60   ~ 0
 BATT-
@@
 F 0 "C6" H 5075 1700 50  0000 L CNN
 F 1 "C" H 5075 1500 50  0000 L CNN
-F 2 "Capacitors_THT:CP_Radial_D8.0mm_P2.50mm" H 5088 1450 50  0001 C CNN
+F 2 "Capacitors_THT:C_Disc_D4.7mm_W2.5mm_P5.00mm" H 5088 1450 50  0001 C CNN
 F 3 "" H 5050 1600 50  0000 C CNN
 	1    5050 1600
@@
 F 0 "C2" H 5075 900 50  0000 L CNN
 F 1 "C" H 5075 700 50  0000 L CNN
-F 2 "Capacitors_THT:CP_Radial_D8.0mm_P2.50mm" H 5088 650 50  0001 C CNN
+F 2 "Capacitors_THT:C_Disc_D4.7mm_W2.5mm_P5.00mm" H 5088 650 50  0001 C CNN
 F 3 "" H 5050 800 50  0000 C CNN
 	1    5050 800
@@
 Text Label 3550 5100 2    60   ~ 0
 CHARGER-
-Text Label 2250 4500 2    60   ~ 0
+Text Label 2250 4500 3    60   ~ 0
 CHARGER+
 Text Label 5050 4950 0    60   ~ 0
@@
 P 2400 4500
 F 0 "F5" V 2480 4500 50  0000 C CNN
-F 1 "Fuse" V 2325 4500 50  0000 C CNN
+F 1 "Charger 60V Fuse" V 2325 4500 50  0000 C CNN
 F 2 "FSFootprints:SMD Fuse" V 2330 4500 50  0001 C CNN
 F 3 "" H 2400 4500 50  0000 C CNN
@@
 	1700 5150 7200 5150
 Wire Wire Line
-	1800 1150 2200 1150
+	1350 1150 2200 1150
 Wire Wire Line
 	2300 1150 2600 1150
@@
 	3100 7550 4650 7550
 $Comp
-L PS2501-4-1 U4
-U 1 1 5A5D2C74
-P 4750 4300
-F 0 "U4" H 4550 5050 50  0000 L CNN
-F 1 "PS2501-4-1" H 4550 3550 50  0000 L CNN
-F 2 "Housings_DIP:DIP-16_W7.62mm" H 4550 4650 50  0001 L CIN
-F 3 "" H 4750 4850 50  0000 L CNN
-	1    4750 4300
-	1    0    0    -1
-$EndComp
-$Comp
 L Conn_01x04 J2
 U 1 1 5A5D61FA
@@
 	-1   0    0    -1
 $EndComp
+Text Label 1350 1150 0    60   ~ 0
+BATT+_DIRECT
+$Comp
+L Fuse F6
+U 1 1 5A78EF5F
+P 4550 5900
+F 0 "F6" V 4630 5900 50  0000 C CNN
+F 1 "Fuse" V 4475 5900 50  0000 C CNN
+F 2 "FSFootprints:SMD Fuse" V 4480 5900 50  0001 C CNN
+F 3 "" H 4550 5900 50  0001 C CNN
+	1    4550 5900
+	1    0    0    -1
+$EndComp
+Text Label 3550 2100 0    60   ~ 0
+BATT+_LVBOARD
+$Comp
+L PS2501-4 U4
+U 1 1 5A7B8267
+P 4750 4500
+F 0 "U4" H 4550 4700 50  0000 L CNN
+F 1 "PS2501-4" H 4550 4300 50  0000 L CNN
+F 2 "" H 4550 4300 50  0000 L CIN
+F 3 "" H 4750 4500 50  0000 L CNN
+	1    4750 4500
+	1    0    0    -1
+$EndComp
+$Comp
+L PS2501-4 U4
+U 2 1 5A7B8465
+P 4750 4850
+F 0 "U4" H 4550 5050 50  0000 L CNN
+F 1 "PS2501-4" H 4550 4650 50  0000 L CNN
+F 2 "" H 4550 4650 50  0000 L CIN
+F 3 "" H 4750 4850 50  0000 L CNN
+	2    4750 4850
+	1    0    0    -1
+$EndComp
+$Comp
+L PS2501-4 U4
+U 3 1 5A7B87CB
+P 4750 3750
+F 0 "U4" H 4550 3950 50  0000 L CNN
+F 1 "PS2501-4" H 4550 3550 50  0000 L CNN
+F 2 "" H 4550 3550 50  0000 L CIN
+F 3 "" H 4750 3750 50  0000 L CNN
+	3    4750 3750
+	1    0    0    -1
+$EndComp
+$Comp
+L PS2501-4 U4
+U 4 1 5A7B8868
+P 4750 4100
+F 0 "U4" H 4550 4300 50  0000 L CNN
+F 1 "PS2501-4" H 4550 3900 50  0000 L CNN
+F 2 "" H 4550 3900 50  0000 L CIN
+F 3 "" H 4750 4100 50  0000 L CNN
+	4    4750 4100
+	1    0    0    -1
+$EndComp
 $EndSCHEMATC
