File: AccumulatorBoardHV/AccumulatorBoardHV.sch (KiCad schematic (older format))
At the start: 42 parts, among them J1 TS -> GLV Regulator Jumper, J2 To LV Board, J3 Batt Voltage, J4 TS (Switched), J5 IMD TS, J6 To LV Board, J7 Acc LED 1, J8 Acc LED 2, J9 Charger Current, U1 V110C12E100BL, U2 DK1A1B-12V, U3 RDD08110S3V3, U4 PS2501-4, U5 G2RL-1A-E, U6 G2RL-1A-E

Commit message: Work for preparation for autorouting
Parts:
- added J9: Charger Current to Batt, Connectors_Molex:Molex_MiniFit-JR-5556-02A_2x01x4.20mm_Straight, symbol Conn_01x02
- added R9: 0, Resistors_THT:R_Axial_DIN0204_L3.6mm_D1.6mm_P1.90mm_Vertical, symbol R
- U4: footprint (none) -> Housings_DIP:DIP-16_W7.62mm
- renumbered J9 to J10
Connections:
- net labels added: BATT+_CHARGER, BATT+_CHGFUSED, BATT-_CHARGER
- wire segments 60 -> 61
Other:
- moved on the sheet: F6
Changed lines of the file:
@@
 GND
 $Comp
-L GND #PWR1
+L GND #PWR01
 U 1 1 58B2C1BD
 P 5350 1450
-F 0 "#PWR1" H 5350 1200 50  0001 C CNN
+F 0 "#PWR01" H 5350 1200 50  0001 C CNN
 F 1 "GND" H 5350 1300 50  0000 C CNN
 F 2 "" H 5350 1450 50  0000 C CNN
@@
 AIRS_FINAL_CHARGER
 $Comp
-L GND #PWR2
+L GND #PWR02
 U 1 1 5959BDAF
 P 5150 6500
-F 0 "#PWR2" H 5150 6250 50  0001 C CNN
+F 0 "#PWR02" H 5150 6250 50  0001 C CNN
 F 1 "GND" H 5150 6350 50  0000 C CNN
 F 2 "" H 5150 6500 50  0001 C CNN
@@
 $EndComp
 $Comp
-L GND #PWR3
+L GND #PWR03
 U 1 1 5959BDF7
 P 5150 7400
-F 0 "#PWR3" H 5150 7150 50  0001 C CNN
+F 0 "#PWR03" H 5150 7150 50  0001 C CNN
 F 1 "GND" H 5150 7250 50  0000 C CNN
 F 2 "" H 5150 7400 50  0001 C CNN
@@
 $EndComp
 $Comp
-L Conn_01x02 J9
+L Conn_01x02 J10
 U 1 1 5959BFDF
 P 2900 6650
-F 0 "J9" H 2900 6800 50  0000 C CNN
+F 0 "J10" H 2900 6800 50  0000 C CNN
 F 1 "Charger Current" V 3000 6650 50  0000 C CNN
 F 2 "Connectors_Molex:Molex_MiniFit-JR-5556-02A_2x01x4.20mm_Straight" H 2900 6650 50  0001 C CNN
@@
 Text Label 3100 6750 0    60   ~ 0
 CHARGER-
-Text Label 4550 5750 2    60   ~ 0
-BATT+_DIRECT
-Text Label 4650 6950 1    60   ~ 0
-BATT-
+Text Label 4250 5950 2    60   ~ 0
+BATT+_CHARGER
+Text Label 4650 6950 2    60   ~ 0
+BATT-_CHARGER
 $Comp
 L R R2
@@
 	1    0    0    -1
 $EndComp
-Text Label 3550 5100 2    60   ~ 0
+Text Label 3250 5100 2    60   ~ 0
 CHARGER-
 Text Label 2250 4500 3    60   ~ 0
@@
 L Fuse F6
 U 1 1 5A78EF5F
-P 4550 5900
-F 0 "F6" V 4630 5900 50  0000 C CNN
-F 1 "Fuse" V 4475 5900 50  0000 C CNN
-F 2 "FSFootprints:SMD Fuse" V 4480 5900 50  0001 C CNN
-F 3 "" H 4550 5900 50  0001 C CNN
-	1    4550 5900
-	1    0    0    -1
+P 4400 5950
+F 0 "F6" V 4480 5950 50  0000 C CNN
+F 1 "Fuse" V 4325 5950 50  0000 C CNN
+F 2 "FSFootprints:SMD Fuse" V 4330 5950 50  0001 C CNN
+F 3 "" H 4400 5950 50  0001 C CNN
+	1    4400 5950
+	0    -1   -1   0
 $EndComp
 Text Label 3550 2100 0    60   ~ 0
@@
 F 0 "U4" H 4550 4700 50  0000 L CNN
 F 1 "PS2501-4" H 4550 4300 50  0000 L CNN
-F 2 "" H 4550 4300 50  0000 L CIN
+F 2 "Housings_DIP:DIP-16_W7.62mm" H 4550 4300 50  0001 L CIN
 F 3 "" H 4750 4500 50  0000 L CNN
 	1    4750 4500
@@
 F 0 "U4" H 4550 5050 50  0000 L CNN
 F 1 "PS2501-4" H 4550 4650 50  0000 L CNN
-F 2 "" H 4550 4650 50  0000 L CIN
+F 2 "Housings_DIP:DIP-16_W7.62mm" H 4550 4650 50  0001 L CIN
 F 3 "" H 4750 4850 50  0000 L CNN
 	2    4750 4850
@@
 F 0 "U4" H 4550 3950 50  0000 L CNN
 F 1 "PS2501-4" H 4550 3550 50  0000 L CNN
-F 2 "" H 4550 3550 50  0000 L CIN
+F 2 "Housings_DIP:DIP-16_W7.62mm" H 4550 3550 50  0001 L CIN
 F 3 "" H 4750 3750 50  0000 L CNN
 	3    4750 3750
@@
 F 0 "U4" H 4550 4300 50  0000 L CNN
 F 1 "PS2501-4" H 4550 3900 50  0000 L CNN
-F 2 "" H 4550 3900 50  0000 L CIN
+F 2 "Housings_DIP:DIP-16_W7.62mm" H 4550 3900 50  0001 L CIN
 F 3 "" H 4750 4100 50  0000 L CNN
 	4    4750 4100
 	1    0    0    -1
 $EndComp
+Wire Wire Line
+	4550 6050 4550 5950
+$Comp
+L Conn_01x02 J9
+U 1 1 5A81246B
+P 2200 5800
+F 0 "J9" H 2200 5900 50  0000 C CNN
+F 1 "Charger Current to Batt" V 2300 5800 50  0000 C CNN
+F 2 "Connectors_Molex:Molex_MiniFit-JR-5556-02A_2x01x4.20mm_Straight" H 2200 5800 50  0001 C CNN
+F 3 "" H 2200 5800 50  0001 C CNN
+	1    2200 5800
+	-1   0    0    -1
+$EndComp
+Text Label 2400 5800 0    60   ~ 0
+BATT+_CHARGER
+Text Label 2400 5900 0    60   ~ 0
+BATT-_CHARGER
+Text Label 4650 6050 1    60   ~ 0
+BATT+_CHGFUSED
+$Comp
+L R R9
+U 1 1 5A81592B
+P 3400 5100
+F 0 "R9" V 3480 5100 50  0000 C CNN
+F 1 "0" V 3400 5100 50  0000 C CNN
+F 2 "Resistors_THT:R_Axial_DIN0204_L3.6mm_D1.6mm_P1.90mm_Vertical" V 3330 5100 50  0001 C CNN
+F 3 "" H 3400 5100 50  0001 C CNN
+	1    3400 5100
+	0    1    1    0
+$EndComp
 $EndSCHEMATC
