File: AccumulatorBoardHV/AccumulatorBoardHV.sch (KiCad schematic (older format))
At the start: 44 parts, among them J1 TS -> GLV Regulator Jumper, J10 Charger Current, J2 To LV Board, J3 Batt Voltage, J4 TS (Switched), J5 IMD TS, J6 To LV Board, J7 Acc LED 1, J8 Acc LED 2, J9 Charger Current to Batt, U1 V110C12E100BL, U2 DK1A1B-12V, U3 RDD08110S3V3, U4 PS2501-4, U5 G2RL-1A-E, U6 G2RL-1A-E

Commit message: Autoroute AccumulatorHV PCB
Connections:
- net labels added: BATT+_DIRFUSED
Changed lines of the file:
@@
 	0    1    1    0
 $EndComp
+Text Label 2300 1150 3    60   ~ 0
+BATT+_DIRFUSED
 $EndSCHEMATC

Commit message: Tweak AccumulatorHV PCB
Parts:
- U5, U6: footprint FSFootprints:G2RL-1A-E -> (none)
Connections:
- net labels added: VICOR_OUT
Other:
- moved on the sheet: C4
Changed lines of the file:
@@
 LIBS:valves
 LIBS:arduino
-LIBS:AccumulatorBoardHV-cache
 EELAYER 25 0
 EELAYER END
@@
 L GND #PWR01
 U 1 1 58B2C1BD
-P 5350 1450
-F 0 "#PWR01" H 5350 1200 50  0001 C CNN
-F 1 "GND" H 5350 1300 50  0000 C CNN
-F 2 "" H 5350 1450 50  0000 C CNN
-F 3 "" H 5350 1450 50  0000 C CNN
-	1    5350 1450
+P 5300 1450
+F 0 "#PWR01" H 5300 1200 50  0001 C CNN
+F 1 "GND" H 5300 1300 50  0000 C CNN
+F 2 "" H 5300 1450 50  0000 C CNN
+F 3 "" H 5300 1450 50  0000 C CNN
+	1    5300 1450
 	1    0    0    -1
 $EndComp
@@
 L CP C4
 U 1 1 594F0A21
-P 5600 1300
-F 0 "C4" H 5625 1400 50  0000 L CNN
-F 1 "CP" H 5625 1200 50  0000 L CNN
-F 2 "Capacitors_THT:CP_Radial_D8.0mm_P2.50mm" H 5638 1150 50  0001 C CNN
-F 3 "" H 5600 1300 50  0000 C CNN
-	1    5600 1300
+P 5300 1300
+F 0 "C4" H 5325 1400 50  0000 L CNN
+F 1 "CP" H 5325 1200 50  0000 L CNN
+F 2 "Capacitors_THT:CP_Radial_D8.0mm_P2.50mm" H 5338 1150 50  0001 C CNN
+F 3 "" H 5300 1300 50  0000 C CNN
+	1    5300 1300
 	1    0    0    -1
 $EndComp
@@
 	2900 1650 2900 1150
 Wire Wire Line
-	5050 1450 5600 1450
-Connection ~ 5350 1450
-Wire Wire Line
-	5600 950  5600 1150
-Wire Wire Line
 	3150 3650 3000 3650
 Wire Wire Line
@@
 	4350 4600 4350 4950
 Connection ~ 4350 4950
-$Comp
-L G2RL-1A-E U5
-U 1 1 5A5D3039
-P 4650 6350
-F 0 "U5" H 4550 6350 60  0000 C CNN
-F 1 "G2RL-1A-E" V 4900 6350 60  0000 C CNN
-F 2 "FSFootprints:G2RL-1A-E" H 4650 6350 60  0001 C CNN
-F 3 "" H 4650 6350 60  0000 C CNN
-	1    4650 6350
-	-1   0    0    -1
-$EndComp
-$Comp
-L G2RL-1A-E U6
-U 1 1 5A5D341A
-P 4650 7250
-F 0 "U6" H 4550 7250 60  0000 C CNN
-F 1 "G2RL-1A-E" V 4900 7250 60  0000 C CNN
-F 2 "FSFootprints:G2RL-1A-E" H 4650 7250 60  0001 C CNN
-F 3 "" H 4650 7250 60  0000 C CNN
-	1    4650 7250
-	-1   0    0    -1
-$EndComp
 Wire Wire Line
 	4650 6950 4550 6950
@@
 Text Label 2300 1150 3    60   ~ 0
 BATT+_DIRFUSED
+Text Label 5300 950  1    60   ~ 0
+VICOR_OUT
+Wire Wire Line
+	5050 1450 5300 1450
+Wire Wire Line
+	5300 950  5300 1150
+$Comp
+L G2RL-1A-E U5
+U 1 1 5A84B689
+P 4650 6350
+F 0 "U5" H 4550 6350 60  0000 C CNN
+F 1 "G2RL-1A-E" V 4900 6350 60  0000 C CNN
+F 2 "" H 4650 6350 60  0000 C CNN
+F 3 "" H 4650 6350 60  0000 C CNN
+	1    4650 6350
+	-1   0    0    -1
+$EndComp
+$Comp
+L G2RL-1A-E U6
+U 1 1 5A84BA1C
+P 4650 7250
+F 0 "U6" H 4550 7250 60  0000 C CNN
+F 1 "G2RL-1A-E" V 4900 7250 60  0000 C CNN
+F 2 "" H 4650 7250 60  0000 C CNN
+F 3 "" H 4650 7250 60  0000 C CNN
+	1    4650 7250
+	-1   0    0    -1
+$EndComp
 $EndSCHEMATC

Commit message: Add mounting holes to Accumulator HV PCB
Parts:
- added H1, H2, H3, H4: MtngHole, Mounting_Holes:MountingHole_4.5mm, symbol Conn_01x01
- U5, U6: footprint (none) -> FSFootprints:G2RL-1A-E
Changed lines of the file:
@@
 GND
 $Comp
-L GND #PWR01
+L GND #PWR1
 U 1 1 58B2C1BD
 P 5300 1450
-F 0 "#PWR01" H 5300 1200 50  0001 C CNN
+F 0 "#PWR1" H 5300 1200 50  0001 C CNN
 F 1 "GND" H 5300 1300 50  0000 C CNN
 F 2 "" H 5300 1450 50  0000 C CNN
@@
 AIRS_FINAL_CHARGER
 $Comp
-L GND #PWR02
+L GND #PWR2
 U 1 1 5959BDAF
 P 5150 6500
-F 0 "#PWR02" H 5150 6250 50  0001 C CNN
+F 0 "#PWR2" H 5150 6250 50  0001 C CNN
 F 1 "GND" H 5150 6350 50  0000 C CNN
 F 2 "" H 5150 6500 50  0001 C CNN
@@
 $EndComp
 $Comp
-L GND #PWR03
+L GND #PWR3
 U 1 1 5959BDF7
 P 5150 7400
-F 0 "#PWR03" H 5150 7150 50  0001 C CNN
+F 0 "#PWR3" H 5150 7150 50  0001 C CNN
 F 1 "GND" H 5150 7250 50  0000 C CNN
 F 2 "" H 5150 7400 50  0001 C CNN
@@
 F 0 "U5" H 4550 6350 60  0000 C CNN
 F 1 "G2RL-1A-E" V 4900 6350 60  0000 C CNN
-F 2 "" H 4650 6350 60  0000 C CNN
+F 2 "FSFootprints:G2RL-1A-E" H 4650 6350 60  0001 C CNN
 F 3 "" H 4650 6350 60  0000 C CNN
 	1    4650 6350
@@
 F 0 "U6" H 4550 7250 60  0000 C CNN
 F 1 "G2RL-1A-E" V 4900 7250 60  0000 C CNN
-F 2 "" H 4650 7250 60  0000 C CNN
+F 2 "FSFootprints:G2RL-1A-E" H 4650 7250 60  0001 C CNN
 F 3 "" H 4650 7250 60  0000 C CNN
 	1    4650 7250
 	-1   0    0    -1
 $EndComp
+$Comp
+L Conn_01x01 H1
+U 1 1 5A9779AD
+P 10750 5500
+F 0 "H1" H 10750 5600 50  0000 C CNN
+F 1 "MtngHole" H 10750 5400 50  0000 C CNN
+F 2 "Mounting_Holes:MountingHole_4.5mm" H 10750 5500 50  0001 C CNN
+F 3 "" H 10750 5500 50  0001 C CNN
+	1    10750 5500
+	1    0    0    -1
+$EndComp
+$Comp
+L Conn_01x01 H2
+U 1 1 5A9783D5
+P 10750 5800
+F 0 "H2" H 10750 5900 50  0000 C CNN
+F 1 "MtngHole" H 10750 5700 50  0000 C CNN
+F 2 "Mounting_Holes:MountingHole_4.5mm" H 10750 5800 50  0001 C CNN
+F 3 "" H 10750 5800 50  0001 C CNN
+	1    10750 5800
+	1    0    0    -1
+$EndComp
+$Comp
+L Conn_01x01 H3
+U 1 1 5A978484
+P 10750 6100
+F 0 "H3" H 10750 6200 50  0000 C CNN
+F 1 "MtngHole" H 10750 6000 50  0000 C CNN
+F 2 "Mounting_Holes:MountingHole_4.5mm" H 10750 6100 50  0001 C CNN
+F 3 "" H 10750 6100 50  0001 C CNN
+	1    10750 6100
+	1    0    0    -1
+$EndComp
+$Comp
+L Conn_01x01 H4
+U 1 1 5A978BA0
+P 10750 6400
+F 0 "H4" H 10750 6500 50  0000 C CNN
+F 1 "MtngHole" H 10750 6300 50  0000 C CNN
+F 2 "Mounting_Holes:MountingHole_4.5mm" H 10750 6400 50  0001 C CNN
+F 3 "" H 10750 6400 50  0001 C CNN
+	1    10750 6400
+	1    0    0    -1
+$EndComp
 $EndSCHEMATC

Commit message: Add larger fuse to AccumulatorHV board
Parts:
- F2: footprint FSFootprints:SMD Fuse -> Fuse_Holders_and_Fuses:Fuseholder6x32_Horiz_Open_Schurter0031-8002
- R9: footprint Resistors_THT:R_Axial_DIN0204_L3.6mm_D1.6mm_P1.90mm_Vertical -> Oddities:NetTie-I_Connected_SMD
Changed lines of the file:
@@
 LIBS:valves
 LIBS:arduino
+LIBS:AccumulatorBoardHV-cache
 EELAYER 25 0
 EELAYER END
@@
 F 0 "F2" V 2830 1150 50  0000 C CNN
 F 1 "IMD/DCDC Fuse" V 2675 1150 50  0000 C CNN
-F 2 "FSFootprints:SMD Fuse" V 2680 1150 50  0001 C CNN
+F 2 "Fuse_Holders_and_Fuses:Fuseholder6x32_Horiz_Open_Schurter0031-8002" V 2680 1150 50  0001 C CNN
 F 3 "" H 2750 1150 50  0000 C CNN
 	1    2750 1150
@@
 GND
 $Comp
-L GND #PWR1
+L GND #PWR01
 U 1 1 58B2C1BD
 P 5300 1450
-F 0 "#PWR1" H 5300 1200 50  0001 C CNN
+F 0 "#PWR01" H 5300 1200 50  0001 C CNN
 F 1 "GND" H 5300 1300 50  0000 C CNN
 F 2 "" H 5300 1450 50  0000 C CNN
@@
 AIRS_FINAL_CHARGER
 $Comp
-L GND #PWR2
+L GND #PWR02
 U 1 1 5959BDAF
 P 5150 6500
-F 0 "#PWR2" H 5150 6250 50  0001 C CNN
+F 0 "#PWR02" H 5150 6250 50  0001 C CNN
 F 1 "GND" H 5150 6350 50  0000 C CNN
 F 2 "" H 5150 6500 50  0001 C CNN
@@
 $EndComp
 $Comp
-L GND #PWR3
+L GND #PWR03
 U 1 1 5959BDF7
 P 5150 7400
-F 0 "#PWR3" H 5150 7150 50  0001 C CNN
+F 0 "#PWR03" H 5150 7150 50  0001 C CNN
 F 1 "GND" H 5150 7250 50  0000 C CNN
 F 2 "" H 5150 7400 50  0001 C CNN
@@
 F 0 "R9" V 3480 5100 50  0000 C CNN
 F 1 "0" V 3400 5100 50  0000 C CNN
-F 2 "Resistors_THT:R_Axial_DIN0204_L3.6mm_D1.6mm_P1.90mm_Vertical" V 3330 5100 50  0001 C CNN
+F 2 "Oddities:NetTie-I_Connected_SMD" V 3330 5100 50  0001 C CNN
 F 3 "" H 3400 5100 50  0001 C CNN
 	1    3400 5100

Commit message: Revise boards based on design review
Parts:
- removed J9: Charger Current to Batt, Connectors_Molex:Molex_MiniFit-JR-5556-02A_2x01x4.20mm_Straight, symbol Conn_01x02
- added R1, R2: 0, FSFootprints:SMDNetTie, symbol R
- F2: footprint Fuse_Holders_and_Fuses:Fuseholder6x32_Horiz_Open_Schurter0031-8002 -> Fuse_Holders_and_Fuses:Fuseholder5x20_vert_closed_Bulgin_FX0456
- F6: value Fuse -> Charger Fuse; footprint FSFootprints:SMD Fuse -> Fuse_Holders_and_Fuses:Fuseholder5x20_vert_closed_Bulgin_FX0456
- R11: renamed from R9; footprint Oddities:NetTie-I_Connected_SMD -> FSFootprints:SMDNetTie
- U1: footprint FSFootprints:VICOR-DCDC -> FSFootprints:Vicor_Micro
- renumbered J10 to J9, R8 to R10, R1 to R3, R2 to R4, R3 to R5, R4 to R6, R5 to R7, R6 to R8, R7 to R9
Connections:
- net labels added: 3.3V_TS_PRE
- wire segments 61 -> 63
Changed lines of the file:
@@
-	-1   0    0    -1
-$EndComp
-$Comp
-L Conn_01x02 J3
-U 1 1 589D2D5E
-P 1150 1150
-F 0 "J3" H 1150 1300 50  0000 C CNN
-F 1 "Batt Voltage" V 1250 1150 50  0000 C CNN
-F 2 "Connectors_Molex:Molex_MiniFit-JR-5556-02A_2x01x4.20mm_Straight" H 1150 1150 50  0001 C CNN
-F 3 "" H 1150 1150 50  0000 C CNN
-	1    1150 1150
 	-1   0    0    -1
 $EndComp
@@
 F 0 "F2" V 2830 1150 50  0000 C CNN
 F 1 "IMD/DCDC Fuse" V 2675 1150 50  0000 C CNN
-F 2 "Fuse_Holders_and_Fuses:Fuseholder6x32_Horiz_Open_Schurter0031-8002" V 2680 1150 50  0001 C CNN
+F 2 "Fuse_Holders_and_Fuses:Fuseholder5x20_vert_closed_Bulgin_FX0456" V 2680 1150 50  0001 C CNN
 F 3 "" H 2750 1150 50  0000 C CNN
 	1    2750 1150
@@
 $EndComp
 $Comp
-L R R4
+L R R6
 U 1 1 58A0E923
 P 3650 4100
-F 0 "R4" V 3730 4100 50  0000 C CNN
+F 0 "R6" V 3730 4100 50  0000 C CNN
 F 1 "1.5kR" V 3650 4100 50  0000 C CNN
 F 2 "Resistors_THT:R_Axial_DIN0207_L6.3mm_D2.5mm_P10.16mm_Horizontal" V 3580 4100 50  0001 C CNN
@@
 F 0 "U1" H 4550 1500 60  0000 C CNN
 F 1 "V110C12E100BL" H 4550 1650 60  0000 C CNN
-F 2 "FSFootprints:VICOR-DCDC" H 4550 1200 60  0001 C CNN
+F 2 "FSFootprints:Vicor_Micro" H 4550 1200 60  0001 C CNN
 F 3 "" H 4550 1200 60  0001 C CNN
 	1    4550 1200
@@
 $EndComp
 $Comp
-L Conn_01x02 J10
+L Conn_01x02 J9
 U 1 1 5959BFDF
 P 2900 6650
-F 0 "J10" H 2900 6800 50  0000 C CNN
+F 0 "J9" H 2900 6800 50  0000 C CNN
 F 1 "Charger Current" V 3000 6650 50  0000 C CNN
 F 2 "Connectors_Molex:Molex_MiniFit-JR-5556-02A_2x01x4.20mm_Straight" H 2900 6650 50  0001 C CNN
@@
 BATT-_CHARGER
 $Comp
-L R R2
+L R R4
 U 1 1 59A35367
 P 2850 3650
-F 0 "R2" V 2930 3650 50  0000 C CNN
+F 0 "R4" V 2930 3650 50  0000 C CNN
 F 1 "1.5kR" V 2850 3650 50  0000 C CNN
 F 2 "Resistors_THT:R_Axial_DIN0207_L6.3mm_D2.5mm_P10.16mm_Horizontal" V 2780 3650 50  0001 C CNN
@@
 $EndComp
 $Comp
-L R R3
+L R R5
 U 1 1 59A354F0
 P 4000 3750
-F 0 "R3" V 4080 3750 50  0000 C CNN
+F 0 "R5" V 4080 3750 50  0000 C CNN
 F 1 "R" V 4000 3750 50  0000 C CNN
 F 2 "Resistors_THT:R_Axial_DIN0207_L6.3mm_D2.5mm_P10.16mm_Horizontal" V 3930 3750 50  0001 C CNN
@@
 $EndComp
 $Comp
-L R R8
+L R R10
 U 1 1 59A3D9D7
 P 3650 4950
-F 0 "R8" V 3730 4950 50  0000 C CNN
+F 0 "R10" V 3730 4950 50  0000 C CNN
 F 1 "1.5kR" V 3650 4950 50  0000 C CNN
 F 2 "Resistors_THT:R_Axial_DIN0207_L6.3mm_D2.5mm_P10.16mm_Horizontal" V 3580 4950 50  0001 C CNN
@@
 $EndComp
 $Comp
-L R R6
+L R R8
 U 1 1 59A3D9EA
 P 2850 4500
-F 0 "R6" V 2930 4500 50  0000 C CNN
+F 0 "R8" V 2930 4500 50  0000 C CNN
 F 1 "1.5kR" V 2850 4500 50  0000 C CNN
 F 2 "Resistors_THT:R_Axial_DIN0207_L6.3mm_D2.5mm_P10.16mm_Horizontal" V 2780 4500 50  0001 C CNN
@@
 $EndComp
 $Comp
-L R R5
+L R R7
 U 1 1 59A3D9F2
 P 4000 4400
-F 0 "R5" V 4080 4400 50  0000 C CNN
+F 0 "R7" V 4080 4400 50  0000 C CNN
 F 1 "R" V 4000 4400 50  0000 C CNN
 F 2 "Resistors_THT:R_Axial_DIN0207_L6.3mm_D2.5mm_P10.16mm_Horizontal" V 3930 4400 50  0001 C CNN
@@
 $EndComp
 $Comp
-L R R1
+L R R3
 U 1 1 5A51F75F
 P 4000 3550
-F 0 "R1" V 4080 3550 50  0000 C CNN
+F 0 "R3" V 4080 3550 50  0000 C CNN
 F 1 "R" V 4000 3550 50  0000 C CNN
 F 2 "Resistors_THT:R_Axial_DIN0207_L6.3mm_D2.5mm_P10.16mm_Horizontal" V 3930 3550 50  0001 C CNN
@@
 $EndComp
 $Comp
-L R R7
+L R R9
 U 1 1 5A51FDE6
 P 4000 4600
-F 0 "R7" V 4080 4600 50  0000 C CNN
+F 0 "R9" V 4080 4600 50  0000 C CNN
 F 1 "R" V 4000 4600 50  0000 C CNN
 F 2 "Resistors_THT:R_Axial_DIN0207_L6.3mm_D2.5mm_P10.16mm_Horizontal" V 3930 4600 50  0001 C CNN
@@
 P 4400 5950
 F 0 "F6" V 4480 5950 50  0000 C CNN
-F 1 "Fuse" V 4325 5950 50  0000 C CNN
-F 2 "FSFootprints:SMD Fuse" V 4330 5950 50  0001 C CNN
+F 1 "Charger Fuse" V 4325 5950 50  0000 C CNN
+F 2 "Fuse_Holders_and_Fuses:Fuseholder5x20_vert_closed_Bulgin_FX0456" V 4330 5950 50  0001 C CNN
 F 3 "" H 4400 5950 50  0001 C CNN
 	1    4400 5950
@@
 Wire Wire Line
 	4550 6050 4550 5950
-$Comp
-L Conn_01x02 J9
-U 1 1 5A81246B
-P 2200 5800
-F 0 "J9" H 2200 5900 50  0000 C CNN
-F 1 "Charger Current to Batt" V 2300 5800 50  0000 C CNN
-F 2 "Connectors_Molex:Molex_MiniFit-JR-5556-02A_2x01x4.20mm_Straight" H 2200 5800 50  0001 C CNN
-F 3 "" H 2200 5800 50  0001 C CNN
-	1    2200 5800
-	-1   0    0    -1
-$EndComp
-Text Label 2400 5800 0    60   ~ 0
+Text Label 1050 1000 0    60   ~ 0
 BATT+_CHARGER
-Text Label 2400 5900 0    60   ~ 0
+Text Label 1050 1450 0    60   ~ 0
 BATT-_CHARGER
 Text Label 4650 6050 1    60   ~ 0
 BATT+_CHGFUSED
 $Comp
-L R R9
+L R R11
 U 1 1 5A81592B
 P 3400 5100
-F 0 "R9" V 3480 5100 50  0000 C CNN
+F 0 "R11" V 3480 5100 50  0000 C CNN
 F 1 "0" V 3400 5100 50  0000 C CNN
-F 2 "Oddities:NetTie-I_Connected_SMD" V 3330 5100 50  0001 C CNN
+F 2 "FSFootprints:SMDNetTie" V 3330 5100 50  0001 C CNN
 F 3 "" H 3400 5100 50  0001 C CNN
 	1    3400 5100
@@
 	1    0    0    -1
 $EndComp
+$Comp
+L Conn_01x02 J3
+U 1 1 589D2D5E
+P 850 1150
+F 0 "J3" H 850 1300 50  0000 C CNN
+F 1 "Batt Voltage" V 950 1150 50  0000 C CNN
+F 2 "Connectors_Molex:Molex_MiniFit-JR-5556-02A_2x01x4.20mm_Straight" H 850 1150 50  0001 C CNN
+F 3 "" H 850 1150 50  0000 C CNN
+	1    850  1150
+	-1   0    0    -1
+$EndComp
+$Comp
+L R R1
+U 1 1 5AA37E93
+P 1200 1150
+F 0 "R1" V 1100 1150 50  0000 C CNN
+F 1 "0" V 1200 1150 50  0000 C CNN
+F 2 "FSFootprints:SMDNetTie" V 1130 1150 50  0001 C CNN
+F 3 "" H 1200 1150 50  0001 C CNN
+	1    1200 1150
+	0    1    1    0
+$EndComp
+$Comp
+L R R2
+U 1 1 5AA38094
+P 1200 1250
+F 0 "R2" V 1280 1250 50  0000 C CNN
+F 1 "0" V 1200 1250 50  0000 C CNN
+F 2 "FSFootprints:SMDNetTie" V 1130 1250 50  0001 C CNN
+F 3 "" H 1200 1250 50  0001 C CNN
+	1    1200 1250
+	0    1    1    0
+$EndComp
+Wire Wire Line
+	1050 1250 1050 1450
+Wire Wire Line
+	1050 1150 1050 1000
+Text Label 2150 2550 0    60   ~ 0
+3.3V_TS_PRE
 $EndSCHEMATC

Commit message: shrink AccumulatorHV PCB
Parts:
- removed C1, C2, C5, C6: C, Capacitors_THT:C_Disc_D4.7mm_W2.5mm_P5.00mm, symbol C
- removed U4: PS2501-4, Housings_DIP:DIP-16_W7.62mm, symbol PS2501-4
- added U4: PS2501-4-1, Housings_DIP:DIP-16_W7.62mm, symbol PS2501-4-1
- D1, D2, D3, D4: footprint Diodes_THT:D_DO-15_P12.70mm_Horizontal -> Diodes_THT:D_A-405_P7.62mm_Horizontal
- F2, F6: footprint Fuse_Holders_and_Fuses:Fuseholder5x20_vert_closed_Bulgin_FX0456 -> FSFootprints:Fuseholder5x20_vert
- J2: footprint Connectors_Molex:Molex_NanoFit_1x04x2.50mm_Straight -> Connectors_Molex:Molex_NanoFit_2x02x2.50mm_Straight
- renumbered C3 to C1, C4 to C2, C7 to C3, C8 to C4, C9 to C5
Connections:
- wire segments 63 -> 60
Changed lines of the file:
@@
 F 0 "F2" V 2830 1150 50  0000 C CNN
 F 1 "IMD/DCDC Fuse" V 2675 1150 50  0000 C CNN
-F 2 "Fuse_Holders_and_Fuses:Fuseholder5x20_vert_closed_Bulgin_FX0456" V 2680 1150 50  0001 C CNN
+F 2 "FSFootprints:Fuseholder5x20_vert" V 2680 1150 50  0001 C CNN
 F 3 "" H 2750 1150 50  0000 C CNN
 	1    2750 1150
@@
 F 0 "D1" H 3300 3750 50  0000 C CNN
 F 1 "48V Zener" H 3300 3550 50  0000 C CNN
-F 2 "Diodes_THT:D_DO-15_P12.70mm_Horizontal" H 3300 3650 50  0001 C CNN
+F 2 "Diodes_THT:D_A-405_P7.62mm_Horizontal" H 3300 3650 50  0001 C CNN
 F 3 "" H 3300 3650 50  0000 C CNN
 	1    3300 3650
@@
 F 0 "D2" H 3650 3900 50  0000 C CNN
 F 1 "12V Zener" H 3650 3700 50  0000 C CNN
-F 2 "Diodes_THT:D_DO-15_P12.70mm_Horizontal" H 3650 3800 50  0001 C CNN
+F 2 "Diodes_THT:D_A-405_P7.62mm_Horizontal" H 3650 3800 50  0001 C CNN
 F 3 "" H 3650 3800 50  0000 C CNN
 	1    3650 3800
@@
 12V_INDICATOR
 $Comp
-L CP C3
+L CP C1
 U 1 1 58AD4675
 P 3350 1300
-F 0 "C3" H 3375 1400 50  0000 L CNN
+F 0 "C1" H 3375 1400 50  0000 L CNN
 F 1 "0.47uF" H 3375 1200 50  0000 L CNN
 F 2 "Capacitors_THT:CP_Radial_D8.0mm_P2.50mm" H 3388 1150 50  0001 C CNN
@@
 Text Label 5600 950  0    60   ~ 0
 12V_SRC
-$Comp
-L V110C12E100BL U1
-U 1 1 58AD6878
-P 4550 1200
-F 0 "U1" H 4550 1500 60  0000 C CNN
-F 1 "V110C12E100BL" H 4550 1650 60  0000 C CNN
-F 2 "FSFootprints:Vicor_Micro" H 4550 1200 60  0001 C CNN
-F 3 "" H 4550 1200 60  0001 C CNN
-	1    4550 1200
-	1    0    0    -1
-$EndComp
-$Comp
-L C C5
-U 1 1 58AD6947
-P 4050 1600
-F 0 "C5" H 4075 1700 50  0000 L CNN
-F 1 "C" H 4075 1500 50  0000 L CNN
-F 2 "Capacitors_THT:C_Disc_D4.7mm_W2.5mm_P5.00mm" H 4088 1450 50  0001 C CNN
-F 3 "" H 4050 1600 50  0000 C CNN
-	1    4050 1600
-	1    0    0    -1
-$EndComp
-$Comp
-L C C1
-U 1 1 58AD6A90
-P 4050 800
-F 0 "C1" H 4075 900 50  0000 L CNN
-F 1 "C" H 4075 700 50  0000 L CNN
-F 2 "Capacitors_THT:C_Disc_D4.7mm_W2.5mm_P5.00mm" H 4088 650 50  0001 C CNN
-F 3 "" H 4050 800 50  0000 C CNN
-	1    4050 800
-	1    0    0    -1
-$EndComp
 NoConn ~ 4050 1100
 NoConn ~ 4050 1300
@@
 GND
 $Comp
-L CP C4
+L CP C2
 U 1 1 594F0A21
 P 5300 1300
-F 0 "C4" H 5325 1400 50  0000 L CNN
+F 0 "C2" H 5325 1400 50  0000 L CNN
 F 1 "CP" H 5325 1200 50  0000 L CNN
 F 2 "Capacitors_THT:CP_Radial_D8.0mm_P2.50mm" H 5338 1150 50  0001 C CNN
@@
 AIRS_FINAL_CHARGER
 $Comp
-L C C6
-U 1 1 59A37CC7
-P 5050 1600
-F 0 "C6" H 5075 1700 50  0000 L CNN
-F 1 "C" H 5075 1500 50  0000 L CNN
-F 2 "Capacitors_THT:C_Disc_D4.7mm_W2.5mm_P5.00mm" H 5088 1450 50  0001 C CNN
-F 3 "" H 5050 1600 50  0000 C CNN
-	1    5050 1600
-	1    0    0    -1
-$EndComp
-$Comp
-L C C2
-U 1 1 59A37EB1
-P 5050 800
-F 0 "C2" H 5075 900 50  0000 L CNN
-F 1 "C" H 5075 700 50  0000 L CNN
-F 2 "Capacitors_THT:C_Disc_D4.7mm_W2.5mm_P5.00mm" H 5088 650 50  0001 C CNN
-F 3 "" H 5050 800 50  0000 C CNN
-	1    5050 800
-	1    0    0    -1
-$EndComp
-$Comp
 L D_Zener D3
 U 1 1 59A3D9CB
@@
 F 0 "D3" H 3300 4600 50  0000 C CNN
 F 1 "48V Zener" H 3300 4400 50  0000 C CNN
-F 2 "Diodes_THT:D_DO-15_P12.70mm_Horizontal" H 3300 4500 50  0001 C CNN
+F 2 "Diodes_THT:D_A-405_P7.62mm_Horizontal" H 3300 4500 50  0001 C CNN
 F 3 "" H 3300 4500 50  0000 C CNN
 	1    3300 4500
@@
 F 0 "D4" H 3650 4750 50  0000 C CNN
 F 1 "12V Zener" H 3650 4550 50  0000 C CNN
-F 2 "Diodes_THT:D_DO-15_P12.70mm_Horizontal" H 3650 4650 50  0001 C CNN
+F 2 "Diodes_THT:D_A-405_P7.62mm_Horizontal" H 3650 4650 50  0001 C CNN
 F 3 "" H 3650 4650 50  0000 C CNN
 	1    3650 4650
@@
 BATT-
 $Comp
-L CP C7
+L CP C3
 U 1 1 59C0E5C6
 P 2100 2250
-F 0 "C7" H 2125 2350 50  0000 L CNN
+F 0 "C3" H 2125 2350 50  0000 L CNN
 F 1 "100uF" H 2125 2150 50  0000 L CNN
 F 2 "Capacitors_THT:CP_Radial_D16.0mm_P7.50mm" H 2138 2100 50  0001 C CNN
@@
 $EndComp
 $Comp
-L CP C8
+L CP C4
 U 1 1 59C0E645
 P 2500 2250
-F 0 "C8" H 2525 2350 50  0000 L CNN
+F 0 "C4" H 2525 2350 50  0000 L CNN
 F 1 "100uF" H 2525 2150 50  0000 L CNN
 F 2 "Capacitors_THT:CP_Radial_D16.0mm_P7.50mm" H 2538 2100 50  0001 C CNN
@@
 BATT-
 $Comp
-L CP C9
+L CP C5
 U 1 1 59C0EDAC
 P 2950 2900
-F 0 "C9" H 2975 3000 50  0000 L CNN
+F 0 "C5" H 2975 3000 50  0000 L CNN
 F 1 "CP" H 2975 2800 50  0000 L CNN
 F 2 "Capacitors_THT:CP_Radial_D8.0mm_P2.50mm" H 2988 2750 50  0001 C CNN
@@
 	3700 950  4050 950
 Wire Wire Line
-	3900 1750 5050 1750
-Wire Wire Line
-	3900 650  3900 1750
-Connection ~ 4050 1750
-Wire Wire Line
 	3650 4250 3550 4250
-Wire Wire Line
-	3900 650  5050 650
 Connection ~ 3650 3650
 Connection ~ 3650 3950
@@
 Wire Notes Line
 	1700 3250 7200 3250
-Connection ~ 4550 1750
-Connection ~ 4050 650
 Wire Wire Line
 	5050 950  5300 950
@@
 F 0 "J2" H 6400 1250 50  0000 C CNN
 F 1 "To LV Board" H 6400 750 50  0000 C CNN
-F 2 "Connectors_Molex:Molex_NanoFit_1x04x2.50mm_Straight" H 6400 1050 50  0001 C CNN
+F 2 "Connectors_Molex:Molex_NanoFit_2x02x2.50mm_Straight" H 6400 1050 50  0001 C CNN
 F 3 "" H 6400 1050 50  0001 C CNN
 	1    6400 1050
@@
 F 0 "F6" V 4480 5950 50  0000 C CNN
 F 1 "Charger Fuse" V 4325 5950 50  0000 C CNN
-F 2 "Fuse_Holders_and_Fuses:Fuseholder5x20_vert_closed_Bulgin_FX0456" V 4330 5950 50  0001 C CNN
+F 2 "FSFootprints:Fuseholder5x20_vert" V 4330 5950 50  0001 C CNN
 F 3 "" H 4400 5950 50  0001 C CNN
 	1    4400 5950
@@
 Text Label 3550 2100 0    60   ~ 0
 BATT+_LVBOARD
-$Comp
-L PS2501-4 U4
-U 1 1 5A7B8267
-P 4750 4500
-F 0 "U4" H 4550 4700 50  0000 L CNN
-F 1 "PS2501-4" H 4550 4300 50  0000 L CNN
-F 2 "Housings_DIP:DIP-16_W7.62mm" H 4550 4300 50  0001 L CIN
-F 3 "" H 4750 4500 50  0000 L CNN
-	1    4750 4500
-	1    0    0    -1
-$EndComp
-$Comp
-L PS2501-4 U4
-U 2 1 5A7B8465
-P 4750 4850
-F 0 "U4" H 4550 5050 50  0000 L CNN
-F 1 "PS2501-4" H 4550 4650 50  0000 L CNN
-F 2 "Housings_DIP:DIP-16_W7.62mm" H 4550 4650 50  0001 L CIN
-F 3 "" H 4750 4850 50  0000 L CNN
-	2    4750 4850
-	1    0    0    -1
-$EndComp
-$Comp
-L PS2501-4 U4
-U 3 1 5A7B87CB
-P 4750 3750
-F 0 "U4" H 4550 3950 50  0000 L CNN
-F 1 "PS2501-4" H 4550 3550 50  0000 L CNN
-F 2 "Housings_DIP:DIP-16_W7.62mm" H 4550 3550 50  0001 L CIN
-F 3 "" H 4750 3750 50  0000 L CNN
-	3    4750 3750
-	1    0    0    -1
-$EndComp
-$Comp
-L PS2501-4 U4
-U 4 1 5A7B8868
-P 4750 4100
-F 0 "U4" H 4550 4300 50  0000 L CNN
-F 1 "PS2501-4" H 4550 3900 50  0000 L CNN
-F 2 "Housings_DIP:DIP-16_W7.62mm" H 4550 3900 50  0001 L CIN
-F 3 "" H 4750 4100 50  0000 L CNN
-	4    4750 4100
-	1    0    0    -1
-$EndComp
 Wire Wire Line
 	4550 6050 4550 5950
@@
 Text Label 2150 2550 0    60   ~ 0
 3.3V_TS_PRE
+$Comp
+L V110C12E100BL U1
+U 1 1 58AD6878
+P 4550 1200
+F 0 "U1" H 4550 1500 60  0000 C CNN
+F 1 "V110C12E100BL" H 4550 1650 60  0000 C CNN
+F 2 "FSFootprints:Vicor_Micro" H 4550 1200 60  0001 C CNN
+F 3 "" H 4550 1200 60  0001 C CNN
+	1    4550 1200
+	1    0    0    -1
+$EndComp
+$Comp
+L PS2501-4-1 U4
+U 1 1 5ABB07D4
+P 4750 4300
+F 0 "U4" H 4550 5050 50  0000 L CNN
+F 1 "PS2501-4-1" H 4550 3550 50  0000 L CNN
+F 2 "Housings_DIP:DIP-16_W7.62mm" H 4550 4650 50  0001 L CIN
+F 3 "" H 4750 4850 50  0000 L CNN
+	1    4750 4300
+	1    0    0    -1
+$EndComp
 $EndSCHEMATC
