File: AccumulatorBoardHV/AccumulatorBoardHV.sch (KiCad schematic (older format))
At the start: 45 parts, among them J1 TS -> GLV Regulator Jumper, J2 To LV Board, J3 Batt Voltage, J4 TS (Switched), J5 IMD TS, J6 To LV Board, J7 Acc LED 1, J8 Acc LED 2, J9 Charger Current, U1 V110C12E100BL, U2 DK1A1B-12V, U3 RDD08110S3V3, U4 PS2501-4-1, U5 G2RL-1A-E, U6 G2RL-1A-E

Commit message: Tweak 60v circuits based on testing results
Parts:
- removed R8: 1.5kR, Resistors_THT:R_Axial_DIN0207_L6.3mm_D2.5mm_P10.16mm_Horizontal, symbol R
- added Q1: Q_NMOS_GDS, TO_SOT_Packages_THT:TO-220-3_Vertical, symbol Q_NMOS_GDS
- D1, D3: value 48V Zener -> 56V Zener
- R3, R5, R7: value R -> 1.2k
- R4: value 1.5kR -> 100
- R6: value 1.5kR -> 1.5k
- R8: renamed from R9; value R -> 1.2k
- R9: renamed from R10; value 1.5kR -> 1.5k
- renumbered R11 to R10
Connections:
- net labels added: 12V_INDICATOR_CTRL
- wire segments 60 -> 56
Other:
- moved on the sheet: F4, F5
Changed lines of the file:
@@
 P 3300 3650
 F 0 "D1" H 3300 3750 50  0000 C CNN
-F 1 "48V Zener" H 3300 3550 50  0000 C CNN
+F 1 "56V Zener" H 3300 3550 50  0000 C CNN
 F 2 "Diodes_THT:D_A-405_P7.62mm_Horizontal" H 3300 3650 50  0001 C CNN
 F 3 "" H 3300 3650 50  0000 C CNN
@@
 P 3650 4100
 F 0 "R6" V 3730 4100 50  0000 C CNN
-F 1 "1.5kR" V 3650 4100 50  0000 C CNN
+F 1 "1.5k" V 3650 4100 50  0000 C CNN
 F 2 "Resistors_THT:R_Axial_DIN0207_L6.3mm_D2.5mm_P10.16mm_Horizontal" V 3580 4100 50  0001 C CNN
 F 3 "" H 3650 4100 50  0000 C CNN
@@
 Text Label 3550 4250 2    60   ~ 0
 TS-
-Text Label 2250 3650 3    60   ~ 0
+Text Label 2850 3650 3    60   ~ 0
 TS+
 Text Label 5050 3850 0    60   ~ 0
-12V_INDICATOR
+12V_INDICATOR_CTRL
 $Comp
 L CP C1
@@
 L Conn_01x02 J7
 U 1 1 58B07EC2
-P 6200 3900
-F 0 "J7" H 6200 4050 50  0000 C CNN
-F 1 "Acc LED 1" V 6300 3900 50  0000 C CNN
-F 2 "Connectors_Molex:Molex_NanoFit_1x02x2.50mm_Straight" H 6200 3900 50  0001 C CNN
-F 3 "" H 6200 3900 50  0000 C CNN
-	1    6200 3900
+P 6200 4250
+F 0 "J7" H 6200 4400 50  0000 C CNN
+F 1 "Acc LED 1" V 6300 4250 50  0000 C CNN
+F 2 "Connectors_Molex:Molex_NanoFit_1x02x2.50mm_Straight" H 6200 4250 50  0001 C CNN
+F 3 "" H 6200 4250 50  0000 C CNN
+	1    6200 4250
 	-1   0    0    -1
 $EndComp
-Text Label 6400 3900 0    60   ~ 0
+Text Label 6400 4350 0    60   ~ 0
 12V_INDICATOR
-Text Label 6400 4000 0    60   ~ 0
-GND
 $Comp
 L GND #PWR01
@@
 L Conn_01x02 J8
 U 1 1 58B9D04E
-P 6200 4350
-F 0 "J8" H 6200 4500 50  0000 C CNN
-F 1 "Acc LED 2" V 6300 4350 50  0000 C CNN
-F 2 "Connectors_Molex:Molex_NanoFit_1x02x2.50mm_Straight" H 6200 4350 50  0001 C CNN
-F 3 "" H 6200 4350 50  0000 C CNN
-	1    6200 4350
+P 6200 4700
+F 0 "J8" H 6200 4850 50  0000 C CNN
+F 1 "Acc LED 2" V 6300 4700 50  0000 C CNN
+F 2 "Connectors_Molex:Molex_NanoFit_1x02x2.50mm_Straight" H 6200 4700 50  0001 C CNN
+F 3 "" H 6200 4700 50  0000 C CNN
+	1    6200 4700
 	-1   0    0    -1
 $EndComp
-Text Label 6400 4350 0    60   ~ 0
+Text Label 6400 4800 0    60   ~ 0
 12V_INDICATOR
-Text Label 6400 4450 0    60   ~ 0
-GND
 $Comp
 L Fuse F1
@@
 L Fuse F4
 U 1 1 58C4B2C9
-P 2400 3650
-F 0 "F4" V 2480 3650 50  0000 C CNN
-F 1 "TS 60V Fuse" V 2325 3650 50  0000 C CNN
-F 2 "FSFootprints:SMD Fuse" V 2330 3650 50  0001 C CNN
-F 3 "" H 2400 3650 50  0000 C CNN
-	1    2400 3650
+P 3000 3650
+F 0 "F4" V 3080 3650 50  0000 C CNN
+F 1 "TS 60V Fuse" V 2925 3650 50  0000 C CNN
+F 2 "FSFootprints:SMD Fuse" V 2930 3650 50  0001 C CNN
+F 3 "" H 3000 3650 50  0000 C CNN
+	1    3000 3650
 	0    1    1    0
 $EndComp
@@
 BATT-_CHARGER
 $Comp
-L R R4
-U 1 1 59A35367
-P 2850 3650
-F 0 "R4" V 2930 3650 50  0000 C CNN
-F 1 "1.5kR" V 2850 3650 50  0000 C CNN
-F 2 "Resistors_THT:R_Axial_DIN0207_L6.3mm_D2.5mm_P10.16mm_Horizontal" V 2780 3650 50  0001 C CNN
-F 3 "" H 2850 3650 50  0000 C CNN
-	1    2850 3650
-	0    1    1    0
-$EndComp
-$Comp
 L R R5
 U 1 1 59A354F0
 P 4000 3750
 F 0 "R5" V 4080 3750 50  0000 C CNN
-F 1 "R" V 4000 3750 50  0000 C CNN
+F 1 "1.2k" V 4000 3750 50  0000 C CNN
 F 2 "Resistors_THT:R_Axial_DIN0207_L6.3mm_D2.5mm_P10.16mm_Horizontal" V 3930 3750 50  0001 C CNN
 F 3 "" H 4000 3750 50  0000 C CNN
@@
 P 3300 4500
 F 0 "D3" H 3300 4600 50  0000 C CNN
-F 1 "48V Zener" H 3300 4400 50  0000 C CNN
+F 1 "56V Zener" H 3300 4400 50  0000 C CNN
 F 2 "Diodes_THT:D_A-405_P7.62mm_Horizontal" H 3300 4500 50  0001 C CNN
 F 3 "" H 3300 4500 50  0000 C CNN
@@
 $EndComp
 $Comp
-L R R10
+L R R9
 U 1 1 59A3D9D7
 P 3650 4950
-F 0 "R10" V 3730 4950 50  0000 C CNN
-F 1 "1.5kR" V 3650 4950 50  0000 C CNN
+F 0 "R9" V 3730 4950 50  0000 C CNN
+F 1 "1.5k" V 3650 4950 50  0000 C CNN
 F 2 "Resistors_THT:R_Axial_DIN0207_L6.3mm_D2.5mm_P10.16mm_Horizontal" V 3580 4950 50  0001 C CNN
 F 3 "" H 3650 4950 50  0000 C CNN
@@
 Text Label 3250 5100 2    60   ~ 0
 CHARGER-
-Text Label 2250 4500 3    60   ~ 0
+Text Label 2850 4500 3    60   ~ 0
 CHARGER+
 Text Label 5050 4950 0    60   ~ 0
-12V_INDICATOR
+12V_INDICATOR_CTRL
 $Comp
 L Fuse F5
 U 1 1 59A3D9E0
-P 2400 4500
-F 0 "F5" V 2480 4500 50  0000 C CNN
-F 1 "Charger 60V Fuse" V 2325 4500 50  0000 C CNN
-F 2 "FSFootprints:SMD Fuse" V 2330 4500 50  0001 C CNN
-F 3 "" H 2400 4500 50  0000 C CNN
-	1    2400 4500
-	0    1    1    0
-$EndComp
-$Comp
-L R R8
-U 1 1 59A3D9EA
-P 2850 4500
-F 0 "R8" V 2930 4500 50  0000 C CNN
-F 1 "1.5kR" V 2850 4500 50  0000 C CNN
-F 2 "Resistors_THT:R_Axial_DIN0207_L6.3mm_D2.5mm_P10.16mm_Horizontal" V 2780 4500 50  0001 C CNN
-F 3 "" H 2850 4500 50  0000 C CNN
-	1    2850 4500
+P 3000 4500
+F 0 "F5" V 3080 4500 50  0000 C CNN
+F 1 "Charger 60V Fuse" V 2925 4500 50  0000 C CNN
+F 2 "FSFootprints:SMD Fuse" V 2930 4500 50  0001 C CNN
+F 3 "" H 3000 4500 50  0000 C CNN
+	1    3000 4500
 	0    1    1    0
 $EndComp
@@
 P 4000 4400
 F 0 "R7" V 4080 4400 50  0000 C CNN
-F 1 "R" V 4000 4400 50  0000 C CNN
+F 1 "1.2k" V 4000 4400 50  0000 C CNN
 F 2 "Resistors_THT:R_Axial_DIN0207_L6.3mm_D2.5mm_P10.16mm_Horizontal" V 3930 4400 50  0001 C CNN
 F 3 "" H 4000 4400 50  0000 C CNN
@@
 12V_SRC
 Text Label 5050 4200 0    60   ~ 0
-12V_INDICATOR
+12V_INDICATOR_CTRL
 Text Label 5050 4600 0    60   ~ 0
-12V_INDICATOR
+12V_INDICATOR_CTRL
 Text Label 6600 1050 0    60   ~ 0
 12V
@@
 P 4000 3550
 F 0 "R3" V 4080 3550 50  0000 C CNN
-F 1 "R" V 4000 3550 50  0000 C CNN
+F 1 "1.2k" V 4000 3550 50  0000 C CNN
 F 2 "Resistors_THT:R_Axial_DIN0207_L6.3mm_D2.5mm_P10.16mm_Horizontal" V 3930 3550 50  0001 C CNN
 F 3 "" H 4000 3550 50  0000 C CNN
@@
 $EndComp
 $Comp
-L R R9
+L R R8
 U 1 1 5A51FDE6
 P 4000 4600
-F 0 "R9" V 4080 4600 50  0000 C CNN
-F 1 "R" V 4000 4600 50  0000 C CNN
+F 0 "R8" V 4080 4600 50  0000 C CNN
+F 1 "1.2k" V 4000 4600 50  0000 C CNN
 F 2 "Resistors_THT:R_Axial_DIN0207_L6.3mm_D2.5mm_P10.16mm_Horizontal" V 3930 4600 50  0001 C CNN
 F 3 "" H 4000 4600 50  0000 C CNN
@@
 	2900 1650 2900 1150
 Wire Wire Line
-	3150 3650 3000 3650
-Wire Wire Line
-	2700 3650 2550 3650
-Wire Wire Line
 	3450 3650 3850 3650
 Wire Notes Line
@@
 Connection ~ 3650 4500
 Connection ~ 3650 4800
-Wire Wire Line
-	3150 4500 3000 4500
-Wire Wire Line
-	2700 4500 2550 4500
 Wire Wire Line
 	3450 4500 3850 4500
@@
 BATT+_CHGFUSED
 $Comp
-L R R11
+L R R10
 U 1 1 5A81592B
 P 3400 5100
-F 0 "R11" V 3480 5100 50  0000 C CNN
+F 0 "R10" V 3480 5100 50  0000 C CNN
 F 1 "0" V 3400 5100 50  0000 C CNN
 F 2 "FSFootprints:SMDNetTie" V 3330 5100 50  0001 C CNN
@@
 	1    0    0    -1
 $EndComp
+$Comp
+L Q_NMOS_GDS Q1
+U 1 1 5ABC3572
+P 6700 3550
+F 0 "Q1" H 6900 3600 50  0000 L CNN
+F 1 "Q_NMOS_GDS" H 6900 3500 50  0000 L CNN
+F 2 "TO_SOT_Packages_THT:TO-220-3_Vertical" H 6900 3650 50  0001 C CNN
+F 3 "" H 6700 3550 50  0001 C CNN
+	1    6700 3550
+	1    0    0    -1
+$EndComp
+Text Label 6800 3750 3    60   ~ 0
+GND
+$Comp
+L R R4
+U 1 1 5ABC51E6
+P 6350 3550
+F 0 "R4" V 6430 3550 50  0000 C CNN
+F 1 "100" V 6350 3550 50  0000 C CNN
+F 2 "Resistors_THT:R_Axial_DIN0207_L6.3mm_D2.5mm_P10.16mm_Horizontal" V 6280 3550 50  0001 C CNN
+F 3 "" H 6350 3550 50  0001 C CNN
+	1    6350 3550
+	0    1    1    0
+$EndComp
+Text Label 6200 3550 2    60   ~ 0
+12V_INDICATOR_CTRL
+Text Label 6800 3350 2    60   ~ 0
+12V_INDICATOR
+Text Label 6400 4250 0    60   ~ 0
+12V_SRC
+Text Label 6400 4700 0    60   ~ 0
+12V_SRC
 $EndSCHEMATC

Commit message: add diodes to relay coils among other things
Parts:
- added D1, D6, D7: D, Diodes_SMD:D_1206, symbol D
- added R11: 0, FSFootprints:SMDNetTie, symbol R
- J1: footprint Connectors_Molex:Molex_MiniFit-JR-5556-02A_2x01x4.20mm_Straight -> Connectors_Molex:Molex_NanoFit_1x02x2.50mm_Straight
- renumbered D1 to D2, D2 to D3, D3 to D4, D4 to D5
Connections:
- net labels added: 12V_SRC_OPTO
Changed lines of the file:
@@
 $EndComp
 $Comp
-L D_Zener D1
+L D_Zener D2
 U 1 1 58A0E5A6
 P 3300 3650
-F 0 "D1" H 3300 3750 50  0000 C CNN
+F 0 "D2" H 3300 3750 50  0000 C CNN
 F 1 "56V Zener" H 3300 3550 50  0000 C CNN
 F 2 "Diodes_THT:D_A-405_P7.62mm_Horizontal" H 3300 3650 50  0001 C CNN
@@
 $EndComp
 $Comp
-L D_Zener D2
+L D_Zener D3
 U 1 1 58A0E67F
 P 3650 3800
-F 0 "D2" H 3650 3900 50  0000 C CNN
+F 0 "D3" H 3650 3900 50  0000 C CNN
 F 1 "12V Zener" H 3650 3700 50  0000 C CNN
 F 2 "Diodes_THT:D_A-405_P7.62mm_Horizontal" H 3650 3800 50  0001 C CNN
@@
 F 0 "J1" H 2200 1100 50  0000 C CNN
 F 1 "TS -> GLV Regulator Jumper" V 2300 950 50  0000 C CNN
-F 2 "Connectors_Molex:Molex_MiniFit-JR-5556-02A_2x01x4.20mm_Straight" H 2200 950 50  0001 C CNN
+F 2 "Connectors_Molex:Molex_NanoFit_1x02x2.50mm_Straight" H 2200 950 50  0001 C CNN
 F 3 "" H 2200 950 50  0000 C CNN
 	1    2200 950
@@
 12V_INDICATOR
 $Comp
-L GND #PWR01
+L GND #PWR1
 U 1 1 58B2C1BD
 P 5300 1450
-F 0 "#PWR01" H 5300 1200 50  0001 C CNN
+F 0 "#PWR1" H 5300 1200 50  0001 C CNN
 F 1 "GND" H 5300 1300 50  0000 C CNN
 F 2 "" H 5300 1450 50  0000 C CNN
@@
 AIRS_FINAL_CHARGER
 $Comp
-L GND #PWR02
+L GND #PWR2
 U 1 1 5959BDAF
 P 5150 6500
-F 0 "#PWR02" H 5150 6250 50  0001 C CNN
+F 0 "#PWR2" H 5150 6250 50  0001 C CNN
 F 1 "GND" H 5150 6350 50  0000 C CNN
 F 2 "" H 5150 6500 50  0001 C CNN
@@
 $EndComp
 $Comp
-L GND #PWR03
+L GND #PWR3
 U 1 1 5959BDF7
 P 5150 7400
-F 0 "#PWR03" H 5150 7150 50  0001 C CNN
+F 0 "#PWR3" H 5150 7150 50  0001 C CNN
 F 1 "GND" H 5150 7250 50  0000 C CNN
 F 2 "" H 5150 7400 50  0001 C CNN
@@
 	0    1    1    0
 $EndComp
-Text Label 5050 3650 0    60   ~ 0
-12V_SRC
+Text Label 6450 5100 0    60   ~ 0
+12V_SRC_OPTO
 Text Notes 4500 7700 0    60   ~ 0
 TS      GLV
@@
 AIRS_FINAL_CHARGER
 $Comp
-L D_Zener D3
+L D_Zener D4
 U 1 1 59A3D9CB
 P 3300 4500
-F 0 "D3" H 3300 4600 50  0000 C CNN
+F 0 "D4" H 3300 4600 50  0000 C CNN
 F 1 "56V Zener" H 3300 4400 50  0000 C CNN
 F 2 "Diodes_THT:D_A-405_P7.62mm_Horizontal" H 3300 4500 50  0001 C CNN
@@
 $EndComp
 $Comp
-L D_Zener D4
+L D_Zener D5
 U 1 1 59A3D9D1
 P 3650 4650
-F 0 "D4" H 3650 4750 50  0000 C CNN
+F 0 "D5" H 3650 4750 50  0000 C CNN
 F 1 "12V Zener" H 3650 4550 50  0000 C CNN
 F 2 "Diodes_THT:D_A-405_P7.62mm_Horizontal" H 3650 4650 50  0001 C CNN
@@
 	0    1    1    0
 $EndComp
-Text Label 5050 4000 0    60   ~ 0
-12V_SRC
-Text Label 5050 4400 0    60   ~ 0
-12V_SRC
-Text Label 5050 4750 0    60   ~ 0
-12V_SRC
 Text Label 5050 4200 0    60   ~ 0
 12V_INDICATOR_CTRL
@@
 Text Label 6400 4700 0    60   ~ 0
 12V_SRC
+$Comp
+L D D1
+U 1 1 5AD81D0E
+P 5200 2300
+F 0 "D1" H 5200 2400 50  0000 C CNN
+F 1 "D" H 5200 2200 50  0000 C CNN
+F 2 "Diodes_SMD:D_1206" H 5200 2300 50  0001 C CNN
+F 3 "" H 5200 2300 50  0001 C CNN
+	1    5200 2300
+	0    1    1    0
+$EndComp
+$Comp
+L D D6
+U 1 1 5AD97C04
+P 5150 6350
+F 0 "D6" H 5150 6450 50  0000 C CNN
+F 1 "D" H 5150 6250 50  0000 C CNN
+F 2 "Diodes_SMD:D_1206" H 5150 6350 50  0001 C CNN
+F 3 "" H 5150 6350 50  0001 C CNN
+	1    5150 6350
+	0    1    1    0
+$EndComp
+$Comp
+L D D7
+U 1 1 5AD980B1
+P 5150 7250
+F 0 "D7" H 5150 7350 50  0000 C CNN
+F 1 "D" H 5150 7150 50  0000 C CNN
+F 2 "Diodes_SMD:D_1206" H 5150 7250 50  0001 C CNN
+F 3 "" H 5150 7250 50  0001 C CNN
+	1    5150 7250
+	0    1    1    0
+$EndComp
+$Comp
+L R R11
+U 1 1 5AD99AB0
+P 6300 5100
+F 0 "R11" V 6380 5100 50  0000 C CNN
+F 1 "0" V 6300 5100 50  0000 C CNN
+F 2 "FSFootprints:SMDNetTie" V 6230 5100 50  0001 C CNN
+F 3 "" H 6300 5100 50  0001 C CNN
+	1    6300 5100
+	0    1    1    0
+$EndComp
+Text Label 6150 5100 2    60   ~ 0
+12V_SRC
+Text Label 5050 4750 0    60   ~ 0
+12V_SRC_OPTO
+Text Label 5050 4400 0    60   ~ 0
+12V_SRC_OPTO
+Text Label 5050 3650 0    60   ~ 0
+12V_SRC_OPTO
+Text Label 5050 4000 0    60   ~ 0
+12V_SRC_OPTO
 $EndSCHEMATC
