File: PEBoardLV/PEBoardLV.sch (KiCad schematic (older format))
At the start: 38 parts, among them J17 STM USB, J6 BSPD Reset, P1 BSPD Test Jumper, U10 4072, U11 LM555N, U2 MCP2515-I/ST, U3 ISO1050, U4 MCP6004, U6 L78S05CV-DG, U7 4071, U9 74HC595

Commit message: Reconfigure dash schematic to take advantage of spare pin
Connections:
- net labels added: BSPD_FLT_LATCHED, LED_BSPD
- wire segments 62 -> 60
- no-connect marks 1 -> 0
Changed lines of the file:
@@
 Text Label 1050 8100 0    60   ~ 0
 AIRS_ACC_OUT
+Text Label 1050 8200 0    60   ~ 0
+AIRS_FINAL
 Text Label 1050 8300 0    60   ~ 0
-AIRS_FINAL
+5V_BMS
 Text Label 1050 8400 0    60   ~ 0
-5V_BMS
-Text Label 1050 8500 0    60   ~ 0
 SIG_CURRENT
+Text Label 1050 8600 0    60   ~ 0
+AIRS_DASH_OUT
 Text Label 1050 8700 0    60   ~ 0
-AIRS_DASH_OUT
-Text Label 1050 8800 0    60   ~ 0
 AIRS_BOTS_OUT
-$Comp
-L +3.3V #PWR?
-U 1 1 59B27500
-P 1700 8900
-F 0 "#PWR?" H 1700 8750 50  0001 C CNN
-F 1 "+3.3V" H 1700 9040 50  0000 C CNN
-F 2 "" H 1700 8900 50  0001 C CNN
-F 3 "" H 1700 8900 50  0001 C CNN
-	1    1700 8900
-	0    1    1    0
-$EndComp
+Text Label 1050 8900 0    60   ~ 0
+SIG_APPS_A
 Text Label 1050 9000 0    60   ~ 0
-SIG_APPS_A
-Text Label 1050 9100 0    60   ~ 0
 GND
 $Comp
 L +3.3V #PWR?
 U 1 1 59B27836
-P 2150 9200
-F 0 "#PWR?" H 2150 9050 50  0001 C CNN
-F 1 "+3.3V" H 2150 9340 50  0000 C CNN
-F 2 "" H 2150 9200 50  0000 C CNN
-F 3 "" H 2150 9200 50  0000 C CNN
-	1    2150 9200
+P 2150 9100
+F 0 "#PWR?" H 2150 8950 50  0001 C CNN
+F 1 "+3.3V" H 2150 9240 50  0000 C CNN
+F 2 "" H 2150 9100 50  0000 C CNN
+F 3 "" H 2150 9100 50  0000 C CNN
+	1    2150 9100
 	0    1    1    0
 $EndComp
@@
 L R R?
 U 1 1 59B2783C
-P 2000 9200
-F 0 "R?" V 2080 9200 50  0000 C CNN
-F 1 "5kR" V 2000 9200 50  0000 C CNN
-F 2 "" V 1930 9200 50  0001 C CNN
-F 3 "" H 2000 9200 50  0000 C CNN
-	1    2000 9200
+P 2000 9100
+F 0 "R?" V 2080 9100 50  0000 C CNN
+F 1 "5kR" V 2000 9100 50  0000 C CNN
+F 2 "" V 1930 9100 50  0001 C CNN
+F 3 "" H 2000 9100 50  0000 C CNN
+	1    2000 9100
 	0    1    1    0
 $EndComp
 Wire Wire Line
-	1050 9200 1850 9200
+	1050 9100 1850 9100
+Text Label 1050 9200 0    60   ~ 0
+SIG_APPS_B
 Text Label 1050 9300 0    60   ~ 0
-SIG_APPS_B
-Text Label 1050 9400 0    60   ~ 0
 GND
-$Comp
-L +3.3V #PWR?
-U 1 1 59B27FDB
-P 1700 9500
-F 0 "#PWR?" H 1700 9350 50  0001 C CNN
-F 1 "+3.3V" H 1700 9640 50  0000 C CNN
-F 2 "" H 1700 9500 50  0001 C CNN
-F 3 "" H 1700 9500 50  0001 C CNN
-	1    1700 9500
-	0    1    1    0
-$EndComp
-Wire Wire Line
-	1050 9500 1700 9500
-Wire Wire Line
-	1700 8900 1050 8900
+Text Label 1050 9500 0    60   ~ 0
+SIG_BSE
 Text Label 1050 9600 0    60   ~ 0
-SIG_BSE
-Text Label 1050 9700 0    60   ~ 0
 GND
 Wire Notes Line
-	550  8600 2550 8600
+	550  8500 2550 8500
 Wire Notes Line
-	550  9700 2550 9700
+	550  9600 2550 9600
+Text Label 1050 9700 0    60   ~ 0
+12V
 Text Label 1050 9800 0    60   ~ 0
-12V
+12V_LVMS
 Text Label 1050 9900 0    60   ~ 0
-12V_LVMS
+CAN_H
 Text Label 1050 10000 0    60   ~ 0
-CAN_H
-Text Label 1050 10100 0    60   ~ 0
 CAN_L
 Text Label 3950 6350 2    60   ~ 0
@@
 Text Label 3950 6450 2    60   ~ 0
 LED_IMD
+Text Label 1050 10100 0    60   ~ 0
+BUTTON_1
 Text Label 1050 10200 0    60   ~ 0
-BUTTON_1
+BUTTON_2
 Text Label 1050 10300 0    60   ~ 0
-BUTTON_2
+BUTTON_3
 Text Label 1050 10400 0    60   ~ 0
-BUTTON_3
+AIRS_DASH_OUT
 Text Label 1050 10500 0    60   ~ 0
-AIRS_DASH_OUT
+LED_AMS
 Text Label 1050 10600 0    60   ~ 0
-LED_AMS
-Text Label 1050 10700 0    60   ~ 0
 LED_IMD
 Text Label 1050 10800 0    60   ~ 0
@@
 	0    1    1    0
 $EndComp
-Text Label 1050 8600 0    60   ~ 0
+Text Label 1050 8500 0    60   ~ 0
 GND
 $Comp
@@
 Text Notes 1950 8500 0    60   ~ 0
 To Accumulator
+Text Notes 2100 9600 0    60   ~ 0
+To Pedals
 Text Notes 2100 9700 0    60   ~ 0
-To Pedals
-Text Notes 2100 9800 0    60   ~ 0
 To Dash
 $Comp
@@
 	-1   0    0    -1
 $EndComp
-NoConn ~ 1050 8200
 Text Label 1100 4500 0    60   ~ 0
 AIRS_FINAL
 Wire Wire Line
 	2150 4500 1100 4500
+Text Label 1050 10700 0    60   ~ 0
+LED_BSPD
+Text Label 1050 8800 0    60   ~ 0
+3.3V
+Text Label 1050 9400 0    60   ~ 0
+3.3V
+Text Label 3950 6550 2    60   ~ 0
+LED_BSPD
+Text Label 15800 1350 1    60   ~ 0
+BSPD_FLT_LATCHED
+$Comp
+L GND #PWR?
+U 1 1 5A525D9A
+P 15800 2450
+F 0 "#PWR?" H 15800 2200 50  0001 C CNN
+F 1 "GND" H 15800 2300 50  0000 C CNN
+F 2 "" H 15800 2450 50  0001 C CNN
+F 3 "" H 15800 2450 50  0001 C CNN
+	1    15800 2450
+	1    0    0    -1
+$EndComp
 $EndSCHEMATC

Commit message: Added charger control pins and organized optos
Parts:
- R?: value 5kR -> 2.2k
Changed lines of the file:
@@
 LIBS:contrib
 LIBS:valves
-LIBS:PEBoardLV-cache
 EELAYER 25 0
 EELAYER END
@@
 P 2000 9100
 F 0 "R?" V 2080 9100 50  0000 C CNN
-F 1 "5kR" V 2000 9100 50  0000 C CNN
+F 1 "2.2k" V 2000 9100 50  0000 C CNN
 F 2 "" V 1930 9100 50  0001 C CNN
 F 3 "" H 2000 9100 50  0000 C CNN

Commit message: Begin PE/dash footprints, continue with accumulator footprints
Parts:
- C1, C5, C6: renamed from C?; footprint (none) -> Capacitors_THT:CP_Radial_D8.0mm_P2.50mm
- C2: renamed from C3; footprint (none) -> Capacitors_THT:CP_Radial_D8.0mm_P2.50mm
- C3: renamed from C4; footprint (none) -> Capacitors_THT:CP_Radial_D8.0mm_P2.50mm
- C4: renamed from C2; footprint (none) -> Capacitors_THT:CP_Radial_D8.0mm_P2.50mm
- J1, J3, J6: renamed from J?; footprint (none) -> Connectors_Molex:Molex_NanoFit_1x02x2.50mm_Straight
- J2: renamed from J?; footprint (none) -> Connectors_Molex:Molex_NanoFit_1x06x2.50mm_Straight
- J4: renamed from J?; footprint (none) -> Connectors_Molex:Molex_NanoFit_1x05x2.50mm_Straight
- J5: renamed from J17; footprint (none) -> Connectors_Molex:Molex_NanoFit_1x04x2.50mm_Straight
- J7: renamed from J?; footprint (none) -> Connectors_Molex:Molex_NanoFit_2x04x2.50mm_Straight
- J9: renamed from J?; footprint (none) -> FSFootprints:Ampseal - 35 pin
- R1: renamed from R7; footprint (none) -> Resistors_THT:R_Axial_DIN0411_L9.9mm_D3.6mm_P12.70mm_Horizontal
- R10, R7: renamed from R?; footprint (none) -> Resistors_THT:R_Axial_DIN0411_L9.9mm_D3.6mm_P12.70mm_Horizontal
- R2: renamed from R6; footprint (none) -> Resistors_THT:R_Axial_DIN0411_L9.9mm_D3.6mm_P12.70mm_Horizontal
- R3: renamed from R2; footprint (none) -> Resistors_THT:R_Axial_DIN0411_L9.9mm_D3.6mm_P12.70mm_Horizontal
- R4: renamed from R1; footprint (none) -> Resistors_THT:R_Axial_DIN0411_L9.9mm_D3.6mm_P12.70mm_Horizontal
- R5: renamed from R4; footprint (none) -> Resistors_THT:R_Axial_DIN0411_L9.9mm_D3.6mm_P12.70mm_Horizontal
- R6: renamed from R5; footprint (none) -> Resistors_THT:R_Axial_DIN0411_L9.9mm_D3.6mm_P12.70mm_Horizontal
- R8: renamed from R13; footprint (none) -> Resistors_THT:R_Axial_DIN0411_L9.9mm_D3.6mm_P12.70mm_Horizontal
- R9: renamed from R14; footprint (none) -> Resistors_THT:R_Axial_DIN0411_L9.9mm_D3.6mm_P12.70mm_Horizontal
- RV1: footprint (none) -> Potentiometers:Potentiometer_Trimmer-EVM3E
- U1: renamed from U4; footprint (none) -> Housings_DIP:DIP-14_W7.62mm
- U2: renamed from U10; footprint Housings_DIP:DIP-12_W7.62mm -> Housings_DIP:DIP-14_W7.62mm
- U3: renamed from U7; footprint (none) -> Housings_DIP:DIP-8_W7.62mm
- U4: renamed from U?; footprint (none) -> FSFootprints:DE1A1B-L2-12V
- gave numbers to parts that had none: 2
- renumbered J6 to J8, U4 to U1, U9 to U5, U11 to U6, U3 to U7, U2 to U8, U6 to U9

Commit message: WIP: Added all parts for dual CAN ECU and wired some components
Parts:
- removed U8: MCP2515-I/ST, Housings_DIP:DIP-18_W7.62mm, symbol MCP2515-I/ST
- added C?: 2.2uF, symbol C
- added C?: 4.7uF, symbol C
- added C? (x2): 0.47uF, Capacitors_THT:CP_Radial_D8.0mm_P2.50mm, symbol C
- added D?: D_TVS_x2_AAC, symbol D_TVS_x2_AAC
- added FL?: EMI_Filter_CommonMode, symbol EMI_Filter_CommonMode
- added U?: 5V-1A, symbol uA7805
- added U?: 3.3V-1A, symbol uA7805
- added U?: STM32F405, LQFP-64, symbol STM32F405
- added U?: ISO1050, SMD_Packages:DIP-8_SMD, symbol ISO1050
- added Y?: 8MHz, symbol Crystal_GND24
Connections:
- net labels added: CAN_H_GLV, CAN_H_TS, CAN_L_GLV, CAN_L_TS, CAN_RX_GLV, CAN_RX_TS, CAN_TX_GLV, CAN_TX_TS, XTAL
- wire segments 60 -> 64

Commit message: Completed dual CAN ECU
Parts:
- removed C?: 2.2uF, symbol C
- removed C?: 4.7uF, symbol C
- removed J5: STM USB, Connectors_Molex:Molex_NanoFit_1x04x2.50mm_Straight, symbol Conn_01x04
- removed U10: stm_nucleo_F303K8, arduino:arduino_mini, symbol stm_nucleo_F303K8
- removed U?: 5V-1A, symbol uA7805
- removed U?: ISO1050, SMD_Packages:DIP-8_SMD, symbol ISO1050
- added C? (x2): 2.2uF, symbol C
- added C?: 0.1uF, Capacitors_THT:CP_Radial_D8.0mm_P2.50mm, symbol CP
- added C? (x6): 0.1uF, symbol C
- added C?: 4.7uF, symbol C
- added D? (x3): LED, symbol LED
- added R? (x3): 330, Resistors_THT:R_Axial_DIN0411_L9.9mm_D3.6mm_P12.70mm_Horizontal, symbol R
- U?: value 3.3V-1A -> NCP1117DT33RKG
Connections:
- net labels added: STATUS_LED_1, STATUS_LED_2, STATUS_LED_3, SWCLK, SWDIO, UART_RX, UART_TX, VCAP_1, VCAP_2
- net labels removed: CAN_H_GLV, CAN_H_TS, CAN_L_GLV, CAN_L_TS, CAN_RX, CAN_TX, SPI_MISO, SPI_MOSI, SPI_SCLK, SPI_SSEL
- wire segments 64 -> 91

Commit message: Moved ECU status LEDs to be on the same port
Connections:
- wire segments 91 -> 109
Changed lines of the file:
@@
 Text Label 6750 9600 0    60   ~ 0
 SIG_RTDS
-Text Label 3850 10000 2    60   ~ 0
+Text Label 4100 10000 2    60   ~ 0
 BUTTON_1
 Text Label 6750 10200 0    60   ~ 0
@@
 L GND #PWR?
 U 1 1 5A900EB8
-P 4000 10200
-F 0 "#PWR?" H 4000 9950 50  0001 C CNN
-F 1 "GND" H 4000 10050 50  0000 C CNN
-F 2 "" H 4000 10200 50  0001 C CNN
-F 3 "" H 4000 10200 50  0001 C CNN
-	1    4000 10200
+P 4150 10200
+F 0 "#PWR?" H 4150 9950 50  0001 C CNN
+F 1 "GND" H 4150 10050 50  0000 C CNN
+F 2 "" H 4150 10200 50  0001 C CNN
+F 3 "" H 4150 10200 50  0001 C CNN
+	1    4150 10200
 	1    0    0    -1
 $EndComp
@@
 L +3.3V #PWR?
 U 1 1 5A9014C4
-P 4150 9850
-F 0 "#PWR?" H 4150 9700 50  0001 C CNN
-F 1 "+3.3V" H 4150 9990 50  0000 C CNN
-F 2 "" H 4150 9850 50  0001 C CNN
-F 3 "" H 4150 9850 50  0001 C CNN
-	1    4150 9850
+P 3600 9850
+F 0 "#PWR?" H 3600 9700 50  0001 C CNN
+F 1 "+3.3V" H 3600 9990 50  0000 C CNN
+F 2 "" H 3600 9850 50  0001 C CNN
+F 3 "" H 3600 9850 50  0001 C CNN
+	1    3600 9850
 	1    0    0    -1
 $EndComp
@@
 	4400 2650 4400 2800
 Wire Wire Line
-	4400 2800 5200 2800
+	4400 2800 4700 2800
+Wire Wire Line
+	4700 2800 5200 2800
 Connection ~ 4700 2800
 Wire Wire Line
@@
 	1050 7600 1550 7600
 Wire Wire Line
-	14200 5400 14500 5400
+	14200 5400 14300 5400
+Wire Wire Line
+	14300 5400 14400 5400
+Wire Wire Line
+	14400 5400 14500 5400
 Connection ~ 14400 5400
 Connection ~ 14300 5400
@@
 	14800 4800 14800 4700
 Wire Wire Line
-	4550 5750 5600 5750
+	4550 5750 4950 5750
+Wire Wire Line
+	4950 5750 5350 5750
+Wire Wire Line
+	5350 5750 5600 5750
 Connection ~ 4950 5750
 Wire Wire Line
@@
 	2150 4500 1100 4500
 Wire Wire Line
-	3350 5750 4150 5750
+	3350 5750 3750 5750
+Wire Wire Line
+	3750 5750 4150 5750
 Connection ~ 3750 5750
 Wire Wire Line
@@
 	3700 8900 4500 8900
 Wire Wire Line
-	4000 9900 4500 9900
-Wire Wire Line
-	4150 10200 4500 10200
-Wire Wire Line
-	4150 9850 4150 10200
+	4150 9900 4500 9900
+Wire Wire Line
+	3600 10200 4500 10200
+Wire Wire Line
+	3600 9850 3600 10200
 Wire Wire Line
 	7150 8700 6750 8700
@@
 	7450 7500 6750 7500
 Wire Wire Line
-	8500 7550 8900 7550
+	8500 7550 8700 7550
+Wire Wire Line
+	8700 7550 8900 7550
 Wire Wire Line
 	8700 7550 8700 7600
@@
 Connection ~ 5350 5750
 Wire Wire Line
-	9450 7550 10950 7550
+	9450 7550 9700 7550
+Wire Wire Line
+	9700 7550 9950 7550
+Wire Wire Line
+	9950 7550 10200 7550
+Wire Wire Line
+	10200 7550 10450 7550
+Wire Wire Line
+	10450 7550 10700 7550
+Wire Wire Line
+	10700 7550 10950 7550
 Connection ~ 9700 7550
 Connection ~ 9950 7550
@@
 	10200 7550 10200 7600
 Wire Wire Line
-	9450 7250 10950 7250
+	9450 7250 9700 7250
+Wire Wire Line
+	9700 7250 9950 7250
+Wire Wire Line
+	9950 7250 10200 7250
+Wire Wire Line
+	10200 7250 10450 7250
+Wire Wire Line
+	10450 7250 10700 7250
+Wire Wire Line
+	10700 7250 10950 7250
 Connection ~ 9700 7250
 Connection ~ 9950 7250
@@
 	9400 5850 9400 5950
 Wire Wire Line
-	10050 5650 10900 5650
+	10050 5650 10750 5650
+Wire Wire Line
+	10750 5650 10900 5650
 $Comp
 L GND #PWR?
@@
 Text Label 6750 10000 0    60   ~ 0
 BSPD_FLT_LATCHED
-Text Label 6750 9700 0    60   ~ 0
+Text Label 4500 9800 2    60   ~ 0
 STATUS_LED_1
-Text Label 6750 9800 0    60   ~ 0
+Text Label 4500 9700 2    60   ~ 0
 STATUS_LED_2
-Text Label 6750 9900 0    60   ~ 0
+Text Label 4500 9600 2    60   ~ 0
 STATUS_LED_3
 $Comp
@@
 $EndComp
 Wire Wire Line
-	4000 9900 4000 10200
-Wire Wire Line
-	4500 10000 3850 10000
+	4150 9900 4150 10200
+Wire Wire Line
+	4500 10000 4100 10000
 Text Label 6750 8400 0    60   ~ 0
 UART_TX
