File: PEBoardLV/PEBoardLV.sch (KiCad schematic (older format))
At the start: 64 parts, among them J1 BSPD Test Jumper, J10 SWD Header, J11 ECU Debug Connector, J12 To TSAL, J2 Beam Interlock, J3 To HV Interlocks, J4 To Left Panel, J5 To Right Panel, J6 To Brake Light, J7 To PE HV, J8 BSPD Reset, J9 Main LV Connector, U1 MCP6004, U10 ISO1050, U11 STM32F405, U2 4072, U3 4071, U4 DE1A1B-L2-12V, U5 74HC595, U6 LM555N, U7 SN754410, U8 NCP1117DT33RKG, U9 L78S05CV-DG, Y1 8MHz

Commit message: PE LV Board will be ready to go once routed
Had to make a couple changes to net size to pass Bay Area Circuit's DFM
Parts:
- added J12: Extra Pin Header, Pin_Headers:Pin_Header_Straight_2x04_Pitch2.54mm, symbol Conn_01x08
- renumbered J12 to J13
Connections:
- net labels added: AIRS_3PHASE1_OUT, PA4, PA5, PA7, PC0, PC1, PC2, PC3, PC4
- net labels removed: SIG_BRAKE, SIG_TORQUEA, SIG_TORQUEB
- no-connect marks 25 -> 18

Commit message: V2 of PE LV PCB
Parts:
- removed FL1: EMI_Filter_CommonMode, Inductors_SMD:L_CommonMode_Wuerth_WE-SL2, symbol EMI_Filter_CommonMode
- removed J11: ECU Debug Connector, FSFootprints:Ampseal-776276-1, symbol Conn_01x08
- removed J12: Extra Pin Header, Pin_Headers:Pin_Header_Straight_2x04_Pitch2.54mm, symbol Conn_01x08
- added C9: CP, Capacitors_THT:CP_Radial_D5.0mm_P2.50mm, symbol CP
- added FL1: EMI_Choke, FSFootprints:L_CommonMode_Choke, symbol EMI_Choke
- added J11: SWD Header, Pin_Headers:Pin_Header_Straight_1x06_Pitch2.54mm, symbol Conn_01x06
- added J12: Extra Pin Header, Pin_Headers:Pin_Header_Straight_1x04_Pitch2.54mm, symbol Conn_01x04
- added J13: CAN Header, Pin_Headers:Pin_Header_Straight_1x03_Pitch2.54mm, symbol Conn_01x03
- added J14: UART Header, Pin_Headers:Pin_Header_Straight_1x02_Pitch2.54mm, symbol Conn_01x02
- added R14: 120, Resistors_THT:R_Axial_DIN0207_L6.3mm_D2.5mm_P10.16mm_Horizontal, symbol R
- J10: value SWD Header -> ECU Debug Connector; footprint Pin_Headers:Pin_Header_Straight_1x08_Pitch2.54mm -> FSFootprints:Ampseal-776276-1
- R1, R10, R11, R12, R13, R2, R3, R4, R5, R6, R7, R8, R9: footprint Resistors_THT:R_Axial_DIN0411_L9.9mm_D3.6mm_P12.70mm_Horizontal -> Resistors_THT:R_Axial_DIN0207_L6.3mm_D2.5mm_P10.16mm_Horizontal
- renumbered C9 to C10, C10 to C11, C11 to C12, C12 to C13, C13 to C14, C14 to C15, C15 to C16, C16 to C17, C17 to C18, C18 to C19, C19 to C20, J13 to J15
Connections:
- net labels added: CAN_H_PRE, CAN_L_PRE
- wire segments 90 -> 95

Commit message: Route PE LV with 4 layers, using center layers as power planes
Connections:
- net labels removed: 5V_BMS
- wire segments 95 -> 96
- no-connect marks 18 -> 19
Changed lines of the file:
@@
 $EndComp
 Text Label 4900 1200 2    60   ~ 0
-5V_BMS
+5V
 Text Notes 5050 750  0    60   ~ 0
 Current Signal Comparator:\nIf Current Signal < 2.6V
@@
 Text Label 3900 5750 3    60   ~ 0
 GND
-Text Label 4700 2500 0    60   ~ 0
-3.3V
 Text Label 1050 6850 0    60   ~ 0
 BSPD_RESET
@@
 $EndComp
 Text Label 3850 1500 0    60   ~ 0
-5V_BMS
+5V
 $Comp
 L GND #PWR027
@@
 Text Label 1050 8200 0    60   ~ 0
 AIRS_FINAL
-Text Label 1050 8300 0    60   ~ 0
-5V_BMS
 Text Label 1050 8400 0    60   ~ 0
 SIG_CURRENT
@@
 	10100 1500 10250 1500
 Wire Wire Line
-	9800 1950 10250 1950
-Wire Wire Line
-	10250 1950 10250 2350
-Wire Wire Line
-	9800 2050 10150 2050
-Wire Wire Line
-	10150 2050 10150 2450
-Wire Wire Line
-	10150 2450 10250 2450
-Wire Wire Line
-	9800 2150 10050 2150
-Wire Wire Line
-	10050 2150 10050 2550
-Wire Wire Line
-	10050 2550 10250 2550
-Wire Wire Line
-	10250 2650 9950 2650
-Wire Wire Line
-	9950 2650 9950 2250
+	10000 2450 10250 2450
 Wire Wire Line
 	9950 2250 9800 2250
@@
 Text Label 8800 10400 2    60   ~ 0
 NRST
+Text Label 11250 10500 2    60   ~ 0
+UART_RX
 Text Label 11250 10400 2    60   ~ 0
-UART_RX
-Text Label 11250 10500 2    60   ~ 0
 UART_TX
 $Comp
@@
 	1    0    0    -1
 $EndComp
+Text Label 8100 10500 2    60   ~ 0
+UART_RX
 Text Label 8100 10400 2    60   ~ 0
-UART_RX
-Text Label 8100 10500 2    60   ~ 0
 UART_TX
 Wire Wire Line
@@
 	1    0    0    -1
 $EndComp
+Wire Wire Line
+	9950 2250 9950 2350
+Wire Wire Line
+	9950 2350 10250 2350
+Wire Wire Line
+	9800 2150 10000 2150
+Wire Wire Line
+	10000 2150 10000 2450
+Wire Wire Line
+	9800 2050 10050 2050
+Wire Wire Line
+	10050 2050 10050 2550
+Wire Wire Line
+	10050 2550 10250 2550
+Wire Wire Line
+	9800 1950 10100 1950
+Wire Wire Line
+	10100 1950 10100 2650
+Wire Wire Line
+	10100 2650 10250 2650
+$Comp
+L +5V #PWR089
+U 1 1 5A993C9C
+P 4700 2500
+F 0 "#PWR089" H 4700 2350 50  0001 C CNN
+F 1 "+5V" H 4700 2640 50  0000 C CNN
+F 2 "" H 4700 2500 50  0000 C CNN
+F 3 "" H 4700 2500 50  0000 C CNN
+	1    4700 2500
+	1    0    0    -1
+$EndComp
+Connection ~ 4700 2500
+NoConn ~ 1050 8300
 $EndSCHEMATC

Commit message: Revise boards based on design review
Parts:
- J9: footprint FSFootprints:Ampseal - 35 pin -> FSFootprints:Ampseal-776231
Connections:
- no-connect marks 19 -> 20
Changed lines of the file:
@@
 F 0 "J9" H 850 11000 50  0000 C CNN
 F 1 "Main LV Connector" V 950 9200 50  0000 C CNN
-F 2 "FSFootprints:Ampseal - 35 pin" H 850 9200 50  0001 C CNN
+F 2 "FSFootprints:Ampseal-776231" H 850 9200 50  0001 C CNN
 F 3 "" H 850 9200 50  0001 C CNN
 	1    850  9200
@@
 F 3 "" H 1100 4600 50  0001 C CNN
 	1    1100 4600
-	1    0    0    -1
+	0    -1   -1   0
 $EndComp
 $Comp
@@
 Connection ~ 4700 2500
 NoConn ~ 1050 8300
+NoConn ~ 1100 4700
 $EndSCHEMATC

Commit message: edit PCBs based on actual parts that have arrived
Parts:
- C14, C15, C16, C17, C18, C19: footprint Capacitors_SMD:C_0402 -> Capacitors_SMD:C_0603_HandSoldering
- D1: footprint TO_SOT_Packages_SMD:SOT-23 -> TO_SOT_Packages_SMD:SOT-23_Handsoldering
- U10: footprint SMD_Packages:DIP-8_SMD -> Housings_DIP:DIP-8_W8.89mm_SMDSocket_LongPads
Changed lines of the file:
@@
 F 0 "U10" H 9050 5750 60  0000 C CNN
 F 1 "ISO1050" H 8750 5750 60  0000 C CNN
-F 2 "SMD_Packages:DIP-8_SMD" H 8800 5050 60  0001 C CNN
+F 2 "Housings_DIP:DIP-8_W8.89mm_SMDSocket_LongPads" H 8800 5050 60  0001 C CNN
 F 3 "" H 8750 5750 60  0000 C CNN
 	1    8800 5750
@@
 F 0 "D1" H 10400 5475 50  0000 C CNN
 F 1 "D_TVS_x2_AAC" H 10400 5400 50  0000 C CNN
-F 2 "TO_SOT_Packages_SMD:SOT-23" H 10250 5300 50  0001 C CNN
+F 2 "TO_SOT_Packages_SMD:SOT-23_Handsoldering" H 10250 5300 50  0001 C CNN
 F 3 "" H 10250 5300 50  0001 C CNN
 	1    10400 5300
@@
 F 0 "C14" H 9475 7500 50  0000 L CNN
 F 1 "0.1uF" H 9475 7300 50  0000 L CNN
-F 2 "Capacitors_SMD:C_0402" H 9488 7250 50  0001 C CNN
+F 2 "Capacitors_SMD:C_0603_HandSoldering" H 9488 7250 50  0001 C CNN
 F 3 "" H 9450 7400 50  0001 C CNN
 	1    9450 7400
@@
 F 0 "C15" H 9725 7500 50  0000 L CNN
 F 1 "0.1uF" H 9725 7300 50  0000 L CNN
-F 2 "Capacitors_SMD:C_0402" H 9738 7250 50  0001 C CNN
+F 2 "Capacitors_SMD:C_0603_HandSoldering" H 9738 7250 50  0001 C CNN
 F 3 "" H 9700 7400 50  0001 C CNN
 	1    9700 7400
@@
 F 0 "C16" H 9975 7500 50  0000 L CNN
 F 1 "0.1uF" H 9975 7300 50  0000 L CNN
-F 2 "Capacitors_SMD:C_0402" H 9988 7250 50  0001 C CNN
+F 2 "Capacitors_SMD:C_0603_HandSoldering" H 9988 7250 50  0001 C CNN
 F 3 "" H 9950 7400 50  0001 C CNN
 	1    9950 7400
@@
 F 0 "C17" H 10225 7500 50  0000 L CNN
 F 1 "0.1uF" H 10225 7300 50  0000 L CNN
-F 2 "Capacitors_SMD:C_0402" H 10238 7250 50  0001 C CNN
+F 2 "Capacitors_SMD:C_0603_HandSoldering" H 10238 7250 50  0001 C CNN
 F 3 "" H 10200 7400 50  0001 C CNN
 	1    10200 7400
@@
 F 0 "C18" H 10475 7500 50  0000 L CNN
 F 1 "0.1uF" H 10475 7300 50  0000 L CNN
-F 2 "Capacitors_SMD:C_0402" H 10488 7250 50  0001 C CNN
+F 2 "Capacitors_SMD:C_0603_HandSoldering" H 10488 7250 50  0001 C CNN
 F 3 "" H 10450 7400 50  0001 C CNN
 	1    10450 7400
@@
 F 0 "C19" H 10725 7500 50  0000 L CNN
 F 1 "0.1uF" H 10725 7300 50  0000 L CNN
-F 2 "Capacitors_SMD:C_0402" H 10738 7250 50  0001 C CNN
+F 2 "Capacitors_SMD:C_0603_HandSoldering" H 10738 7250 50  0001 C CNN
 F 3 "" H 10700 7400 50  0001 C CNN
 	1    10700 7400

Commit message: prepare to re-send PE LV board
Parts:
- C14, C15, C16, C17, C18, C19: footprint Capacitors_SMD:C_0603_HandSoldering -> FSFootprints:C_0402_HandSoldering
- U11: footprint Housings_QFP:LQFP-64_10x10mm_Pitch0.5mm -> FSFootprints:LQFP-64_10x10mm_Pitch0.5mm_HandSoldering
Changed lines of the file:
@@
 F 0 "U11" H 5700 7500 60  0000 C CNN
 F 1 "STM32F405" H 5700 7400 60  0000 C CNN
-F 2 "Housings_QFP:LQFP-64_10x10mm_Pitch0.5mm" H 5700 7200 60  0001 C CNN
+F 2 "FSFootprints:LQFP-64_10x10mm_Pitch0.5mm_HandSoldering" H 5700 7200 60  0001 C CNN
 F 3 "" H 4500 7100 60  0000 C CNN
 	1    4500 7100
@@
 F 0 "C14" H 9475 7500 50  0000 L CNN
 F 1 "0.1uF" H 9475 7300 50  0000 L CNN
-F 2 "Capacitors_SMD:C_0603_HandSoldering" H 9488 7250 50  0001 C CNN
+F 2 "FSFootprints:C_0402_HandSoldering" H 9488 7250 50  0001 C CNN
 F 3 "" H 9450 7400 50  0001 C CNN
 	1    9450 7400
@@
 F 0 "C15" H 9725 7500 50  0000 L CNN
 F 1 "0.1uF" H 9725 7300 50  0000 L CNN
-F 2 "Capacitors_SMD:C_0603_HandSoldering" H 9738 7250 50  0001 C CNN
+F 2 "FSFootprints:C_0402_HandSoldering" H 9738 7250 50  0001 C CNN
 F 3 "" H 9700 7400 50  0001 C CNN
 	1    9700 7400
@@
 F 0 "C16" H 9975 7500 50  0000 L CNN
 F 1 "0.1uF" H 9975 7300 50  0000 L CNN
-F 2 "Capacitors_SMD:C_0603_HandSoldering" H 9988 7250 50  0001 C CNN
+F 2 "FSFootprints:C_0402_HandSoldering" H 9988 7250 50  0001 C CNN
 F 3 "" H 9950 7400 50  0001 C CNN
 	1    9950 7400
@@
 F 0 "C17" H 10225 7500 50  0000 L CNN
 F 1 "0.1uF" H 10225 7300 50  0000 L CNN
-F 2 "Capacitors_SMD:C_0603_HandSoldering" H 10238 7250 50  0001 C CNN
+F 2 "FSFootprints:C_0402_HandSoldering" H 10238 7250 50  0001 C CNN
 F 3 "" H 10200 7400 50  0001 C CNN
 	1    10200 7400
@@
 F 0 "C18" H 10475 7500 50  0000 L CNN
 F 1 "0.1uF" H 10475 7300 50  0000 L CNN
-F 2 "Capacitors_SMD:C_0603_HandSoldering" H 10488 7250 50  0001 C CNN
+F 2 "FSFootprints:C_0402_HandSoldering" H 10488 7250 50  0001 C CNN
 F 3 "" H 10450 7400 50  0001 C CNN
 	1    10450 7400
@@
 F 0 "C19" H 10725 7500 50  0000 L CNN
 F 1 "0.1uF" H 10725 7300 50  0000 L CNN
-F 2 "Capacitors_SMD:C_0603_HandSoldering" H 10738 7250 50  0001 C CNN
+F 2 "FSFootprints:C_0402_HandSoldering" H 10738 7250 50  0001 C CNN
 F 3 "" H 10700 7400 50  0001 C CNN
 	1    10700 7400

Commit message: update for sending out second round of PE LV pcb
Parts:
- C14, C15, C16, C17, C18, C19: footprint FSFootprints:C_0402_HandSoldering -> Capacitors_SMD:C_0805_HandSoldering
Changed lines of the file:
@@
 F 0 "C14" H 9475 7500 50  0000 L CNN
 F 1 "0.1uF" H 9475 7300 50  0000 L CNN
-F 2 "FSFootprints:C_0402_HandSoldering" H 9488 7250 50  0001 C CNN
+F 2 "Capacitors_SMD:C_0805_HandSoldering" H 9488 7250 50  0001 C CNN
 F 3 "" H 9450 7400 50  0001 C CNN
 	1    9450 7400
@@
 F 0 "C15" H 9725 7500 50  0000 L CNN
 F 1 "0.1uF" H 9725 7300 50  0000 L CNN
-F 2 "FSFootprints:C_0402_HandSoldering" H 9738 7250 50  0001 C CNN
+F 2 "Capacitors_SMD:C_0805_HandSoldering" H 9738 7250 50  0001 C CNN
 F 3 "" H 9700 7400 50  0001 C CNN
 	1    9700 7400
@@
 F 0 "C16" H 9975 7500 50  0000 L CNN
 F 1 "0.1uF" H 9975 7300 50  0000 L CNN
-F 2 "FSFootprints:C_0402_HandSoldering" H 9988 7250 50  0001 C CNN
+F 2 "Capacitors_SMD:C_0805_HandSoldering" H 9988 7250 50  0001 C CNN
 F 3 "" H 9950 7400 50  0001 C CNN
 	1    9950 7400
@@
 F 0 "C17" H 10225 7500 50  0000 L CNN
 F 1 "0.1uF" H 10225 7300 50  0000 L CNN
-F 2 "FSFootprints:C_0402_HandSoldering" H 10238 7250 50  0001 C CNN
+F 2 "Capacitors_SMD:C_0805_HandSoldering" H 10238 7250 50  0001 C CNN
 F 3 "" H 10200 7400 50  0001 C CNN
 	1    10200 7400
@@
 F 0 "C18" H 10475 7500 50  0000 L CNN
 F 1 "0.1uF" H 10475 7300 50  0000 L CNN
-F 2 "FSFootprints:C_0402_HandSoldering" H 10488 7250 50  0001 C CNN
+F 2 "Capacitors_SMD:C_0805_HandSoldering" H 10488 7250 50  0001 C CNN
 F 3 "" H 10450 7400 50  0001 C CNN
 	1    10450 7400
@@
 F 0 "C19" H 10725 7500 50  0000 L CNN
 F 1 "0.1uF" H 10725 7300 50  0000 L CNN
-F 2 "FSFootprints:C_0402_HandSoldering" H 10738 7250 50  0001 C CNN
+F 2 "Capacitors_SMD:C_0805_HandSoldering" H 10738 7250 50  0001 C CNN
 F 3 "" H 10700 7400 50  0001 C CNN
 	1    10700 7400

Commit message: tweak boards slightly
Parts:
- C1, C2, C6, C7, C8, C9: footprint Capacitors_THT:CP_Radial_D5.0mm_P2.50mm -> Capacitors_THT:C_Disc_D3.0mm_W1.6mm_P2.50mm
Connections:
- net labels added: PC5
- no-connect marks 20 -> 19
Changed lines of the file:
@@
 F 0 "C8" H 10425 4100 50  0000 L CNN
 F 1 "CP" H 10425 3900 50  0000 L CNN
-F 2 "Capacitors_THT:CP_Radial_D5.0mm_P2.50mm" H 10438 3850 50  0001 C CNN
+F 2 "Capacitors_THT:C_Disc_D3.0mm_W1.6mm_P2.50mm" H 10438 3850 50  0001 C CNN
 F 3 "" H 10400 4000 50  0000 C CNN
 	1    10400 4000
@@
 F 0 "C1" H 6825 2850 50  0000 L CNN
 F 1 "CP" H 6825 2650 50  0000 L CNN
-F 2 "Capacitors_THT:CP_Radial_D5.0mm_P2.50mm" H 6838 2600 50  0001 C CNN
+F 2 "Capacitors_THT:C_Disc_D3.0mm_W1.6mm_P2.50mm" H 6838 2600 50  0001 C CNN
 F 3 "" H 6800 2750 50  0001 C CNN
 	1    6800 2750
@@
 F 0 "C6" H 13825 4050 50  0000 L CNN
 F 1 "CP" H 13825 3850 50  0000 L CNN
-F 2 "Capacitors_THT:CP_Radial_D5.0mm_P2.50mm" H 13838 3800 50  0001 C CNN
+F 2 "Capacitors_THT:C_Disc_D3.0mm_W1.6mm_P2.50mm" H 13838 3800 50  0001 C CNN
 F 3 "" H 13800 3950 50  0001 C CNN
 	1    13800 3950
@@
 F 0 "C7" H 14575 4050 50  0000 L CNN
 F 1 "CP" H 14575 3850 50  0000 L CNN
-F 2 "Capacitors_THT:CP_Radial_D5.0mm_P2.50mm" H 14588 3800 50  0001 C CNN
+F 2 "Capacitors_THT:C_Disc_D3.0mm_W1.6mm_P2.50mm" H 14588 3800 50  0001 C CNN
 F 3 "" H 14550 3950 50  0001 C CNN
 	1    14550 3950
@@
 F 0 "C2" H 9675 3150 50  0000 L CNN
 F 1 "CP" H 9675 2950 50  0000 L CNN
-F 2 "Capacitors_THT:CP_Radial_D5.0mm_P2.50mm" H 9688 2900 50  0001 C CNN
+F 2 "Capacitors_THT:C_Disc_D3.0mm_W1.6mm_P2.50mm" H 9688 2900 50  0001 C CNN
 F 3 "" H 9650 3050 50  0001 C CNN
 	1    9650 3050
@@
 NoConn ~ 4500 7300
 NoConn ~ 4500 7200
-NoConn ~ 4500 9500
 NoConn ~ 4500 8400
 NoConn ~ 4500 7600
@@
 PC4
 Text Label 9450 10200 2    60   ~ 0
-PA4
+PA7
 Text Label 9450 10300 2    60   ~ 0
-PA5
-Text Label 9450 10400 2    60   ~ 0
-PA7
-Text Label 9450 10500 2    60   ~ 0
 PC4
 NoConn ~ 9800 2450
@@
 F 0 "C9" H 9075 5350 50  0000 L CNN
 F 1 "CP" H 9075 5150 50  0000 L CNN
-F 2 "Capacitors_THT:CP_Radial_D5.0mm_P2.50mm" H 9088 5100 50  0001 C CNN
+F 2 "Capacitors_THT:C_Disc_D3.0mm_W1.6mm_P2.50mm" H 9088 5100 50  0001 C CNN
 F 3 "" H 9050 5250 50  0001 C CNN
 	1    9050 5250
@@
 NoConn ~ 1050 8300
 NoConn ~ 1100 4700
+Text Label 4500 9500 2    60   ~ 0
+PC5
+Text Label 9450 10400 2    60   ~ 0
+PC5
+Text Label 9450 10500 2    60   ~ 0
+GND
 $EndSCHEMATC
