File: ChargerSwitchbox/ChargerSwitchbox.sch (KiCad schematic (older format))
At the start: 13 parts, among them J1 Charger Control, J2 Charger LV, J3 Charger Current Direct, J4 Estop Connector, J5 Charger Current Out, J6 Connector Interlock, U1 PS2501-1, U2 G2RL-1A-E, U3 G2RL-1A-E

Commit message: Revise boards based on design review
Parts:
- added F1: Fuse, Fuse_Holders_and_Fuses:Fuseholder5x20_vert_closed_Bulgin_FX0456, symbol Fuse
- R2: footprint Oddities:NetTie-I_Connected_SMD -> FSFootprints:SMDNetTie
Connections:
- net labels added: CHARGER_OUT+_FUSED
Changed lines of the file:
@@
 Wire Wire Line
 	4250 3300 4150 3300
-Text Label 4250 1500 0    60   ~ 0
+Text Label 4550 1500 0    60   ~ 0
 CHARGER_OUT+
 Text Label 4150 2100 3    60   ~ 0
@@
 F 0 "R2" V 4580 900 50  0000 C CNN
 F 1 "R" V 4500 900 50  0000 C CNN
-F 2 "Oddities:NetTie-I_Connected_SMD" V 4430 900 50  0001 C CNN
+F 2 "FSFootprints:SMDNetTie" V 4430 900 50  0001 C CNN
 F 3 "" H 4500 900 50  0001 C CNN
 	1    4500 900
@@
 Wire Wire Line
 	1150 3200 1150 2550
+$Comp
+L Fuse F1
+U 1 1 5AA304A6
+P 4400 1500
+F 0 "F1" V 4480 1500 50  0000 C CNN
+F 1 "Fuse" V 4325 1500 50  0000 C CNN
+F 2 "Fuse_Holders_and_Fuses:Fuseholder5x20_vert_closed_Bulgin_FX0456" V 4330 1500 50  0001 C CNN
+F 3 "" H 4400 1500 50  0001 C CNN
+	1    4400 1500
+	0    1    1    0
+$EndComp
+Text Label 4150 1500 2    60   ~ 0
+CHARGER_OUT+_FUSED
 $EndSCHEMATC

Commit message: add diodes to relay coils among other things
Parts:
- removed R1: R, Resistors_THT:R_Axial_DIN0207_L6.3mm_D2.5mm_P10.16mm_Horizontal, symbol R
- removed U1: PS2501-1, Housings_DIP:DIP-4_W7.62mm, symbol PS2501-1
- added D1, D2, D3: D, Diodes_SMD:D_1206, symbol D
- added U1: G2RL-1A-E, FSFootprints:G2RL-1A-E, symbol G2RL-1A-E
- renumbered R2 to R1
Connections:
- wire segments 11 -> 12
Other:
- moved on the sheet: R1
Changed lines of the file:
@@
 NoConn ~ 1150 1350
-$Comp
-L PS2501-1 U1
-U 1 1 5A9F3852
-P 4050 800
-F 0 "U1" H 3850 1000 50  0000 L CNN
-F 1 "PS2501-1" H 3800 600 50  0000 L CNN
-F 2 "Housings_DIP:DIP-4_W7.62mm" H 3850 600 50  0001 L CIN
-F 3 "" H 4050 800 50  0000 L CNN
-	1    4050 800
-	1    0    0    -1
-$EndComp
-$Comp
-L R R1
-U 1 1 5A9F3A53
-P 3600 900
-F 0 "R1" V 3680 900 50  0000 C CNN
-F 1 "R" V 3600 900 50  0000 C CNN
-F 2 "Resistors_THT:R_Axial_DIN0207_L6.3mm_D2.5mm_P10.16mm_Horizontal" V 3530 900 50  0001 C CNN
-F 3 "" H 3600 900 50  0001 C CNN
-	1    3600 900
-	0    1    1    0
-$EndComp
 $Comp
 L GND #PWR01
@@
 	1    0    0    -1
 $EndComp
-Text Label 3450 900  2    60   ~ 0
+Text Label 3650 1150 2    60   ~ 0
 CHARGER_CONTROL
 $Comp
 L +12V #PWR05
 U 1 1 5A9F6CDD
-P 3750 700
-F 0 "#PWR05" H 3750 550 50  0001 C CNN
-F 1 "+12V" H 3750 840 50  0000 C CNN
-F 2 "" H 3750 700 50  0001 C CNN
-F 3 "" H 3750 700 50  0001 C CNN
-	1    3750 700
-	1    0    0    -1
-$EndComp
-Text Label 4350 700  0    60   ~ 0
+P 3650 850
+F 0 "#PWR05" H 3650 700 50  0001 C CNN
+F 1 "+12V" H 3650 990 50  0000 C CNN
+F 2 "" H 3650 850 50  0001 C CNN
+F 3 "" H 3650 850 50  0001 C CNN
+	1    3650 850
+	1    0    0    -1
+$EndComp
+Text Label 4250 700  0    60   ~ 0
 CHARGER_TEMP
 $Comp
-L R R2
+L R R1
 U 1 1 5A9F7258
-P 4500 900
-F 0 "R2" V 4580 900 50  0000 C CNN
-F 1 "R" V 4500 900 50  0000 C CNN
-F 2 "FSFootprints:SMDNetTie" V 4430 900 50  0001 C CNN
-F 3 "" H 4500 900 50  0001 C CNN
-	1    4500 900
-	0    1    1    0
-$EndComp
-Text Label 4650 900  0    60   ~ 0
+P 4650 1300
+F 0 "R1" V 4730 1300 50  0000 C CNN
+F 1 "R" V 4650 1300 50  0000 C CNN
+F 2 "FSFootprints:SMDNetTie" V 4580 1300 50  0001 C CNN
+F 3 "" H 4650 1300 50  0001 C CNN
+	1    4650 1300
+	0    1    1    0
+$EndComp
+Text Label 4800 1300 0    60   ~ 0
 CHARGER_OUT-
 $Comp
@@
 Text Label 6150 850  2    60   ~ 0
 CHARGER_TEMP
-Wire Wire Line
-	4350 900  4350 1100
-Wire Wire Line
-	4350 1100 6150 1100
-Wire Wire Line
-	6150 1100 6150 950
 $Comp
 L Conn_01x01 H2
@@
 Text Label 4150 1500 2    60   ~ 0
 CHARGER_OUT+_FUSED
+$Comp
+L D D2
+U 1 1 5ADA8471
+P 3650 1800
+F 0 "D2" H 3650 1900 50  0000 C CNN
+F 1 "D" H 3650 1700 50  0000 C CNN
+F 2 "Diodes_SMD:D_1206" H 3650 1800 50  0001 C CNN
+F 3 "" H 3650 1800 50  0001 C CNN
+	1    3650 1800
+	0    1    1    0
+$EndComp
+$Comp
+L D D3
+U 1 1 5ADA8662
+P 3650 3000
+F 0 "D3" H 3650 3100 50  0000 C CNN
+F 1 "D" H 3650 2900 50  0000 C CNN
+F 2 "Diodes_SMD:D_1206" H 3650 3000 50  0001 C CNN
+F 3 "" H 3650 3000 50  0001 C CNN
+	1    3650 3000
+	0    1    1    0
+$EndComp
+$Comp
+L G2RL-1A-E U1
+U 1 1 5ADA9EB0
+P 4150 1000
+F 0 "U1" H 4050 1000 60  0000 C CNN
+F 1 "G2RL-1A-E" V 4400 1000 60  0000 C CNN
+F 2 "FSFootprints:G2RL-1A-E" H 4150 1000 60  0001 C CNN
+F 3 "" H 4150 1000 60  0000 C CNN
+	1    4150 1000
+	1    0    0    -1
+$EndComp
+Wire Wire Line
+	4150 1300 4500 1300
+Connection ~ 4250 1300
+Wire Wire Line
+	4150 700  4250 700
+$Comp
+L D D1
+U 1 1 5ADAA4B8
+P 3650 1000
+F 0 "D1" H 3650 1100 50  0000 C CNN
+F 1 "D" H 3650 900 50  0000 C CNN
+F 2 "Diodes_SMD:D_1206" H 3650 1000 50  0001 C CNN
+F 3 "" H 3650 1000 50  0001 C CNN
+	1    3650 1000
+	0    1    1    0
+$EndComp
+Wire Wire Line
+	4500 1300 4500 950
+Wire Wire Line
+	4500 950  6150 950
 $EndSCHEMATC

Commit message: hopefully finalize PCBs for send to manufacturing
Parts:
- F1: footprint Fuse_Holders_and_Fuses:Fuseholder5x20_vert_closed_Bulgin_FX0456 -> FSFootprints:Fuseholder5x20_vert
Changed lines of the file:
@@
 LIBS:valves
 LIBS:arduino
-LIBS:ChargerSwitchbox-cache
 EELAYER 25 0
 EELAYER END
@@
 F 0 "F1" V 4480 1500 50  0000 C CNN
 F 1 "Fuse" V 4325 1500 50  0000 C CNN
-F 2 "Fuse_Holders_and_Fuses:Fuseholder5x20_vert_closed_Bulgin_FX0456" V 4330 1500 50  0001 C CNN
+F 2 "FSFootprints:Fuseholder5x20_vert" V 4330 1500 50  0001 C CNN
 F 3 "" H 4400 1500 50  0001 C CNN
 	1    4400 1500
