File: Temperature Shield/Temp Board.kicad_pcb (KiCad board)
At the start: 2 copper layers, 437 x 35.2 mm, 35 parts, among them P101 CONN_01X06, P102 Elithion_7_s, P103 Elithion_6_s, P104 Elithion_5_s, P105 Elithion_4_s, P106 Elithion_3_s, P107 Energus 7, P108 7_temp, P109 Elithion_2_s, P110 Elithion_1_s, P111 CONN_01X06, P112 Elithion_1_l, P114 Energus 6, P115 6_temp, P120 Energus 5, P121 5_temp, P126 Energus 4, P127 4_temp, P132 Energus 3, P133 3_temp, P138 Energus 2, P139 2_temp, P144 Energus 1, P147 1_temp, U101 MCP3008, U102 MCP3008, U103 SI8641, U104 SI8641

Commit message: rip
Parts:
- P101, P111: footprint Connectors_Molex:Molex_NanoFit_1x06x2.50mm_Straight -> Connectors_Molex:Molex_NanoFit_2x03x2.50mm_Straight
- moved R101 25.0 mm to (344.5, 79.0)
- moved P111 7.76 mm to (339.5, 77.0)
- moved U101 5.10 mm to (317.6, 77.4)
- moved U104 1.84 mm to (325.6, 77.4), turned to 180 degrees
Routing:
- net (no net): track 72.1 -> 74.0 mm

Commit message: Temp Board
Parts:
- removed U101, U102: MCP3008, Housings_SOIC:SOIC-16_3.9x9.9mm_Pitch1.27mm
- removed U103, U104: SI8641, Housings_SOIC:SOIC-16_3.9x9.9mm_Pitch1.27mm
- added P113: CONN_01X01, Mounting_Holes:MountingHole_4.3mm_M4_Pad, F.Cu at (61.5, 54.2)
- added P116: CONN_01X01, Mounting_Holes:MountingHole_4.3mm_M4_Pad, F.Cu at (493.5, 54.2)
- P101, P111: value CONN_01X06 -> CONN_01X08; footprint Connectors_Molex:Molex_NanoFit_2x03x2.50mm_Straight -> Connectors_JST:JST_XH_B09B-XH-A_09x2.50mm_Straight
- P108, P115, P121, P127, P133, P139, P147: footprint Connectors_Molex:Molex_NanoFit_1x02x2.50mm_Straight -> Connectors_JST:JST_XH_B02B-XH-A_02x2.50mm_Straight
- moved P101 185.8 mm to (93.8, 39.0), turned to 0 degrees
- moved R101 143.1 mm to (481.8, 38.5), turned to 270 degrees
- moved P108 141.4 mm to (486.2, 39.0)
- moved P102 134.4 mm to (487.5, 54.2)
- moved P103 134.4 mm to (417.5, 54.2)
- moved P104 134.4 mm to (347.5, 54.2)
- moved P105 134.4 mm to (277.5, 54.2)
- moved P106 134.4 mm to (207.5, 54.2)
- moved P109 134.4 mm to (137.5, 54.2)
- moved P110 134.4 mm to (67.5, 54.2)
- moved P112 134.4 mm to (71.5, 54.2)
- moved R102 134.3 mm to (411.8, 38.5), turned to 270 degrees
- moved P115 133.9 mm to (416.2, 39.0)
- moved P121 133.8 mm to (346.2, 39.0)
- moved P107 133.7 mm to (487.5, 54.2)
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Connections:
- P101 pad 1: Net-(P101-Pad1) -> +3V3
- P101 pad 2: Net-(P101-Pad2) -> 1_temp
- P101 pad 3: Net-(P101-Pad3) -> 2_temp
- P101 pad 4: Net-(P101-Pad4) -> 3_temp
- P101 pad 5: Net-(P101-Pad5) -> 4_temp
- P101 pad 6: Net-(P101-Pad6) -> 5_temp
- P111 pad 1: Net-(P111-Pad1) -> +3V3
- P111 pad 2: Net-(P111-Pad2) -> 1_temp
- P111 pad 3: Net-(P111-Pad3) -> 2_temp
- P111 pad 4: Net-(P111-Pad4) -> 3_temp
- P111 pad 5: Net-(P111-Pad5) -> 4_temp
- P111 pad 6: Net-(P111-Pad6) -> 5_temp
Routing:
- net GND: track 0.00 -> 441.0 mm, vias 0 -> 8
- net +3V3: track 0.00 -> 423.0 mm
- net 1_temp: track 0.00 -> 393.9 mm, vias 0 -> 1
- net 7_temp: track 0.00 -> 380.1 mm, vias 0 -> 1
- net 2_temp: track 0.00 -> 366.0 mm, vias 0 -> 2
- net 3_temp: track 0.00 -> 365.0 mm, vias 0 -> 2
- net 4_temp: track 0.00 -> 364.0 mm, vias 0 -> 2
- net 5_temp: track 0.00 -> 363.0 mm, vias 0 -> 2
- net 6_temp: track 0.00 -> 361.8 mm, vias 0 -> 2
- net 1_C+: track 8.13 -> 94.2 mm
- net 6_C+: track 0.00 -> 81.8 mm
- net 4_C+: track 0.00 -> 81.8 mm
- net 3_C+: track 0.00 -> 81.8 mm
- net 2_C+: track 0.00 -> 81.8 mm
- net 5_C+: track 0.00 -> 81.7 mm
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Other:
- board size 437 x 35.2 mm -> 436 x 30.8 mm
- net class Default: clearance 0.2 -> 0.1778; trace_width 0.25 -> 0.254
- rule trace_clearance: 0.2 -> 0.1778
- rule trace_min: 0.2 -> 0.254
- rule via_min_size: 0.4 -> 0.381

Commit message: temp shield FUCKINGSENDIT
Parts:
- removed P112: Elithion_1_l, FS FINAL:Elithion_Long
- added J1: Conn_01x02, Connectors_Molex:Molex_NanoFit_1x02x2.50mm_Straight, F.Cu at (91.2, 39.0)
- added J2: Conn_01x02, Connectors_Molex:Molex_NanoFit_1x02x2.50mm_Straight, F.Cu at (441.2, 39.0)
- P101, P111: value CONN_01X08 -> Conn_01x07; footprint Connectors_JST:JST_XH_B09B-XH-A_09x2.50mm_Straight -> Connectors_Molex:Molex_NanoFit_1x07x2.50mm_Straight
- P102, P103, P104, P105, P106, P109, P110: footprint FS FINAL:Elithion_Short -> FSFootprints:Elithion_R_A
- P107, P114, P120, P126, P132, P138, P144: footprint FS FINAL:Energus -> FSFootprints:Energus
- P113, P116: footprint Mounting_Holes:MountingHole_4.3mm_M4_Pad -> Mounting_Holes:MountingHole_3.2mm_M3_Pad
- R101, R102, R103, R104, R105, R106, R107: footprint Resistors_SMD:R_0805 -> Resistors_SMD:R_0805_HandSoldering
- moved P102 36.9 mm to (452.5, 66.0)
- moved P110 36.9 mm to (102.5, 66.0)
- moved R107 12.8 mm to (74.5, 39.0), turned to 180 degrees
- moved P103 11.8 mm to (417.5, 66.0)
- moved P104 11.8 mm to (347.5, 66.0)
- moved P105 11.8 mm to (277.5, 66.0)
- moved P106 11.8 mm to (207.5, 66.0)
- moved P109 11.8 mm to (137.5, 66.0)
- moved P101 5.00 mm to (98.8, 39.0)
- moved P111 5.00 mm to (448.8, 39.0)
- moved P113 3.50 mm to (65.0, 54.2)
- moved P116 3.50 mm to (490.0, 54.2)
- moved R101 1.35 mm to (480.5, 39.0), turned to 0 degrees
- moved R102 1.35 mm to (410.5, 39.0), turned to 0 degrees
- moved R103 1.35 mm to (340.5, 39.0), turned to 180 degrees
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Connections:
- P101 pad 1: +3V3 -> 1_temp
- P101 pad 2: 1_temp -> 2_temp
- P101 pad 3: 2_temp -> 3_temp
- P101 pad 4: 3_temp -> 4_temp
- P101 pad 5: 4_temp -> 5_temp
- P101 pad 6: 5_temp -> 6_temp
- P101 pad 7: 6_temp -> 7_temp
- P110 pad C-: 1_C- -> (no net)
- P111 pad 1: +3V3 -> 1_temp
- P111 pad 2: 1_temp -> 2_temp
- P111 pad 3: 2_temp -> 3_temp
- P111 pad 4: 3_temp -> 4_temp
- P111 pad 5: 4_temp -> 5_temp
- P111 pad 6: 5_temp -> 6_temp
- P111 pad 7: 6_temp -> 7_temp
Routing:
- net 1_C+: track 94.2 -> 26.1 mm
- net 6_C+: track 81.8 -> 26.1 mm
- net 7_B+: track 11.5 -> 48.1 mm
- net 1_B-: track 18.8 -> 48.1 mm
- net 2_C+: track 81.8 -> 61.1 mm
- net 3_C+: track 81.8 -> 61.1 mm
- net 4_C+: track 81.8 -> 61.1 mm
- net 5_C+: track 81.7 -> 61.1 mm
- net 5_B+: track 77.1 -> 64.2 mm
- net 4_B+: track 77.1 -> 64.2 mm
- net 3_B+: track 77.1 -> 64.2 mm
- net 2_B+: track 77.1 -> 64.2 mm
- net 6_B+: track 77.1 -> 64.6 mm
- net 1_B+: track 77.1 -> 64.6 mm
- net 7_temp: track 380.1 -> 388.5 mm
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Other:
- board size 436 x 30.8 mm -> 429 x 30 mm
- net class Default: clearance 0.1778 -> 0.24; via_dia 0.6 -> 0.8
- rule trace_clearance: 0.1778 -> 0.24

Commit message: hopefully finalize PCBs for send to manufacturing
Parts:
- removed P113, P116: CONN_01X01, Mounting_Holes:MountingHole_3.2mm_M3_Pad
- P107: footprint FSFootprints:Energus -> FSFootprints:Energus_End_R
- P144: footprint FSFootprints:Energus -> FSFootprints:Energus_End_L
Routing:
- net 7_B+: track 48.1 -> 33.6 mm
- net 1_B-: track 48.1 -> 33.6 mm
Other:
- board size 429 x 30 mm -> 432 x 30 mm

Commit message: Edit some component labels and other items for PCB send out
Changed lines of the file:
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@@
       (psnegative false)
       (psa4output false)
-      (plotreference false)
-      (plotvalue false)
+      (plotreference true)
+      (plotvalue true)
       (plotinvisibletext false)
       (padsonsilk false)
@@
   (module FSFootprints:Elithion_R_A (layer F.Cu)
     (at 452.5 66)
-    (fp_text reference P102 (at 0 0.5) (layer F.SilkS)
+    (fp_text reference P102 (at 0.25 -1.75) (layer F.SilkS)
       (effects (font (size 1 1) (thickness 0.15)))
     )
@@
   (module FSFootprints:Elithion_R_A (layer F.Cu)
     (at 417.5 66)
-    (fp_text reference P103 (at 0 0.5) (layer F.SilkS)
+    (fp_text reference P103 (at 0.25 -1.75) (layer F.SilkS)
       (effects (font (size 1 1) (thickness 0.15)))
     )
@@
   (module FSFootprints:Elithion_R_A (layer F.Cu)
     (at 347.5 66)
-    (fp_text reference P104 (at 0 0.5) (layer F.SilkS)
+    (fp_text reference P104 (at 0.25 -1.75) (layer F.SilkS)
       (effects (font (size 1 1) (thickness 0.15)))
     )
@@
   (module FSFootprints:Elithion_R_A (layer F.Cu)
     (at 277.5 66)
-    (fp_text reference P105 (at 0 0.5) (layer F.SilkS)
+    (fp_text reference P105 (at 0.25 -1.75) (layer F.SilkS)
       (effects (font (size 1 1) (thickness 0.15)))
     )
@@
   (module FSFootprints:Elithion_R_A (layer F.Cu)
     (at 207.5 66)
-    (fp_text reference P106 (at 0 0.5) (layer F.SilkS)
+    (fp_text reference P106 (at 0.25 -1.75) (layer F.SilkS)
       (effects (font (size 1 1) (thickness 0.15)))
     )
@@
   (module FSFootprints:Elithion_R_A (layer F.Cu)
     (at 137.5 66)
-    (fp_text reference P109 (at 0 0.5) (layer F.SilkS)
+    (fp_text reference P109 (at 0.25 -1.75) (layer F.SilkS)
       (effects (font (size 1 1) (thickness 0.15)))
     )
@@
   (module FSFootprints:Elithion_R_A (layer F.Cu)
     (at 102.5 66)
-    (fp_text reference P110 (at 0 0.5) (layer F.SilkS)
+    (fp_text reference P110 (at 0.25 -1.75) (layer F.SilkS)
       (effects (font (size 1 1) (thickness 0.15)))
     )
@@
   (module FSFootprints:Energus_End_R (layer F.Cu)
     (at 487.5 54.25)
-    (fp_text reference P107 (at 0 0.5) (layer F.SilkS)
+    (fp_text reference P107 (at -3.75 1) (layer F.SilkS)
       (effects (font (size 1 1) (thickness 0.15)))
     )
@@
   (module FSFootprints:Energus_End_L locked (layer F.Cu)
     (at 67.5 54.25)
-    (fp_text reference P144 (at 0 0.5) (layer F.SilkS)
-      (effects (font (size 1 1) (thickness 0.15)))
-    )
+    (fp_text reference P144 (at 3.25 1) (layer F.SilkS)
+      (effects (font (size 1 1) (thickness 0.15)))
+    )

Commit message: Fixed temp shields
Added serial connection between shields bc im dumb and forgot
Parts:
- added J3: Conn_01x02, Connectors_Molex:Molex_NanoFit_1x02x2.50mm_Straight, F.Cu at (488.8, 63.8)
- added J4: Conn_01x02, Connectors_Molex:Molex_NanoFit_1x02x2.50mm_Straight, F.Cu at (63.8, 63.8)
Connections:
- P102 pad C+: (no net) -> 7_C+
- P110 pad C-: (no net) -> 1_C-
Routing:
- net 7_C+: track 0.00 -> 35.3 mm
- net 1_C-: track 0.00 -> 35.3 mm
