File: TSAL/TSAL_2019/TSAL.sch (KiCad schematic (older format))
At the start: 50 parts, among them J1 Main Connector

Commit message: TSAL Schematic done
Parts:
- added D1: LT A6SG-V2AB-35-Z, FSFootprints:LED_SMD-2, symbol Device:LED_Small
- added D32, D33, D34, D35, D36, D37, D38, D39, D40, D41, D42, D43, D44, D45, D46, D47, D48, D49, D50, D51, D52, D53, D54, D55, D56, D57, D58, D59, D60: LR A67F-U2AB-1-1-30-R33-Z, FSFootprints:LED_SMD-2, symbol Device:LED_Small
- added Q1, Q4, Q?: TSM320N03CX, TO_SOT_Packages_SMD:SOT-23, symbol Device:Q_NMOS_GDS
- added R10, R11, R12, R13, R14, R15, R16, R17, R8, R9: 120, Resistors_SMD:R_0805_HandSoldering, symbol Device:R
- added R26, R4: 1k, Resistors_SMD:R_0805_HandSoldering, symbol Device:R_Small
- added R27, R6: 100k, Resistors_SMD:R_0805_HandSoldering, symbol Device:R_Small
- added R5: 100, Resistors_SMD:R_0805_HandSoldering, symbol Device:R_Small
- added R7, R?: 10k, Resistors_SMD:R_0805_HandSoldering, symbol Device:R_Small
- added R?: 4.7k, Resistors_SMD:R_0805_HandSoldering, symbol Device:R_Small
- C1: renamed from C?; footprint (none) -> Capacitors_SMD:C_0805_HandSoldering
- C2: renamed from C?; footprint (none) -> Capacitors_SMD:CP_Elec_5x5.3
- D10, D11, D12, D13, D14, D15, D16, D17, D18, D19, D2, D20, D21, D22, D23, D24, D25, D26, D27, D28, D29, D3, D30, D4, D5, D6, D7, D8, D9: value Led_Small -> LT A6SG-V2AB-35-Z
- D31: renamed from D1; value Led_Small -> LR A67F-U2AB-1-1-30-R33-Z
- J1: footprint Connectors_Molex:Molex_NanoFit_2x02x2.50mm_Straight -> Connectors_Molex:Molex_NanoFit_1x04x2.50mm_Angled
- Q2: renamed from Q?; value Q_NMOS_DGS -> TSM320N03CX; footprint (none) -> TO_SOT_Packages_SMD:SOT-23; symbol Device:Q_NMOS_DGS -> Device:Q_NMOS_GDS
- R1: renamed from R?; value R -> 10k; footprint (none) -> Resistors_SMD:R_0805_HandSoldering; symbol Device:R -> Device:R_Small
- R2, R3: renamed from R?; footprint (none) -> Resistors_SMD:R_0805_HandSoldering; symbol Device:R -> Device:R_Small
- U1: renamed from U?; footprint (none) -> Housings_SOIC:SOIC-8_3.9x4.9mm_Pitch1.27mm
- renumbered R3 to R20, R4 to R21, R5 to R22, R6 to R23, R7 to R24, R8 to R25
Connections:
- net labels added: Reset
- net labels removed: OSC, RTDS_H
- wire segments 38 -> 134
Other:
- note added: "Green LEDs"
- note added: "Red LEDs"
- moved on the sheet: C1, C2, D31, LS1, LS2, R1, R2, R20, R21, R22, R23, R24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
