File: BMS/BMS.sch (KiCad schematic (older format))
At the start: 39 parts

Commit message: Updated BMS Schematics
Parts:
- added C? (x3): 1uF, symbol Device:C
- added C?: .1uF, symbol Device:C
- added J?: Conn_01x02_Male, symbol Connector:Conn_01x02_Male
- added Q?: Q_NPN_BCEC, symbol Device:Q_NPN_BCEC
- added R? (x4): 10k, symbol Device:R
- added R?: 100, symbol Device:R
- added R? (x2): R, symbol Device:R
- added R?: 1M, symbol Device:R
- added SW?: SW_DIP_x04, symbol Switch:SW_DIP_x04
- added T?: Transformer_1P_1S, symbol Device:Transformer_1P_1S
Connections:
- net labels added: +5V, +BATT, GND
- wire segments 140 -> 184

Commit message: BMS update
Parts:
- removed R? (x3): 10k, symbol Device:R
- added R6, R7, R8: 10k, Resistors_SMD:R_0805_HandSoldering, symbol Device:R
- C1, C10, C11, C2, C3, C4, C5, C6, C7, C8, C9: renamed from C?; footprint (none) -> Capacitors_SMD:C_0805_HandSoldering
- J1: renamed from J?; value Conn_01x08_Male -> Cell Taps; footprint (none) -> FSFootprints:Cell Taps
- Q1: renamed from Q?; value Q_NPN_BCEC -> NSV1C201MZ4; footprint (none) -> TO_SOT_Packages_SMD:SOT-223
- Q2, Q3, Q4, Q5, Q6, Q7, Q8: renamed from Q?; footprint Package_TO_SOT_SMD:SOT-23 -> TO_SOT_Packages_SMD:SOT-23
- R1, R10, R11, R12, R13, R15, R16, R17, R19, R2, R20, R22, R23, R25, R26, R28, R29, R3, R31, R4, R5: renamed from R?; footprint (none) -> Resistors_SMD:R_0805_HandSoldering
- R14, R18, R21, R24, R27, R30, R9: renamed from R?; footprint (none) -> Resistors_SMD:R_2512_HandSoldering
- SW1: renamed from SW?; footprint (none) -> Buttons_Switches_SMD:SW_DIP_x4_W8.61mm_Slide_LowProfile
- U1: renamed from U?; footprint (none) -> Housings_SSOP:SSOP-48_7.5x15.9mm_Pitch0.635mm; symbol FS_FINAL:LTC6811 -> BMS-rescue:LTC6811-FS_FINAL
- gave numbers to parts that had none: 2
Connections:
- net labels added: A0, A1, A2, A3, V-, VREG
- net labels removed: +5V, +BATT, GND
- wire segments 184 -> 210
Other:
- moved on the sheet: C1, C3, C6, C7, Q1, R12, R13, R17, R2, R5, SW1

Commit message: Updated BMS
Parts:
- removed T1: Transformer_1P_1S, symbol Device:Transformer_1P_1S
- added C12: 15pF, Capacitors_SMD:C_0805_HandSoldering, symbol Device:C
- added C13, C14: 1uF, Capacitors_SMD:C_0805_HandSoldering, symbol Device:C_Small
- added J10: Current Sensor, Connectors_Molex:Molex_NanoFit_1x03x2.50mm_Straight, symbol Connector:Conn_01x03_Male
- added J3: Temp 1, Connectors_Molex:Molex_NanoFit_1x02x2.50mm_Straight, symbol Connector:Conn_01x02_Male
- added J4: Temp 2, Connectors_Molex:Molex_NanoFit_1x02x2.50mm_Straight, symbol Connector:Conn_01x02_Male
- added J5: Temp 3, Connectors_Molex:Molex_NanoFit_1x02x2.50mm_Straight, symbol Connector:Conn_01x02_Male
- added J6: Temp 4, Connectors_Molex:Molex_NanoFit_1x02x2.50mm_Straight, symbol Connector:Conn_01x02_Male
- added J7: Temp 5, Connectors_Molex:Molex_NanoFit_1x02x2.50mm_Straight, symbol Connector:Conn_01x02_Male
- added J8: Temp 6, Connectors_Molex:Molex_NanoFit_1x02x2.50mm_Straight, symbol Connector:Conn_01x02_Male
- added J9: Temp 7, Connectors_Molex:Molex_NanoFit_1x02x2.50mm_Straight, symbol Connector:Conn_01x02_Male
- added L1: HM2113ZNL, FSFootprints:HM2113ZNL, symbol FS_FINAL:HM2113ZNL
- added R32: 402, Resistors_SMD:R_0805_HandSoldering, symbol Device:R
- added R33, R34, R35, R36, R37, R38, R39: R, Resistors_SMD:R_0805_HandSoldering, symbol Device:R
- added R40, R41: 22, Resistors_SMD:R_0805_HandSoldering, symbol Device:R
- added U2: ADG708, Package_SO:TSSOP-16_4.4x5mm_P0.65mm, symbol FS_FINAL:ADG708
- J2: value Conn_01x02_Male -> IsoSPI; footprint (none) -> Connectors_Molex:Molex_NanoFit_1x02x2.50mm_Straight
Connections:
- net labels added: IBIAS, ICMP, IMA, IPA, MUX_A0, MUX_A1, MUX_A2, TEMP
- wire segments 210 -> 233
Other:
- moved on the sheet: C1, C10, C11, C2, C3, C4, C5, C6, C7, C8, C9, J1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
