File: TSAL/TSAL/TSAL.sch (KiCad schematic (older format))
At the start: 51 parts, among them J1 CONN_01X04, U1 L78S05CV-DG, U2 LM555N

Commit message: Need to correct Bay Area DFM warnings on TSAL. Brake Light passed and ready to be sent.
Parts:
- added J2, J3, J4, J5: Conn_01x01, Mounting_Holes:MountingHole_3.2mm_M3, symbol Conn_01x01
Changed lines of the file:
@@
 	1    0    0    -1
 $EndComp
+$Comp
+L Conn_01x01 J2
+U 1 1 5AA25485
+P 3900 5150
+F 0 "J2" H 3900 5250 50  0000 C CNN
+F 1 "Conn_01x01" H 3900 5050 50  0000 C CNN
+F 2 "Mounting_Holes:MountingHole_3.2mm_M3" H 3900 5150 50  0001 C CNN
+F 3 "" H 3900 5150 50  0001 C CNN
+	1    3900 5150
+	-1   0    0    1
+$EndComp
+$Comp
+L Conn_01x01 J3
+U 1 1 5AA2591E
+P 3900 5400
+F 0 "J3" H 3900 5500 50  0000 C CNN
+F 1 "Conn_01x01" H 3900 5300 50  0000 C CNN
+F 2 "Mounting_Holes:MountingHole_3.2mm_M3" H 3900 5400 50  0001 C CNN
+F 3 "" H 3900 5400 50  0001 C CNN
+	1    3900 5400
+	-1   0    0    1
+$EndComp
+$Comp
+L Conn_01x01 J4
+U 1 1 5AA259D3
+P 3900 5650
+F 0 "J4" H 3900 5750 50  0000 C CNN
+F 1 "Conn_01x01" H 3900 5550 50  0000 C CNN
+F 2 "Mounting_Holes:MountingHole_3.2mm_M3" H 3900 5650 50  0001 C CNN
+F 3 "" H 3900 5650 50  0001 C CNN
+	1    3900 5650
+	-1   0    0    1
+$EndComp
+$Comp
+L Conn_01x01 J5
+U 1 1 5AA25A8B
+P 3900 5900
+F 0 "J5" H 3900 6000 50  0000 C CNN
+F 1 "Conn_01x01" H 3900 5800 50  0000 C CNN
+F 2 "Mounting_Holes:MountingHole_3.2mm_M3" H 3900 5900 50  0001 C CNN
+F 3 "" H 3900 5900 50  0001 C CNN
+	1    3900 5900
+	-1   0    0    1
+$EndComp
 $EndSCHEMATC

Commit message: Updated TSAL. passed DFM
Parts:
- LS1, LS2: footprint FSfootprints:RTDS_H -> Connectors_Molex:Molex_NanoFit_1x02x2.50mm_Straight
Changed lines of the file:
@@
 LIBS:FS FINAL
 LIBS:symbols
-LIBS:TSAL-cache
 EELAYER 25 0
 EELAYER END
@@
 F 0 "LS1" H 4350 3375 50  0000 R CNN
 F 1 "RTDS Piezo" H 4650 3300 50  0000 R CNN
-F 2 "FSfootprints:RTDS_H" H 4300 2950 50  0001 C CNN
+F 2 "Connectors_Molex:Molex_NanoFit_1x02x2.50mm_Straight" H 4300 2950 50  0001 C CNN
 F 3 "" H 4290 3100 50  0001 C CNN
 	1    4300 3150
@@
 F 0 "LS2" H 5300 3375 50  0000 R CNN
 F 1 "RTDS Piezo" H 5600 3300 50  0000 R CNN
-F 2 "FSfootprints:RTDS_H" H 5250 2950 50  0001 C CNN
+F 2 "Connectors_Molex:Molex_NanoFit_1x02x2.50mm_Straight" H 5250 2950 50  0001 C CNN
 F 3 "" H 5240 3100 50  0001 C CNN
 	1    5250 3150

Commit message: Some changes to hopefully make some projects openable in Kicad 5 and 6
Parts:
- C301, C303: symbol CP -> Device:CP
- C302: symbol C -> Device:C
- D301, D302, D303, D304, D305, D306, D307, D308, D309, D310, D311, D312, D313, D314, D315, D316, D317, D318, D319, D320, D321, D322, D323, D324, D325, D326, D327, D328, D329, D330, D331, D332: symbol LED_Small -> Device:LED_Small
- H301: symbol SN754410 -> FS-FINAL:SN754410
- J1: symbol Conn_01x04 -> TSAL-rescue:Conn_01x04
- J2, J3, J4, J5: symbol Conn_01x01 -> TSAL-rescue:Conn_01x01
- LS1, LS2: symbol Speaker -> Device:Speaker
- R301, R302, R303, R304, R305, R306, R307, R308, R309, R310: symbol R -> Device:R
- U1: symbol L78S05CV-DG -> FS-FINAL:L78S05CV-DG
- U2: symbol LM555N -> FS-FINAL:LM555N
Connections:
- wire segments 55 -> 82
